File: kicad/pogo-block-1.kicad_sch (KiCad schematic)
At the start: 22 parts, among them J3 ALT_BP_L, J4 ALT_BP_R, SW1 GAIN_MAIN, SW2 GAIN_BP3, U2 OPA1612, U3 OPA1612

Commit message: kicad: block-8 LP2 + fix multi-unit op-amp placement bug (7 of 10)
block-8 (LP2): OTA-C SVF mirroring LP1 minus tilt (single shared expo); Q VCA via
the shared-q sheet cell B (U9/U10); added LP2's own IRES_AMP (U65, was missing from
the BOM) + full SVF expansion (R_LIN, expo network, Q V->I, buffer pulldowns,
decoupling). 51 parts / 36 nets; LP2 boundary nets match shared-q byte-for-byte.
shared-q gains the LP2 cell-B Iabc bypass caps (C84/C85).

GENERATOR CORRECTNESS FIX (exposed by block-8's spare op-amp half): dual op-amps
were placed as a single instance while pins from BOTH halves were connected at the
lib_symbol's overlapping origin -> unit-A and unit-B pins landed on the same canvas
point, shorting the two halves. This was latent in EVERY dual-op-amp block (A,B,1,2,
4,5). Fix:
- place each gate unit (A/B/power) as its own instance at distinct offsets
  (MULTI_UNIT + opamp_unit_pins);
- make structural_check unit-aware (per-sub-symbol unit pins);
- add a short detector: 2+ distinct nets whose labels coincide at one point now fail.
All blocks regenerated and re-verified clean (the detector finds no shorts).

STATUS+plan: 7/10 blocks. All gates green.
Parts:
- added J3: ALT_BP_L, POGO_Connector_Audio:Jack_3.5mm_QingPu_WQP-PJ398SM_Vertical_CircularHoles, symbol Device:Audio_Jack_3.5mm_SwitchT
- added J4: ALT_BP_R, POGO_Connector_Audio:Jack_3.5mm_QingPu_WQP-PJ398SM_Vertical_CircularHoles, symbol Device:Audio_Jack_3.5mm_SwitchT
- added SW1: GAIN_MAIN, POGO_Button_Switch_THT:SW_Dailywell_DW3_DPDT, symbol Switch:SW_Dailywell_DW3
- added SW2: GAIN_BP3, POGO_Button_Switch_THT:SW_Dailywell_DW3_DPDT, symbol Switch:SW_Dailywell_DW3
- C3: renamed from SW1; value GAIN_MAIN -> 100nF; footprint POGO_Button_Switch_THT:SW_Dailywell_DW3_DPDT -> (none); symbol Switch:SW_Dailywell_DW3 -> Device:C
- C4: renamed from SW2; value GAIN_BP3 -> 100nF; footprint POGO_Button_Switch_THT:SW_Dailywell_DW3_DPDT -> (none); symbol Switch:SW_Dailywell_DW3 -> Device:C
- C5: renamed from J3; value ALT_BP_L -> 100nF; footprint POGO_Connector_Audio:Jack_3.5mm_QingPu_WQP-PJ398SM_Vertical_CircularHoles -> (none); symbol Device:Audio_Jack_3.5mm_SwitchT -> Device:C
- C6: renamed from J4; value ALT_BP_R -> 100nF; footprint POGO_Connector_Audio:Jack_3.5mm_QingPu_WQP-PJ398SM_Vertical_CircularHoles -> (none); symbol Device:Audio_Jack_3.5mm_SwitchT -> Device:C
- D8: renamed from C5; value 100nF -> BAT54S; footprint (none) -> POGO_Package_TO_SOT_SMD:SOT-23; symbol Device:C -> Diode:BAT54S
- D9: renamed from C6; value 100nF -> BAT54S; footprint (none) -> POGO_Package_TO_SOT_SMD:SOT-23; symbol Device:C -> Diode:BAT54S
- R38: renamed from C3; value 100nF -> 100R; symbol Device:C -> Device:R
- R39: renamed from C4; value 100nF -> 100R; symbol Device:C -> Device:R
- R5L: renamed from R38; value 100R -> 4k7
- R5R: renamed from R39; value 100R -> 4k7
- R6L: renamed from D8; value BAT54S -> 18k; footprint POGO_Package_TO_SOT_SMD:SOT-23 -> (none); symbol Diode:BAT54S -> Device:R
- R6R: renamed from D9; value BAT54S -> 18k; footprint POGO_Package_TO_SOT_SMD:SOT-23 -> (none); symbol Diode:BAT54S -> Device:R
- U2: renamed from R3L; value 4k7 -> OPA1612; symbol Device:R -> Amplifier_Operational:OPA1612
- U2: renamed from U3; footprint POGO_Package_SO:SOIC-8_3.9x4.9mm_P1.27mm -> (none)
- U3: renamed from R4L; value 18k -> OPA1612; symbol Device:R -> Amplifier_Operational:OPA1612
- U3: renamed from R3R; value 4k7 -> OPA1612; footprint (none) -> POGO_Package_SO:SOIC-8_3.9x4.9mm_P1.27mm; symbol Device:R -> Amplifier_Operational:OPA1612
- U3: renamed from R4R; value 18k -> OPA1612; symbol Device:R -> Amplifier_Operational:OPA1612
- renumbered R5L to R3L, R5R to R3R, R6L to R4L, R6R to R4R
Connections:
- net +12V: now also C3.2, C5.2, D8.3 (K2), D9.3 (K2), U2.4 (V-), U3.4 (V-); no longer D8.2, R38.2, R6L.3 (K2), R6R.3 (K2)
- net -12V: now also C4.2, C6.2, D8.1 (A1), D9.1 (A1), U2.8 (V+), U3.8 (V+); no longer D9.2, R39.2, R6L.1 (A1), R6R.1 (A1)
- net ALT5X_L: now also R6L.1, U3.1 (Out), SW2.6 (B2); no longer C4.3 (A2), C4.6 (B2), R4L.1, R4R.1, U2.1 (Out)
- net ALT_L_IN: now also R38.1, U3.2 (In-), SW2.4 (B1); no longer C4.1 (A1), C4.4 (B1), R5L.1, R5R.1, U2.2 (In-)
- net ALT_L_TIP: now also R38.2, J3.1 (T); no longer C5.1 (T), R5L.2
- net ALT_OUT_L: now also SW2.5 (B_COM); no longer C4.5 (B_COM)
- net ALT_OUT_R: now also SW2.2 (A_COM); no longer C4.2 (A_COM)
- net ALT_R_TIP: now also R39.2, J4.1 (T); no longer C6.1 (T), R5R.2
- net GND: now also C3.1 (+), C4.1 (+), C5.1 (+), C6.1 (+), R5L.1, R5R.1, J3.2 (S), J4.2 (S); no longer C5.2 (S), C6.2 (S), D8.1 (+), D9.1 (+), R38.1 (+), R39.1 (+), U2.1, U3.1
- net L_OUT: now also SW1.4 (B1); no longer C3.1 (A1), C3.4 (B1)
- net PG5X_L: now also R4L.1, SW1.6 (B2); no longer C3.3 (A2), C3.6 (B2), U3.1, U3.1
- net PG_OUT_L: now also SW1.5 (B_COM); no longer C3.5 (B_COM)
- net PG_OUT_R: now also SW1.2 (A_COM); no longer C3.2 (A_COM)
- net U2A_INV: now also R3L.2, R4L.2; no longer U2.2, U3.2, U3.2, U3.2
- net U3A_INV: now also R5L.2, R6L.2, U3.3 (In+); no longer R3L.2, R3R.2, R4L.2, R4R.2, U2.3 (In+)
- net U3B_INV: now reaches R6R.2
- net U3B_INV: now also R5R.2, U3.5 (In+)
- new net ALT5X_R: R6R.1, SW2.3 (A2), U3.7 (Out)
- new net ALT_R_IN: R39.1, SW2.1 (A1), U3.6 (In-)
- new net PG5X_R: R4R.1, SW1.3 (A2), U2.7 (Out)
- new net R_OUT: SW1.1 (A1), U2.6 (In-)
- new net U2B_INV: R3R.2, R4R.2, U2.5 (In+)
Other:
- moved on the sheet: R3L, R3R, R4L, R4R, R5L, R5R, U2B, U2C, U3C
