File: kicad/pogo-block-2.kicad_sch (KiCad schematic)
At the start: 28 parts, among them J5 LFO1, J6 LFO2, U1 TL072, U2 TL072

Commit message: kicad: block-8 LP2 + fix multi-unit op-amp placement bug (7 of 10)
block-8 (LP2): OTA-C SVF mirroring LP1 minus tilt (single shared expo); Q VCA via
the shared-q sheet cell B (U9/U10); added LP2's own IRES_AMP (U65, was missing from
the BOM) + full SVF expansion (R_LIN, expo network, Q V->I, buffer pulldowns,
decoupling). 51 parts / 36 nets; LP2 boundary nets match shared-q byte-for-byte.
shared-q gains the LP2 cell-B Iabc bypass caps (C84/C85).

GENERATOR CORRECTNESS FIX (exposed by block-8's spare op-amp half): dual op-amps
were placed as a single instance while pins from BOTH halves were connected at the
lib_symbol's overlapping origin -> unit-A and unit-B pins landed on the same canvas
point, shorting the two halves. This was latent in EVERY dual-op-amp block (A,B,1,2,
4,5). Fix:
- place each gate unit (A/B/power) as its own instance at distinct offsets
  (MULTI_UNIT + opamp_unit_pins);
- make structural_check unit-aware (per-sub-symbol unit pins);
- add a short detector: 2+ distinct nets whose labels coincide at one point now fail.
All blocks regenerated and re-verified clean (the detector finds no shorts).

STATUS+plan: 7/10 blocks. All gates green.
Parts:
- added J5: LFO1, POGO_Connector_Audio:Jack_3.5mm_QingPu_WQP-PJ398SM_Vertical_CircularHoles, symbol Device:Audio_Jack_3.5mm_SwitchT
- added J6: LFO2, POGO_Connector_Audio:Jack_3.5mm_QingPu_WQP-PJ398SM_Vertical_CircularHoles, symbol Device:Audio_Jack_3.5mm_SwitchT
- added RV1: LFO1_RATE, POGO_Potentiometer_THT:Potentiometer_Bourns_3296W_Vertical, symbol Device:R_POT
- added RV2: LFO2_RATE, POGO_Potentiometer_THT:Potentiometer_Bourns_3296W_Vertical, symbol Device:R_POT
- C1: renamed from C5A; value 100nF -> 47nF
- C2: renamed from C5B; value 100nF -> 47nF
- C3A: renamed from R1; value 590k -> 100nF; symbol Device:R -> Device:C
- C3B: renamed from R2; value 590k -> 100nF; symbol Device:R -> Device:C
- C5A: renamed from R3; value 2k4 -> 100nF; symbol Device:R -> Device:C
- C5B: renamed from R4; value 2k4 -> 100nF; symbol Device:R -> Device:C
- D1: renamed from RV1; value LFO1_RATE -> 1N4148W; footprint POGO_Potentiometer_THT:Potentiometer_Bourns_3296W_Vertical -> POGO_Diode_SMD:D_SOD-123; symbol Device:R_POT -> Device:D
- D2: renamed from RV2; value LFO2_RATE -> 1N4148W; footprint POGO_Potentiometer_THT:Potentiometer_Bourns_3296W_Vertical -> POGO_Diode_SMD:D_SOD-123; symbol Device:R_POT -> Device:D
- LED1: renamed from J5; footprint POGO_Connector_Audio:Jack_3.5mm_QingPu_WQP-PJ398SM_Vertical_CircularHoles -> POGO_LED_THT:LED_D3.0mm; symbol Device:Audio_Jack_3.5mm_SwitchT -> Device:LED
- LED2: renamed from J6; footprint POGO_Connector_Audio:Jack_3.5mm_QingPu_WQP-PJ398SM_Vertical_CircularHoles -> POGO_LED_THT:LED_D3.0mm; symbol Device:Audio_Jack_3.5mm_SwitchT -> Device:LED
- R1: renamed from R5; value 100k -> 590k
- R10: renamed from D2; value 1N4148W -> 1k2; footprint POGO_Diode_SMD:D_SOD-123 -> (none); symbol Device:D -> Device:R
- R11: renamed from LED1; value LFO1 -> 1k; footprint POGO_LED_THT:LED_D3.0mm -> (none); symbol Device:LED -> Device:R
- R12: renamed from LED2; value LFO2 -> 1k; footprint POGO_LED_THT:LED_D3.0mm -> (none); symbol Device:LED -> Device:R
- R2: renamed from R6; value 100k -> 590k
- R3: renamed from R7; value 82k -> 2k4
- R4: renamed from R8; value 82k -> 2k4
- R5: renamed from R9; value 1k2 -> 100k
- R6: renamed from R10; value 1k2 -> 100k
- R7: renamed from R11; value 1k -> 82k
- R8: renamed from R12; value 1k -> 82k
- R9: renamed from D1; value 1N4148W -> 1k2; footprint POGO_Diode_SMD:D_SOD-123 -> (none); symbol Device:D -> Device:R
- U1: renamed from C1; value 47nF -> TL072; symbol Device:C -> Amplifier_Operational:OPA1612
- U1: renamed from U2; footprint POGO_Package_SO:SOIC-8_3.9x4.9mm_P1.27mm -> (none)
- U2: renamed from C3A; value 100nF -> TL072; symbol Device:C -> Amplifier_Operational:OPA1612
- U2: renamed from C2; value 47nF -> TL072; footprint (none) -> POGO_Package_SO:SOIC-8_3.9x4.9mm_P1.27mm; symbol Device:C -> Amplifier_Operational:OPA1612
- U2: renamed from C3B; value 100nF -> TL072; symbol Device:C -> Amplifier_Operational:OPA1612
Connections:
- net +12V: now also C3A.2, C5A.2, U1.4 (V-), U2.4 (V-); no longer C1.2, U2.2
- net -12V: now also C3B.2, C5B.2, U1.8 (V+), U2.8 (V+); no longer C2.2, U2.2
- net DLEDK1: now also D1.A, R9.2; no longer R5.2, R9.A
- net DLEDK2: now also D2.A, R10.2; no longer R10.A, R6.2
- net FLOORN1: now also R3.2, RV1.3; no longer C5A.2, D1.3
- net FLOORN2: now also R4.2, RV2.3; no longer C5B.2, D2.3
- net GND: now also C3A.1 (+), C3B.1 (+), LED1.A, LED2.A, R7.1, R8.1, U2.2 (In-), J5.2 (S), J6.2 (S); no longer C1.1 (+), C2.1 (+), LED1.2 (S), LED2.2 (S), R1.1, R11.A, R12.A, R2.1, R3.2, R4.2, U1.2 (In-), U2.1 (+), U2.1 (+)
- net LEDA1: now also LED1.K, R9.1; no longer R11.K, R5.1
- net LEDA2: now also LED2.K, R10.1; no longer R12.K, R6.1
- net LFO1_OUT: now also R11.1, J5.1 (T); no longer LED1.1 (T), R7.1
- net LFO2_OUT: now also R12.1, J6.1 (T); no longer LED2.1 (T), R8.1
- net SUM1: now also C1.1 (+), R1.1; no longer C3A.1, D1.1, R1.2, R7.2, R9.K, U1.1 (+), U1.1 (Out), U1.2
- net SUM2: now also C2.1 (+), R2.1, U2.3 (In+); no longer C3B.1, D2.1, R10.K, R2.2, R8.2, U1.1 (Out), U1.3 (In+), U2.1 (+), U2.2
- net WIPER1: now also R1.2, RV1.2 (Wiper); no longer C3A.2, D1.2 (Wiper)
- net WIPER2: now also R2.2, RV2.2 (Wiper); no longer C3B.2, D2.2 (Wiper)
- new net HYS1: R5.1, R7.2, U1.6 (In-)
- new net HYS2: R6.1, R8.2, U2.6 (In-)
- new net V_SQ1: R5.2, RV1.1, U1.7 (Out)
- new net V_SQ2: R6.2, RV2.1, U2.7 (Out)
- new net V_TRI1: C1.2, D1.K, R11.2, U1.1 (Out), U1.5 (In+)
- new net V_TRI2: C2.2, D2.K, R12.2, U2.1 (Out), U2.5 (In+)
Other:
- moved on the sheet: C1, C2, LED1, LED2, R1, R2, R3, R4, R5, R6, R7, R8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
