File: kicad/pogo-block-2.kicad_sch (KiCad schematic)
At the start: 28 parts, among them J5 LFO1, J6 LFO2, U1 TL072, U2 TL072

Commit message: 0015-lfo-rate-panel-pot: LFO Rate → 9mm log panel pot (like attenuverters)
LFO1/2 Rate (block-2 RV1/RV2) were specced as Bourns 3296W screwdriver
trimmers despite being front-panel controls. The plugin (Trimpot widget)
and panel (type: trimpot) already treat them like the attenuverters; only
the hardware part diverged. Swap to the attenuverter panel-pot family:

- components.yaml + block-2.nets.yaml RV1/RV2: 'Bourns 3296W'/through-hole
  -> 'log pot'/9mm (resolves to Alpha RD901F-40, the attenuverter footprint)
- block-2/spec.md: 9mm log panel pot, player-adjustable; drive-attenuator
  topology retained; log taper gives the ~exponential rate sweep matching
  the plugin 0.05x400^param law; prototype-verify note on wiper loading
- aux-lfo-core.md: resolved the stale Phase-3R taper open-item + superseded
  vary-R_int table -> drive-attenuator + 9mm log panel pot
- regenerated pogo-block-2.kicad_sch + pogo-bom.csv

Plugin/panel unchanged (no DSP, no panel geometry). All 5 gates green.

https://claude.ai/code/session_01MsjDdC2SbAb3J3qGafGBjk
Parts:
- RV1, RV2: footprint POGO_Potentiometer_THT:Potentiometer_Bourns_3296W_Vertical -> POGO_Potentiometer_THT:Potentiometer_Alpha_RD901F-40-00D_Single_Vertical_CircularHoles
Changed lines of the file:
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@@
   (property "Value" "LFO1_RATE" (at 43.000 479.500 0)
     (effects (font (size 1.016 1.016)) (justify left) (hide yes)))
-  (property "Footprint" "POGO_Potentiometer_THT:Potentiometer_Bourns_3296W_Vertical" (at 40.000 480.000 0)
+  (property "Footprint" "POGO_Potentiometer_THT:Potentiometer_Alpha_RD901F-40-00D_Single_Vertical_CircularHoles" (at 40.000 480.000 0)
     (effects (font (size 1.016 1.016)) (hide yes)))
 )
@@
   (property "Value" "LFO2_RATE" (at 103.000 479.500 0)
     (effects (font (size 1.016 1.016)) (justify left) (hide yes)))
-  (property "Footprint" "POGO_Potentiometer_THT:Potentiometer_Bourns_3296W_Vertical" (at 100.000 480.000 0)
+  (property "Footprint" "POGO_Potentiometer_THT:Potentiometer_Alpha_RD901F-40-00D_Single_Vertical_CircularHoles" (at 100.000 480.000 0)
     (effects (font (size 1.016 1.016)) (hide yes)))
 )
