File: kicad/pogo-block-2.kicad_sch (KiCad schematic)
At the start: 28 parts, among them J5 LFO1, J6 LFO2, U1 TL072, U2 TL072

Commit message: 0016: source Song Huei R0904N + repoint panel-pot BOM refs (G6a)
- new part components/parts/songhuei_r0904n (matches lin/log/bipolar pot)
- move taper tags off alpha_rd901f (keeps knob/large/xl knob)
- RV41/RV43 (HP_RES/LP2_RES) Bourns 3296W -> R0904N finger pot
- regen block-2/3/4 schematics (att/LFO/VCA pot footprint) + BOM
Parts:
- RV1, RV2: footprint POGO_Potentiometer_THT:Potentiometer_Alpha_RD901F-40-00D_Single_Vertical_CircularHoles -> POGO_Potentiometer_THT:Potentiometer_Songhuei_9mm_TallTrimmer_Vertical
Changed lines of the file:
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@@
   (property "Value" "LFO1_RATE" (at 43.000 479.500 0)
     (effects (font (size 1.016 1.016)) (justify left) (hide yes)))
-  (property "Footprint" "POGO_Potentiometer_THT:Potentiometer_Alpha_RD901F-40-00D_Single_Vertical_CircularHoles" (at 40.000 480.000 0)
+  (property "Footprint" "POGO_Potentiometer_THT:Potentiometer_Songhuei_9mm_TallTrimmer_Vertical" (at 40.000 480.000 0)
     (effects (font (size 1.016 1.016)) (hide yes)))
 )
@@
   (property "Value" "LFO2_RATE" (at 103.000 479.500 0)
     (effects (font (size 1.016 1.016)) (justify left) (hide yes)))
-  (property "Footprint" "POGO_Potentiometer_THT:Potentiometer_Alpha_RD901F-40-00D_Single_Vertical_CircularHoles" (at 100.000 480.000 0)
+  (property "Footprint" "POGO_Potentiometer_THT:Potentiometer_Songhuei_9mm_TallTrimmer_Vertical" (at 100.000 480.000 0)
     (effects (font (size 1.016 1.016)) (hide yes)))
 )
