File: kicad/pogo-block-4.kicad_sch (KiCad schematic)
At the start: 28 parts, among them J26 VCA_IN, U4 THAT2180, U5 THAT2180, U6 TL072, U63 TL072

Commit message: kicad: block-8 LP2 + fix multi-unit op-amp placement bug (7 of 10)
block-8 (LP2): OTA-C SVF mirroring LP1 minus tilt (single shared expo); Q VCA via
the shared-q sheet cell B (U9/U10); added LP2's own IRES_AMP (U65, was missing from
the BOM) + full SVF expansion (R_LIN, expo network, Q V->I, buffer pulldowns,
decoupling). 51 parts / 36 nets; LP2 boundary nets match shared-q byte-for-byte.
shared-q gains the LP2 cell-B Iabc bypass caps (C84/C85).

GENERATOR CORRECTNESS FIX (exposed by block-8's spare op-amp half): dual op-amps
were placed as a single instance while pins from BOTH halves were connected at the
lib_symbol's overlapping origin -> unit-A and unit-B pins landed on the same canvas
point, shorting the two halves. This was latent in EVERY dual-op-amp block (A,B,1,2,
4,5). Fix:
- place each gate unit (A/B/power) as its own instance at distinct offsets
  (MULTI_UNIT + opamp_unit_pins);
- make structural_check unit-aware (per-sub-symbol unit pins);
- add a short detector: 2+ distinct nets whose labels coincide at one point now fail.
All blocks regenerated and re-verified clean (the detector finds no shorts).

STATUS+plan: 7/10 blocks. All gates green.
Parts:
- added C42, C43, C44: 100nF, symbol Device:C
- added J26: VCA_IN, POGO_Connector_Audio:Jack_3.5mm_QingPu_WQP-PJ398SM_Vertical_CircularHoles, symbol Device:Audio_Jack_3.5mm_SwitchT
- C41: renamed from J26; value VCA_IN -> 100nF; footprint POGO_Connector_Audio:Jack_3.5mm_QingPu_WQP-PJ398SM_Vertical_CircularHoles -> (none); symbol Device:Audio_Jack_3.5mm_SwitchT -> Device:C
- D3: renamed from RV25; value VCA_OFS -> BAT54S; footprint POGO_Potentiometer_THT:Potentiometer_Alpha_RD901F-40-00D_Single_Vertical_CircularHoles -> POGO_Package_TO_SOT_SMD:SOT-23; symbol Device:R_POT -> Diode:BAT54S
- R40: renamed from R44; value 100k -> 20k
- R41: renamed from R45; value 100k -> 20k
- R42: renamed from R46; value 2k4 -> 10k
- R43: renamed from R9; value 100R -> 10k
- R44: renamed from D3; value BAT54S -> 100k; footprint POGO_Package_TO_SOT_SMD:SOT-23 -> (none); symbol Diode:BAT54S -> Device:R
- R45: renamed from RV1; value VCA_UNITY_L -> 100k; footprint POGO_Potentiometer_SMD:Potentiometer_Bourns_3224W -> (none); symbol Device:R_POT -> Device:R
- R46: renamed from RV2; value VCA_UNITY_R -> 2k4; footprint POGO_Potentiometer_SMD:Potentiometer_Bourns_3224W -> (none); symbol Device:R_POT -> Device:R
- R7: renamed from R42; value 10k -> 20k
- R8: renamed from R43; value 10k -> 20k
- R9: renamed from RV24; value VCA_AMT -> 100R; footprint POGO_Potentiometer_THT:Potentiometer_Alpha_RD901F-40-00D_Single_Vertical_CircularHoles -> (none); symbol Device:R_POT -> Device:R
- RV1: renamed from C7; value 100nF -> VCA_UNITY_L; footprint (none) -> POGO_Potentiometer_SMD:Potentiometer_Bourns_3224W; symbol Device:C -> Device:R_POT
- RV2: renamed from C8; value 100nF -> VCA_UNITY_R; footprint (none) -> POGO_Potentiometer_SMD:Potentiometer_Bourns_3224W; symbol Device:C -> Device:R_POT
- RV24: renamed from C9; value 100nF -> VCA_AMT; footprint (none) -> POGO_Potentiometer_THT:Potentiometer_Alpha_RD901F-40-00D_Single_Vertical_CircularHoles; symbol Device:C -> Device:R_POT
- RV25: renamed from C10; value 100nF -> VCA_OFS; footprint (none) -> POGO_Potentiometer_THT:Potentiometer_Alpha_RD901F-40-00D_Single_Vertical_CircularHoles; symbol Device:C -> Device:R_POT
- U6: renamed from R7; value 20k -> TL072; symbol Device:R -> Amplifier_Operational:OPA1612
- U6: renamed from U63; footprint POGO_Package_SO:SOIC-8_3.9x4.9mm_P1.27mm -> (none)
- U63: renamed from R40; value 20k -> TL072; symbol Device:R -> Amplifier_Operational:OPA1612
- U63: renamed from R41; value 20k -> TL072; symbol Device:R -> Amplifier_Operational:OPA1612
- U63: renamed from R8; value 20k -> TL072; footprint (none) -> POGO_Package_SO:SOIC-8_3.9x4.9mm_P1.27mm; symbol Device:R -> Amplifier_Operational:OPA1612
- renumbered C44 to C10, C41 to C7, C42 to C8, C43 to C9
Connections:
- net +12V: now also C41.2, D3.3 (K2), RV25.1, U6.4 (V-), U63.4 (V-), C43.2; no longer D3.1, R44.3 (K2), RV1.2, RV24.2
- net -12V: now also D3.1 (A1), U6.8 (V+), U63.8 (V+), C42.2, C44.2; no longer R44.1 (A1), RV2.2, RV25.2
- net AMT_W: now also R44.2, RV24.2 (Wiper); no longer R40.2, R9.2 (Wiper)
- net CVP: now also R42.2, RV24.1; no longer R43.1, R7.2
- net EC_L: now also RV1.2 (Wiper), RV1.3; no longer R45.2 (Wiper), R45.3
- net EC_R: now also RV2.2 (Wiper), RV2.3; no longer R46.2 (Wiper), R46.3
- net GND: now also C41.1 (+), RV25.3, U6.6 (In-), U63.2 (In-), U63.6 (In-), C42.1 (+), C43.1 (+), C44.1 (+), J26.2 (S); no longer C41.2 (S), D3.3, RV1.1 (+), RV2.1 (+), RV24.1 (+), RV25.1 (+), U6.2 (In-)
- net IV_L_IN: now also R40.2; no longer U63.2, U63.2
- net NCVP: now also R43.1, RV24.3, U63.1 (Out); no longer R42.1, R45.1, R46.1, R8.1, R9.3, U6.1 (Out)
- net OFS_W: now also R45.2, RV25.2 (Wiper); no longer D3.2 (Wiper), R41.2
- net PG_OUT_L: now also R7.2; no longer U6.2
- net PG_OUT_R: now also R8.2; no longer U63.2
- net U63A_INV: now also R42.1, R43.2, U63.3 (In+); no longer R40.1, R41.1, R42.2, R7.1, R8.2, U6.3 (In+)
- net VCA_CV_TIP: now also R9.2, J26.1 (T); no longer C41.1 (T), R43.2
- net VCA_IN_L: now also R7.1; no longer U6.1
- net VCA_IN_R: now also R8.1; no longer U63.1
- net VCA_OUT_L: now also R40.1; no longer U63.1, U63.1
- new net IV_R_IN: R41.2, U6.5 (In+)
- new net U63B_SUM: R44.1, R45.1, R46.2, U63.5 (In+)
- new net VCA_OUT_R: R41.1, U6.7 (Out)
- new net V_CTRL: R46.1, RV1.1, RV2.1, U63.7 (Out)
Other:
- moved on the sheet: C10, C7, C8, C9, R40, R41, R42, R43, R7, R8, U5, U63C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
