File: kicad/pogo-block-8.kicad_sch (KiCad schematic)
At the start: 65 parts, among them U11 OPA1612, U12 OPA1612, U13 TL072, U14 THAT340, U64 THAT340, U7 LM13700, U8 LM13700

Commit message: kicad: block-8 LP2 + fix multi-unit op-amp placement bug (7 of 10)
block-8 (LP2): OTA-C SVF mirroring LP1 minus tilt (single shared expo); Q VCA via
the shared-q sheet cell B (U9/U10); added LP2's own IRES_AMP (U65, was missing from
the BOM) + full SVF expansion (R_LIN, expo network, Q V->I, buffer pulldowns,
decoupling). 51 parts / 36 nets; LP2 boundary nets match shared-q byte-for-byte.
shared-q gains the LP2 cell-B Iabc bypass caps (C84/C85).

GENERATOR CORRECTNESS FIX (exposed by block-8's spare op-amp half): dual op-amps
were placed as a single instance while pins from BOTH halves were connected at the
lib_symbol's overlapping origin -> unit-A and unit-B pins landed on the same canvas
point, shorting the two halves. This was latent in EVERY dual-op-amp block (A,B,1,2,
4,5). Fix:
- place each gate unit (A/B/power) as its own instance at distinct offsets
  (MULTI_UNIT + opamp_unit_pins);
- make structural_check unit-aware (per-sub-symbol unit pins);
- add a short detector: 2+ distinct nets whose labels coincide at one point now fail.
All blocks regenerated and re-verified clean (the detector finds no shorts).

STATUS+plan: 7/10 blocks. All gates green.
Parts:
- removed C50, C51, C52, C53, C58, C59, C60, C61, C62, C63, C64, C65, C67, C68: 100nF, symbol Device:C
- C33A: renamed from U64; value THAT340 -> 47nF; footprint POGO_Package_SO:SOIC-14_3.9x8.7mm_P1.27mm -> (none); symbol POGO:THAT340 -> Device:C
- C69: renamed from R64; value 1k -> 100nF; symbol Device:R -> Device:C
- C70: renamed from R65; value 1M -> 10nF; symbol Device:R -> Device:C
- C71: renamed from R66; value 47k -> 10nF; symbol Device:R -> Device:C
- C72: renamed from R67; value 1k -> 100nF; symbol Device:R -> Device:C
- C73: renamed from RV3; value LP1_FREF_L -> 100nF; footprint POGO_Potentiometer_SMD:Potentiometer_Bourns_3224W -> (none); symbol Device:R_POT -> Device:C
- C74: renamed from RV4; value LP1_1VOCT_L -> 100nF; footprint POGO_Potentiometer_SMD:Potentiometer_Bourns_3224W -> (none); symbol Device:R_POT -> Device:C
- C75: renamed from RV22; value LP1_FREF_R -> 100nF; footprint POGO_Potentiometer_SMD:Potentiometer_Bourns_3224W -> (none); symbol Device:R_POT -> Device:C
- C76: renamed from RV23; value LP1_1VOCT_R -> 100nF; footprint POGO_Potentiometer_SMD:Potentiometer_Bourns_3224W -> (none); symbol Device:R_POT -> Device:C
- C77: renamed from RV5; value LP1_QMAX -> 100nF; footprint POGO_Potentiometer_SMD:Potentiometer_Bourns_3224W -> (none); symbol Device:R_POT -> Device:C
- C78: renamed from RV6; value LP1_TILTNULL -> 100nF; footprint POGO_Potentiometer_SMD:Potentiometer_Bourns_3224W -> (none); symbol Device:R_POT -> Device:C
- C79: renamed from D10; value 1N4148W -> 100nF; footprint POGO_Diode_SMD:D_SOD-123 -> (none); symbol Device:D -> Device:C
- C82: renamed from C46; value 10nF -> 100nF
- C83: renamed from C47; value 10nF -> 100nF
- D11: renamed from R63; value 47k -> 1N4148W; footprint (none) -> POGO_Diode_SMD:D_SOD-123; symbol Device:R -> Device:D
- R32: renamed from C14; value 47nF -> 100k; symbol Device:C -> Device:R
- R76: renamed from R54; value 100k -> 1k
- R80: renamed from R71; value 10k -> 1M
- R81: renamed from R55; value 100k -> 1M
- R86: renamed from R58; value 1M -> 47k
- R87: renamed from R59; value 100k -> 1k
- R88: renamed from R52; value 1k -> 10k
- RV19: renamed from R60; value 100k -> LP2_FREF; footprint (none) -> POGO_Potentiometer_SMD:Potentiometer_Bourns_3224W; symbol Device:R -> Device:R_POT
- RV20: renamed from R61; value 100k -> LP2_1VOCT; footprint (none) -> POGO_Potentiometer_SMD:Potentiometer_Bourns_3224W; symbol Device:R -> Device:R_POT
- RV21: renamed from R62; value 1M -> LP2_QMAX; footprint (none) -> POGO_Potentiometer_SMD:Potentiometer_Bourns_3224W; symbol Device:R -> Device:R_POT
- renumbered C11 to C33B, C12 to C33C, C13 to C33D, C45 to C80, C66 to C81, R10 to R33, R11 to R72, R47 to R73, R48 to R74, R53 to R75, R49 to R77, R50 to R78, R51 to R79, R56 to R82, R_TILT_INV_IN to R83, R_TILT_INV_FB to R84, R57 to R85, R68 to R89, R69 to R90, R70 to R91, U7 to U56, U8 to U57, U11 to U58, U12 to U59, U14 to U60, U13 to U65
Connections:
- net LP1_RES is gone; now on net LP2_IREF_TR: RV19.2 (Wiper)
- net VCA_OUT_R is gone; now on net LP2_LP_L: R72.2
- net +12V: now also C72.2, C74.2, C76.2, C78.2, C80.2, C82.2, R85.2, RV21.1; no longer C70.2, C77.1, C78.1, RV21.2
- net -12V: now also C73.2, C75.2, C77.2, C79.2, C81.2, C83.2, R87.1, R88.1; no longer C33A.11 (SUB), C33A.4 (SUB), C69.1, C72.1, C78.3, R80.1
- net GND: now also C33A.1 (+), C69.1 (+), C70.1 (+), C71.1 (+), C72.1 (+), C73.1 (+), C74.1 (+), C75.1 (+), C76.1 (+), C77.1 (+), C78.1 (+), C79.1 (+), D11.K, R76.1, RV21.3; no longer C77.3, C79.K, R32.1 (+), R88.1, U65.6 (In-)
- net LP2_V1CAP_L: now reaches C33A.2
- net LP2_V1CAP_L: now also U56.2 (DiodeBias_A), U56.4 (In-_A)
- removed net LP1_EXPO_BASE_L: C74.1, R81.1, U60.6 (Q3_B)
- removed net LP1_EXPO_BASE_R: C33A.6 (Q3_B), C76.1, C78.2 (Wiper), R82.1
- net LP1_EXPO_EMIT_L renamed LP2_EXPO_EMIT
- net LP2_EXPO_EMIT: now also R87.2; no longer C69.2
- removed net LP1_EXPO_EMIT_R: C33A.10 (Q4_E), C33A.5 (Q3_E), C72.2
- net LP1_HP_L renamed LP2_HP_L
- net LP2_HP_L: now also R74.1; no longer R75.1
- net LP1_HP_R renamed LP2_HP_R
- net LP2_HP_R: now also R75.1; no longer R76.1
- net LP1_IABC_L renamed LP2_IABC
- net LP2_IABC: now also C70.2, C71.2, U57.8 (BufOut_A), U57.9 (BufOut_B); no longer C82.2
- removed net LP1_IABC_R: C33A.7 (Q3_C), C83.2, U57.8 (BufOut_A), U57.9 (BufOut_B)
- net LP1_IREF_L renamed LP2_IREF
- net LP2_IREF: now also C69.2, RV19.1; no longer C73.1, C80.2
- removed net LP1_IREF_R: C33A.8 (Q4_C), C33A.9 (Q4_B), C75.1, C81.2
- removed net LP1_IREF_TR_L: C73.2 (Wiper), C73.3, RV21.1
- removed net LP1_IREF_TR_R: C70.1, C75.2 (Wiper), C75.3
- removed net LP1_IRES_SUM: R87.1, RV19.1, RV20.2, U65.5 (In+)
- net LP1_LIN_A_L renamed LP2_LIN_A_L
- net LP2_LIN_A_L: now also R76.2; no longer R77.2
- net LP1_LIN_A_R renamed LP2_LIN_A_R
- net LP2_LIN_A_R: now also R78.2; no longer R79.2
- net LP1_LIN_B_L renamed LP2_LIN_B_L
- net LP2_LIN_B_L: now also R77.2; no longer R78.2
- net LP1_LIN_B_R renamed LP2_LIN_B_R
- net LP2_LIN_B_R: now also R79.2; no longer R88.2
- net LP1_LP_L renamed LP2_LP_L
- net LP2_LP_L: now also R89.2; no longer R73.2, R90.2
- net LP1_LP_R renamed LP2_LP_R
- net LP2_LP_R: now also R73.2, R91.2; no longer R74.2, R80.2
- net LP1_NTILT renamed LP2_VIRES
- net LP2_VIRES: now also D11.A, R80.2, R81.2; no longer R82.2
- net LP1_OUT_L renamed LP2_OUT_L
- net LP1_OUT_R renamed LP2_OUT_R
- net LP1_QIABC_L renamed LP2_IREF_TR
- net LP2_IREF_TR: now also RV19.3
- net LP1_QIABC_R renamed LP2_VOCT_TR
- net LP2_VOCT_TR: now also RV20.2 (Wiper), RV20.3
- net LP1_SUMINV_L renamed LP2_SUMINV_R
- net LP2_SUMINV_R: now also U59.3 (In+); no longer U58.3 (In+)
- removed net LP1_SUMINV_R: R72.1, R74.1, R76.2, U59.3 (In+)
- net LP1_TILT renamed LP2_RES
- net LP2_RES: no longer R81.2
- net LP1_TILT_INVN renamed LP2_IRES_SUM
- net LP2_IRES_SUM: now also R82.1
- removed net LP1_V1CAP_L: C33B.2, U56.2 (DiodeBias_A), U56.4 (In-_A)
- net LP1_V1CAP_R renamed LP2_V1CAP_R
- net LP2_V1CAP_R: now also C33C.2; no longer C33D.2
- net LP1_V1_L renamed LP2_V1_L
- net LP2_V1_L: now also R88.2; no longer R89.2
- net LP1_V1_R renamed LP2_V1_R
- net LP2_V1_R: now also R90.2; no longer R91.2
- net LP1_V2CAP_L renamed LP2_V2CAP_L
- net LP2_V2CAP_L: now also C33B.2; no longer C33C.2
- net LP1_V2CAP_R renamed LP2_V2CAP_R
- net LP2_V2CAP_R: now also C33D.2; no longer R32.2
- removed net LP1_VBIAS: C77.2 (Wiper), R87.2
- removed net LP1_VCTRL: C71.2, D11.2
- removed net LP1_VIRES: C79.A, R85.2, R86.2, RV20.1, U65.7 (Out)
- removed net LP1_VOCT_TR_L: C74.2 (Wiper), C74.3, D11.1
- removed net LP1_VOCT_TR_R: C71.1, C76.2 (Wiper), C76.3
- net VCA_OUT_L renamed HP_OUT_R
- new net HP_OUT_L: R32.2
- new net LP2_EXPO_BASE: RV20.1, U60.6 (Q3_B)
- new net LP2_QIABC_L: R80.1
- new net LP2_QIABC_R: R81.1
- new net LP2_SUMINV_L: R32.1, R72.1, R74.2, U58.3 (In+)
- new net LP2_VBIAS: R82.2, RV21.2 (Wiper)
- new net LP2_VCTRL: R86.2
