File: kicad/pogo-block-8.kicad_sch (KiCad schematic)
At the start: 51 parts, among them U56 LM13700, U57 LM13700, U58 OPA1612, U59 OPA1612, U60 THAT340, U65 TL072

Commit message: 0020 §A: expo V/oct divider fix - block-8 LP2 (mono, same template as block-7)
R86 R_VOCT 47k->49.9k + R230 Vishay TFPT 1k tempco shunt on LP2_EXPO_BASE->GND.
Resolves in BOM to TFPT0805L1001FM + footprint + datasheet. block-8 schematic
regenerated (52 parts/36 nets); all --check gates green.

https://claude.ai/code/session_013jFXG5oeMVSYP7iRpwGvtQ
Parts:
- added C83: 100nF, symbol Device:C
- C69: renamed from C70; value 10nF -> 100nF
- C71: renamed from C72; value 100nF -> 10nF
- D11: renamed from C69; value 100nF -> 1N4148W; footprint (none) -> POGO_Diode_SMD:D_SOD-123; symbol Device:C -> Device:D
- R230: renamed from RV19; value LP2_FREF -> 1k; footprint POGO_Potentiometer_SMD:Potentiometer_Bourns_3224W -> POGO_Resistor_SMD:R_0805_2012Metric; symbol Device:R_POT -> Device:R
- R86: value 47k -> 49k9
- RV19: renamed from RV20; value LP2_1VOCT -> LP2_FREF
- RV20: renamed from RV21; value LP2_QMAX -> LP2_1VOCT
- RV21: renamed from D11; value 1N4148W -> LP2_QMAX; footprint POGO_Diode_SMD:D_SOD-123 -> POGO_Potentiometer_SMD:Potentiometer_Bourns_3224W; symbol Device:D -> Device:R_POT
- renumbered C71 to C70, C73 to C72, C74 to C73, C75 to C74, C76 to C75, C77 to C76, C78 to C77, C79 to C78, C80 to C79, C81 to C80, C82 to C81, C83 to C82
Connections:
- net +12V: now also C72.2, C74.2, C76.2, C78.2, C80.2, C82.2, RV21.1; no longer C71.2, C73.2, C75.2, C77.2, C79.2, C81.2, RV20.1
- net -12V: now also C73.2, C75.2, C77.2, C79.2, C81.2, C83.2; no longer C72.2, C74.2, C76.2, C78.2, C80.2, C82.2
- net GND: now also D11.K, R230.1, RV21.3, C83.1; no longer D11.1, RV20.3, RV21.K
- net LP2_EXPO_BASE: now also R230.2, RV20.1; no longer RV19.1
- net LP2_IABC: now also C71.2; no longer C69.2
- net LP2_IREF: now also C69.2, RV19.1; no longer D11.2, R230.1
- net LP2_IREF_TR: now also RV19.2 (Wiper), RV19.3; no longer R230.2 (Wiper), R230.3
- net LP2_VBIAS: now also RV21.2 (Wiper); no longer RV20.2 (Wiper)
- net LP2_VIRES: now also D11.A; no longer RV21.A
- net LP2_VOCT_TR: now also RV20.2 (Wiper), RV20.3; no longer RV19.2 (Wiper), RV19.3

Commit message: 0020 §C+§D: block-8 LP2 OTA tap + Q-cell R_Iabc (same pattern as block-7)
§C (H5): tap v1/v2 from unbuffered OTA outputs (pins 5/12); v2 now drives the LP
output buffer + R_FB from the clean cap node (no Darlington offset in the loop).
Removed R88-R91 pulldowns; buffer pins 7/8/9/10 -> no_connect. LP2_V1_* boundary
to block-5 Q-VCAs preserved.
§D/M5: R80/R81 R_Iabc 1M->100k. (Negative-V_ires IRES_AMP redesign deferred to
the block-5 combined pass, [NV]/trim-backed.)

block-8 schematic regenerated (48 parts/32 nets); all --check gates green, 0 FAIL.

https://claude.ai/code/session_013jFXG5oeMVSYP7iRpwGvtQ
Parts:
- removed C80, C81, C82, C83: 100nF, symbol Device:C
- C69: renamed from RV19; value LP2_FREF -> 100nF; footprint POGO_Potentiometer_SMD:Potentiometer_Bourns_3224W -> (none); symbol Device:R_POT -> Device:C
- C70: renamed from RV20; value LP2_1VOCT -> 10nF; footprint POGO_Potentiometer_SMD:Potentiometer_Bourns_3224W -> (none); symbol Device:R_POT -> Device:C
- C71: renamed from RV21; value LP2_QMAX -> 10nF; footprint POGO_Potentiometer_SMD:Potentiometer_Bourns_3224W -> (none); symbol Device:R_POT -> Device:C
- C72: renamed from D11; value 1N4148W -> 100nF; footprint POGO_Diode_SMD:D_SOD-123 -> (none); symbol Device:D -> Device:C
- C74: renamed from C70; value 10nF -> 100nF
- C75: renamed from C71; value 10nF -> 100nF
- D11: renamed from R230; value 1k -> 1N4148W; footprint POGO_Resistor_SMD:R_0805_2012Metric -> POGO_Diode_SMD:D_SOD-123; symbol Device:R -> Device:D
- R230: renamed from R84; value 100k -> 1k; footprint (none) -> POGO_Resistor_SMD:R_0805_2012Metric
- R80: renamed from R88; value 10k -> 100k
- R81: renamed from R89; value 10k -> 100k
- R82: renamed from R90; value 10k -> 100k
- R83: renamed from R91; value 10k -> 100k
- R84: renamed from R80; value 1M -> 100k
- R86: renamed from R82; value 100k -> 49k9
- R87: renamed from R83; value 100k -> 1k
- RV19: renamed from R85; value 1M -> LP2_FREF; footprint (none) -> POGO_Potentiometer_SMD:Potentiometer_Bourns_3224W; symbol Device:R -> Device:R_POT
- RV20: renamed from R86; value 49k9 -> LP2_1VOCT; footprint (none) -> POGO_Potentiometer_SMD:Potentiometer_Bourns_3224W; symbol Device:R -> Device:R_POT
- RV21: renamed from R87; value 1k -> LP2_QMAX; footprint (none) -> POGO_Potentiometer_SMD:Potentiometer_Bourns_3224W; symbol Device:R -> Device:R_POT
- renumbered C69 to C73, C72 to C76, C73 to C77, C74 to C78, C75 to C79, C76 to C80, C77 to C81, C78 to C82, C79 to C83, R81 to R85
Connections:
- net +12V: now also C72.2, C74.2, R85.2, RV21.1; no longer C71.1, RV19.2
- net -12V: now also C73.2, C75.2, R87.1; no longer R80.1, R81.1, R82.1, R83.1, RV21.1
- net GND: now also C69.1, C70.1, C71.1, C72.1, D11.K, R230.1, RV21.3; no longer C71.3, C72.K, D11.1
- net LP2_EXPO_BASE: now also R230.2, RV20.1; no longer C70.1, D11.2
- net LP2_EXPO_EMIT: now also R87.2; no longer RV21.2
- net LP2_IABC: now also C70.2, C71.2; no longer C74.2, C75.2
- net LP2_IREF: now also C69.2, RV19.1; no longer C69.1, C73.2
- net LP2_IREF_TR: now also R85.1, RV19.2 (Wiper), RV19.3; no longer C69.2 (Wiper), C69.3, RV19.1
- net LP2_IRES_SUM: now also R82.1, R83.1, R84.2; no longer R230.2, R86.1, R87.1
- net LP2_QIABC_L: now also R80.1; no longer R84.1
- net LP2_QIABC_R: now also R81.1; no longer R85.1
- net LP2_RES: now also R83.2; no longer R87.2
- net LP2_V1_L: now also C33A.2, U56.4 (In-_A); no longer R80.2, U56.1 (Iabc_A)
- net LP2_V1_R: now also C33C.2, U57.4 (In-_A); no longer R82.2, U57.1 (Iabc_A)
- net LP2_VBIAS: now also R82.2, RV21.2 (Wiper); no longer C71.2 (Wiper), R86.2
- net LP2_VCTRL: now also R86.2; no longer RV20.2
- net LP2_VIRES: now also D11.A, R80.2, R81.2, R84.1; no longer C72.A, R230.1, R84.2, R85.2
- net LP2_VOCT_TR: now also R86.1, RV20.2 (Wiper), RV20.3; no longer C70.2 (Wiper), C70.3, RV20.1
- net LP2_LP_L renamed LP2_V2_L
- net LP2_V2_L: now also C33B.2, U56.13 (In-_B); no longer R81.2, U56.16 (Iabc_B)
- net LP2_LP_R renamed LP2_V2_R
- net LP2_V2_R: now also C33D.2, U57.13 (In-_B); no longer R83.2, U57.16 (Iabc_B)
- removed net LP2_V1CAP_L: C33A.2, U56.2 (DiodeBias_A), U56.4 (In-_A)
- removed net LP2_V1CAP_R: C33C.2, U57.2 (DiodeBias_A), U57.4 (In-_A)
- removed net LP2_V2CAP_L: C33B.2, U56.13 (In-_B), U56.15 (DiodeBias_B)
- removed net LP2_V2CAP_R: C33D.2, U57.13 (In-_B), U57.15 (DiodeBias_B)
