File: kicad/pogo-block-5.kicad_sch (KiCad schematic)
At the start: 65 parts, among them U11 OPA1612, U12 OPA1612, U13 TL072, U14 THAT340, U64 THAT340, U7 LM13700, U8 LM13700

Commit message: shared: replace block-Q with dual-ownership + shared flag (fold into block-5)
Per the chosen model: shared parts carry block: [block-5, block-8] + shared: true
in components.yaml (dual ownership, one refdes), and the U9/U10 Q-VCAs are folded
onto block-5's sheet (the host / first owner). Removes the synthetic block-Q, its
pseudo-spec (specs/block-Q/), and the separate pogo-shared-q.kicad_sch.

- components.yaml: 10 shared rows -> block: [block-5, block-8], shared: true.
- block-5.nets.yaml: U9/U10 + caps folded in; LP1 Q nets now internal; LP2_*
  become block-5->block-8 boundary nets. block-5 sch regenerates (75 parts/51 nets).
- build_components.gen_bom: render list-valued Block ('block-5, block-8').
- docs/bom.html: group-by-block puts a shared part under each of its blocks.
- Scrub: §4 'Shared resource' pointers (block-5 hosts / block-8 references),
  SCHEMATIC-GEN-PLAN decision reversed, CLAUDE/README/STATUS/build.yml, block-8
  netlist comments. Deleted .gitattributes shared-q line + CI artifact glob entry.

All 5 --check gates green; block-8 LP2_* boundary nets match block-5's producers.

https://claude.ai/code/session_01MsjDdC2SbAb3J3qGafGBjk
Parts:
- added C48, C49, C84, C85: 10nF, symbol Device:C
- added C54, C55, C56, C57: 100nF, symbol Device:C
- added U10, U9: LM13700, POGO_Package_SO:SOIC-16_3.9x9.9mm_P1.27mm, symbol Amplifier_Operational:LM13700
Connections:
- net +12V: now also C54.2, C56.2, U10.14 (In+_B), U9.14 (In+_B)
- net -12V: now also C55.2, C57.2, U10.3 (In+_A), U9.3 (In+_A)
- net GND: now also C48.1 (+), C49.1 (+), C54.1 (+), C55.1 (+), C56.1 (+), C57.1 (+), C84.1 (+), C85.1 (+)
- net LP1_QIABC_L: now also C48.2, U9.8 (BufOut_A)
- net LP1_QIABC_R: now also C49.2, U10.8 (BufOut_A)
- net LP1_SUMINV_L: now also U9.4 (In-_A), U9.5 (Out_A)
- net LP1_SUMINV_R: now also U10.4 (In-_A), U10.5 (Out_A)
- net LP1_V1_L: now also U9.6 (V-)
- net LP1_V1_R: now also U10.6 (V-)
- new net LP2_QIABC_L: C84.2, U9.9 (BufOut_B)
- new net LP2_QIABC_R: C85.2, U10.9 (BufOut_B)
- new net LP2_SUMINV_L: U9.12 (Out_B), U9.13 (In-_B)
- new net LP2_SUMINV_R: U10.12 (Out_B), U10.13 (In-_B)
- new net LP2_V1_L: U9.11 (V+)
- new net LP2_V1_R: U10.11 (V+)
