File: kicad/pogo-block-5.kicad_sch (KiCad schematic)
At the start: 75 parts, among them U10 LM13700, U11 OPA1612, U12 OPA1612, U13 TL072, U14 THAT340, U64 THAT340, U7 LM13700, U8 LM13700, U9 LM13700

Commit message: 0020 §A+§B+§C+§D: block-5 LP1 combined filter-core edit (stereo)
The convergence block, done as one coherent edit:
- §A expo divider: R63/R66 R_VOCT 47k->49.9k + R231/R232 Vishay TFPT 1k tempco
  shunts on both expo bases (L+R). Centers 17.92mV/oct at mid-trim.
- §B tilt: SPICE (lp1_tilt_passive.cir) showed tilt can sum PASSIVELY with V_freq
  at the tempco-shunted base via an equal series R -> R55/R56 100k->54.9k
  (=R_VOCT+RV_mid, 1:1 octave weight, freq=tilt=17.57mV/V). NO extra op-amp needed
  (dropped the planned +1 TL072). U13-A still makes -V_tilt for R; RV6 null kept.
- §C OTA tap: v1/v2 from unbuffered OTA pins 5/12 (not Darlington 8/9); removed
  R68-R71 pulldowns; buffer pins 7-10 -> no_connect. LP1_V1/V2 + Q-cell boundary
  preserved.
- §D/M5: R57/R58 R_Iabc 1M->100k.

block-5 schematic regenerated (73 parts/47 nets); all --check gates + JS/Py
parity green, 0 FAIL. (Negative-V_ires IRES_AMP bias redesign still [NV]/trim,
shared across 5/7/8 - tracked.)

https://claude.ai/code/session_013jFXG5oeMVSYP7iRpwGvtQ
Parts:
- removed C84, C85: 10nF, symbol Device:C
- C45: renamed from RV6; value LP1_TILTNULL -> 100nF; footprint POGO_Potentiometer_SMD:Potentiometer_Bourns_3224W -> (none); symbol Device:R_POT -> Device:C
- C46: renamed from C45; value 100nF -> 10nF
- C47: renamed from C66; value 100nF -> 10nF
- C48: renamed from U9; value LM13700 -> 10nF; footprint POGO_Package_SO:SOIC-16_3.9x9.9mm_P1.27mm -> (none); symbol Amplifier_Operational:LM13700 -> Device:C
- C49: renamed from U10; value LM13700 -> 10nF; footprint POGO_Package_SO:SOIC-16_3.9x9.9mm_P1.27mm -> (none); symbol Amplifier_Operational:LM13700 -> Device:C
- C50: renamed from C46; value 10nF -> 100nF
- C51: renamed from C47; value 10nF -> 100nF
- C54: renamed from C48; value 10nF -> 100nF
- C55: renamed from C49; value 10nF -> 100nF
- C66: renamed from D10; value 1N4148W -> 100nF; footprint POGO_Diode_SMD:D_SOD-123 -> (none); symbol Device:D -> Device:C
- C84: renamed from C56; value 100nF -> 10nF
- C85: renamed from C57; value 100nF -> 10nF
- D10: renamed from RV5; value LP1_QMAX -> 1N4148W; footprint POGO_Potentiometer_SMD:Potentiometer_Bourns_3224W -> POGO_Diode_SMD:D_SOD-123; symbol Device:R_POT -> Device:D
- R231: renamed from R64; footprint (none) -> POGO_Resistor_SMD:R_0805_2012Metric
- R232: renamed from R65; value 1M -> 1k; footprint (none) -> POGO_Resistor_SMD:R_0805_2012Metric
- R55: renamed from R68; value 10k -> 54k9
- R56: renamed from R69; value 10k -> 54k9
- R61: renamed from R57; value 1M -> 100k
- R63: renamed from R59; value 100k -> 49k9
- R64: renamed from R60; value 100k -> 1k
- R65: renamed from R61; value 100k -> 1M
- R66: renamed from R62; value 1M -> 49k9
- R67: renamed from R63; value 47k -> 1k
- RV22: renamed from RV3; value LP1_FREF_L -> LP1_FREF_R
- RV23: renamed from RV4; value LP1_1VOCT_L -> LP1_1VOCT_R
- RV3: renamed from R66; value 47k -> LP1_FREF_L; footprint (none) -> POGO_Potentiometer_SMD:Potentiometer_Bourns_3224W; symbol Device:R -> Device:R_POT
- RV4: renamed from R67; value 1k -> LP1_1VOCT_L; footprint (none) -> POGO_Potentiometer_SMD:Potentiometer_Bourns_3224W; symbol Device:R -> Device:R_POT
- RV5: renamed from RV22; value LP1_FREF_R -> LP1_QMAX
- RV6: renamed from RV23; value LP1_1VOCT_R -> LP1_TILTNULL
- R_TILT_INV_FB: renamed from R71; value 10k -> 100k
- R_TILT_INV_IN: renamed from R70; value 10k -> 100k
- U10: renamed from C68; value 100nF -> LM13700; footprint (none) -> POGO_Package_SO:SOIC-16_3.9x9.9mm_P1.27mm; symbol Device:C -> Amplifier_Operational:LM13700
- U9: renamed from C67; value 100nF -> LM13700; footprint (none) -> POGO_Package_SO:SOIC-16_3.9x9.9mm_P1.27mm; symbol Device:C -> Amplifier_Operational:LM13700
- renumbered C50 to C52, C51 to C53, C54 to C56, C55 to C57, C52 to C58, C53 to C59, C58 to C60, C59 to C61, C60 to C62, C61 to C63, C62 to C64, C63 to C65, C64 to C67, C65 to C68, R55 to R57, R56 to R58, R_TILT_INV_IN to R59, R_TILT_INV_FB to R60, R58 to R62
Connections:
- net +12V: now also C50.2, C54.2, R62.2, R65.2, RV5.1, RV6.1, U10.14 (In+_B), U9.14 (In+_B); no longer C45.1, C48.14 (In+_B), C49.14 (In+_B), C84.2, D10.1, R232.2, R66.2, U9.2
- net -12V: now also C51.2, C55.2, R64.1, R67.1, RV6.3, U10.3 (In+_A), U9.3 (In+_A); no longer C45.3, C48.3 (In+_A), C49.3 (In+_A), C85.2, R231.1, R55.1, R56.1, RV4.1, R_TILT_INV_FB.1, R_TILT_INV_IN.1, U10.2
- net GND: now also C45.1, C48.1, C49.1, C66.1, D10.K, R231.1, R232.1, RV5.3; no longer C66.K, D10.3, U10.1, U9.1
- net LP1_EXPO_BASE_L: now also R231.2, R55.1, RV4.1; no longer R57.1, RV23.1
- net LP1_EXPO_BASE_R: now also R232.2, R56.1, RV23.1, RV6.2 (Wiper); no longer C45.2 (Wiper), R58.1, RV6.1
- net LP1_EXPO_EMIT_L: now also R64.2; no longer R231.2
- net LP1_EXPO_EMIT_R: now also R67.2; no longer RV4.2
- net LP1_IABC_L: now also C46.2; no longer C50.2
- net LP1_IABC_R: now also C47.2; no longer C51.2
- net LP1_IREF_L: now also C45.2, RV3.1; no longer C46.2, RV22.1
- net LP1_IREF_R: now also C66.2, RV22.1; no longer C47.2, RV5.1
- net LP1_IREF_TR_L: now also R62.1, RV3.2 (Wiper), RV3.3; no longer R66.1, RV22.2 (Wiper), RV22.3
- net LP1_IREF_TR_R: now also R65.1, RV22.2 (Wiper), RV22.3; no longer R232.1, RV5.2 (Wiper), RV5.3
- net LP1_IRES_SUM: now also R59.1, R60.1, R61.2; no longer R63.1, R64.1, R65.2
- net LP1_NTILT: now also R56.2, R_TILT_INV_FB.1; no longer R58.2, R60.1
- net LP1_QIABC_L: now also C48.2, R57.1, U9.8 (BufOut_A); no longer C48.8 (BufOut_A), C54.2, R61.1
- net LP1_QIABC_R: now also C49.2, R58.1, U10.8 (BufOut_A); no longer C49.8 (BufOut_A), C55.2, R62.1
- net LP1_RES: now also R60.2; no longer R64.2
- net LP1_SUMINV_L: now also U9.4 (In-_A), U9.5 (Out_A); no longer C48.4 (In-_A), C48.5 (Out_A)
- net LP1_SUMINV_R: now also U10.4 (In-_A), U10.5 (Out_A); no longer C49.4 (In-_A), C49.5 (Out_A)
- net LP1_TILT: now also R55.2, R_TILT_INV_IN.2; no longer R57.2, R59.2
- net LP1_TILT_INVN: now also R_TILT_INV_FB.2, R_TILT_INV_IN.1; no longer R59.1, R60.2
- net LP1_V1_L: now also C11.2, U7.4 (In-_A), U9.6 (V-); no longer C48.6 (V-), R55.2, U7.1 (Iabc_A)
- net LP1_V1_R: now also C13.2, U10.6 (V-), U8.4 (In-_A); no longer C49.6 (V-), R_TILT_INV_IN.2, U8.1 (Iabc_A)
- net LP1_VBIAS: now also R59.2, RV5.2 (Wiper); no longer D10.2 (Wiper), R63.2
- net LP1_VCTRL: now also R63.2, R66.2; no longer R67.2, RV3.2
- net LP1_VIRES: now also D10.A, R57.2, R58.2, R61.1; no longer C66.A, R61.2, R62.2, R65.1
- net LP1_VOCT_TR_L: now also R63.1, RV4.2 (Wiper), RV4.3; no longer R67.1, RV23.2 (Wiper), RV23.3
- net LP1_VOCT_TR_R: now also R66.1, RV23.2 (Wiper), RV23.3; no longer RV3.1, RV6.2 (Wiper), RV6.3
- net LP2_QIABC_L: now also C84.2, U9.9 (BufOut_B); no longer C48.9 (BufOut_B)
- net LP2_QIABC_R: now also C85.2, U10.9 (BufOut_B); no longer C49.9 (BufOut_B)
- net LP2_SUMINV_L: now also U9.12 (Out_B), U9.13 (In-_B); no longer C48.12 (Out_B), C48.13 (In-_B)
- net LP2_SUMINV_R: now also U10.12 (Out_B), U10.13 (In-_B); no longer C49.12 (Out_B), C49.13 (In-_B)
- net LP2_V1_L: now also U9.11 (V+); no longer C48.11 (V+)
- net LP2_V1_R: now also U10.11 (V+); no longer C49.11 (V+)
- net LP1_LP_L renamed LP1_V2_L
- net LP1_V2_L: now also C12.2, U7.13 (In-_B); no longer R56.2, U7.16 (Iabc_B)
- net LP1_LP_R renamed LP1_V2_R
- net LP1_V2_R: now also C14.2, U8.13 (In-_B); no longer R_TILT_INV_FB.2, U8.16 (Iabc_B)
- removed net LP1_V1CAP_L: C11.2, U7.2 (DiodeBias_A), U7.4 (In-_A)
- removed net LP1_V1CAP_R: C13.2, U8.2 (DiodeBias_A), U8.4 (In-_A)
- removed net LP1_V2CAP_L: C12.2, U7.13 (In-_B), U7.15 (DiodeBias_B)
- removed net LP1_V2CAP_R: C14.2, U8.13 (In-_B), U8.15 (DiodeBias_B)
