File: kicad/pogo-block-6-svf1.kicad_sch (KiCad schematic)
At the start: 67 parts, among them U15 LM13700, U16 LM13700, U21 OPA1612, U22 OPA1612, U28 THAT340, U67 LM13700, U70 THAT340, U73 TL072

Commit message: 0018: block-6 stage 1 - F_REF 400Hz all bands + pole-count doc
Per user confirmation, the plugin's F_REF = {400,400,400} is correct (the
{200,1500,6000} formant spread was a stale code comment). Align the hardware:
- All 3 BP integrator caps (C15/C19/C23) -> 68nF C0G 0805 (was 150/22/4.7nF),
  trimmed to 400Hz by each band's f_ref trim. Bands now default to the same
  center and the player spreads them via the FREQ knobs.
- spec §2 f_ref table, expo-trim targets, and cap derivation updated to 400Hz;
  fixed the stale '3x THAT340 shared L/R' -> 6x per-channel.
- Resolved the long-standing BP '4-pole vs 2-pole' question: the plugin BP is a
  single 2-pole SVFGroup (returns v1), so hardware 2-pole MATCHES. Corrected
  the wrong '4-pole DSP cascade' claim in aux-ota-c-svf.

All five --check gates + parity green.

https://claude.ai/code/session_013jFXG5oeMVSYP7iRpwGvtQ
Parts:
- C15_Lv1, C15_Lv2, C15_Rv1, C15_Rv2: value 150nF -> 68nF
Changed lines of the file:
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@@
   (property "Reference" "C15_Lv1" (at 103.000 593.000 0)
     (effects (font (size 1.27 1.27)) (justify left)))
-  (property "Value" "150nF" (at 103.000 589.500 0)
+  (property "Value" "68nF" (at 103.000 589.500 0)
     (effects (font (size 1.016 1.016)) (justify left) (hide yes)))
 )
@@
   (property "Reference" "C15_Lv2" (at 163.000 593.000 0)
     (effects (font (size 1.27 1.27)) (justify left)))
-  (property "Value" "150nF" (at 163.000 589.500 0)
+  (property "Value" "68nF" (at 163.000 589.500 0)
     (effects (font (size 1.016 1.016)) (justify left) (hide yes)))
 )
@@
   (property "Reference" "C15_Rv1" (at 103.000 813.000 0)
     (effects (font (size 1.27 1.27)) (justify left)))
-  (property "Value" "150nF" (at 103.000 809.500 0)
+  (property "Value" "68nF" (at 103.000 809.500 0)
     (effects (font (size 1.016 1.016)) (justify left) (hide yes)))
 )
@@
   (property "Reference" "C15_Rv2" (at 163.000 813.000 0)
     (effects (font (size 1.27 1.27)) (justify left)))
-  (property "Value" "150nF" (at 163.000 809.500 0)
+  (property "Value" "68nF" (at 163.000 809.500 0)
     (effects (font (size 1.016 1.016)) (justify left) (hide yes)))
 )

Commit message: 0018: block-6 stage 2 - distortion BEFORE bandpass (0017 reorder)
The core 0017 change: flip the per-band order from SVF->DIST to DIST->SVF to
match the plugin (Pogo.cpp:443-451). Realized as a net re-point across the 7
split sections (no part changes):
  LP1_OUT / BP3IN  ->  distN (R18/R20/R22 distortion inputs)
                   ->  mux out (BPn_DISTOUT)  ->  svfN SUM_AMP (R13)
                   ->  SVF v1 buffer (BPn_BANDOUT / BP3_TAP)  ->  mix wet summer
- BP1/BP2 take the LP1 band; BP3 takes BP3IN (the ALT/LP1 selector, stage 3).
- BP3 OUT tap now taken post-bandpass (BP3_TAP = svf3 v1), matching the plugin
  (prevOut[2]); block-B keeps the BP3_TAP net name (no block-B change).
- spec §1/§2 updated: signal order, DIST knob, ALT path (through-VCA/BP3-only),
  BP3 tap point.

Boundary symmetry verified for all re-pointed nets; all 5 --check gates +
parity green.

https://claude.ai/code/session_013jFXG5oeMVSYP7iRpwGvtQ
Connections:
- net BP1_BPBUF_L renamed BP1_BANDOUT_L
- net BP1_BPBUF_R renamed BP1_BANDOUT_R
- net LP1_OUT_L renamed BP1_DISTOUT_L
- net LP1_OUT_R renamed BP1_DISTOUT_R
Changed lines of the file:
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@@
   (effects (font (size 1.016 1.016)) (justify left))
 )
-(global_label "LP1_OUT_L"
+(global_label "BP1_DISTOUT_L"
   (shape output)
   (at 40.000 483.810 0)
   (effects (font (size 1.016 1.016)) (justify left))
 )
-(global_label "LP1_OUT_R"
+(global_label "BP1_DISTOUT_R"
   (shape output)
   (at 40.000 703.810 0)
@@
   (effects (font (size 1.016 1.016)) (justify left))
 )
-(global_label "BP1_BPBUF_L"
+(global_label "BP1_BANDOUT_L"
   (shape output)
   (at 47.620 172.000 0)
   (effects (font (size 1.016 1.016)) (justify left))
 )
-(global_label "BP1_BPBUF_L"
+(global_label "BP1_BANDOUT_L"
   (shape output)
   (at 32.380 174.540 0)
@@
   (effects (font (size 1.016 1.016)) (justify left))
 )
-(global_label "BP1_BPBUF_R"
+(global_label "BP1_BANDOUT_R"
   (shape output)
   (at 47.620 227.000 0)
   (effects (font (size 1.016 1.016)) (justify left))
 )
-(global_label "BP1_BPBUF_R"
+(global_label "BP1_BANDOUT_R"
   (shape output)
   (at 32.380 229.540 0)

Commit message: 0018: block-6 stage 4 - per-band BP TILT (summer+inverter/band)
The per-band tilt was entirely unbuilt (the panel BP1/2/3 TILT knobs had no
hardware control component at all, and only the master tilt was wired). Build
it to match the plugin's groupTiltV[i] = BPn_TILT_PARAM + CV*0.22:
- Per band (svf1/2/3): +1 TL072 (U82-84) as an inverting summer + inverter.
  Summer combines master tilt (BP_TILT_CV, 100k) + the per-band TILT knob
  (RV48-50 bipolar, 100k) + the per-band TILT CV (MOD_BPn_TILT from block-3,
  470k -> x0.213 ~= the plugin's x0.22). -total feeds the R expo base; the
  inverter's +total feeds the L expo base.
- Re-pointed R127_nL/R from the old shared master tilt onto the per-band
  +/-total; removed the shared master inverter (U27-A) so BP_NTILT is gone
  everywhere; U27 kept for its still-live polarity-restore half.
- New parts: U82-84, RV48-50, R135-152, C119-124. New boundary MOD_BPn_TILT.
- Exact tilt-range reference/scaling is Phase-3R (noted), like block-6's other
  calibration items.

All 5 --check gates + parity green; boundary symmetry verified (BP_NTILT gone,
MOD_BPn_TILT symmetric). G5/G6a.

https://claude.ai/code/session_013jFXG5oeMVSYP7iRpwGvtQ
Parts:
- added C119, C120: 100nF, symbol Device:C
- added R135, R136, R138, R139, R140: 100k, symbol Device:R
- added R137: 470k, symbol Device:R
- added RV48: BP1_TILT, POGO_Potentiometer_THT:Potentiometer_Songhuei_9mm_TallTrimmer_Vertical, symbol Device:R_POT
- added U82: TL072, symbol Amplifier_Operational:OPA1612
Connections:
- net +12V: now also C119.2, RV48.1, U82.4 (V-)
- net -12V: now also C120.2, RV48.3, U82.8 (V+)
- net BP_TILT_CV: now also R135.2; no longer R127_1L.2
- net GND: now also C119.1, C120.1, U82.2 (In-), U82.6 (In-)
- net BP_NTILT renamed BP1_TILT_NEG
- net BP1_TILT_NEG: now also R138.1, R139.2, U82.1 (Out)
- new net BP1_TILTSUM: R135.1, R136.1, R137.1, R138.2, U82.3 (In+)
- new net BP1_TILT_INVN: R139.1, R140.2, U82.5 (In+)
- new net BP1_TILT_KNOB: R136.2, RV48.2 (Wiper)
- new net BP1_TILT_POS: R127_1L.2, R140.1, U82.7 (Out)
- new net MOD_BP1_TILT: R137.2
