File: kicad/pogo-block-6-svf2.kicad_sch (KiCad schematic)
At the start: 64 parts, among them U17 LM13700, U18 LM13700, U23 OPA1612, U24 OPA1612, U29 THAT340, U68 LM13700, U71 THAT340

Commit message: 0018: block-6 stage 1 - F_REF 400Hz all bands + pole-count doc
Per user confirmation, the plugin's F_REF = {400,400,400} is correct (the
{200,1500,6000} formant spread was a stale code comment). Align the hardware:
- All 3 BP integrator caps (C15/C19/C23) -> 68nF C0G 0805 (was 150/22/4.7nF),
  trimmed to 400Hz by each band's f_ref trim. Bands now default to the same
  center and the player spreads them via the FREQ knobs.
- spec §2 f_ref table, expo-trim targets, and cap derivation updated to 400Hz;
  fixed the stale '3x THAT340 shared L/R' -> 6x per-channel.
- Resolved the long-standing BP '4-pole vs 2-pole' question: the plugin BP is a
  single 2-pole SVFGroup (returns v1), so hardware 2-pole MATCHES. Corrected
  the wrong '4-pole DSP cascade' claim in aux-ota-c-svf.

All five --check gates + parity green.

https://claude.ai/code/session_013jFXG5oeMVSYP7iRpwGvtQ
Parts:
- C19_Lv1, C19_Lv2, C19_Rv1, C19_Rv2: value 22nF -> 68nF
Changed lines of the file:
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@@
   (property "Reference" "C19_Lv1" (at 103.000 538.000 0)
     (effects (font (size 1.27 1.27)) (justify left)))
-  (property "Value" "22nF" (at 103.000 534.500 0)
+  (property "Value" "68nF" (at 103.000 534.500 0)
     (effects (font (size 1.016 1.016)) (justify left) (hide yes)))
 )
@@
   (property "Reference" "C19_Lv2" (at 163.000 538.000 0)
     (effects (font (size 1.27 1.27)) (justify left)))
-  (property "Value" "22nF" (at 163.000 534.500 0)
+  (property "Value" "68nF" (at 163.000 534.500 0)
     (effects (font (size 1.016 1.016)) (justify left) (hide yes)))
 )
@@
   (property "Reference" "C19_Rv1" (at 103.000 758.000 0)
     (effects (font (size 1.27 1.27)) (justify left)))
-  (property "Value" "22nF" (at 103.000 754.500 0)
+  (property "Value" "68nF" (at 103.000 754.500 0)
     (effects (font (size 1.016 1.016)) (justify left) (hide yes)))
 )
@@
   (property "Reference" "C19_Rv2" (at 163.000 758.000 0)
     (effects (font (size 1.27 1.27)) (justify left)))
-  (property "Value" "22nF" (at 163.000 754.500 0)
+  (property "Value" "68nF" (at 163.000 754.500 0)
     (effects (font (size 1.016 1.016)) (justify left) (hide yes)))
 )

Commit message: 0018: block-6 stage 2 - distortion BEFORE bandpass (0017 reorder)
The core 0017 change: flip the per-band order from SVF->DIST to DIST->SVF to
match the plugin (Pogo.cpp:443-451). Realized as a net re-point across the 7
split sections (no part changes):
  LP1_OUT / BP3IN  ->  distN (R18/R20/R22 distortion inputs)
                   ->  mux out (BPn_DISTOUT)  ->  svfN SUM_AMP (R13)
                   ->  SVF v1 buffer (BPn_BANDOUT / BP3_TAP)  ->  mix wet summer
- BP1/BP2 take the LP1 band; BP3 takes BP3IN (the ALT/LP1 selector, stage 3).
- BP3 OUT tap now taken post-bandpass (BP3_TAP = svf3 v1), matching the plugin
  (prevOut[2]); block-B keeps the BP3_TAP net name (no block-B change).
- spec §1/§2 updated: signal order, DIST knob, ALT path (through-VCA/BP3-only),
  BP3 tap point.

Boundary symmetry verified for all re-pointed nets; all 5 --check gates +
parity green.

https://claude.ai/code/session_013jFXG5oeMVSYP7iRpwGvtQ
Connections:
- net BP2_BPBUF_L renamed BP2_BANDOUT_L
- net BP2_BPBUF_R renamed BP2_BANDOUT_R
- net LP1_OUT_L renamed BP2_DISTOUT_L
- net LP1_OUT_R renamed BP2_DISTOUT_R
Changed lines of the file:
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@@
   (effects (font (size 1.016 1.016)) (justify left))
 )
-(global_label "LP1_OUT_L"
+(global_label "BP2_DISTOUT_L"
   (shape output)
   (at 40.000 428.810 0)
   (effects (font (size 1.016 1.016)) (justify left))
 )
-(global_label "LP1_OUT_R"
+(global_label "BP2_DISTOUT_R"
   (shape output)
   (at 40.000 648.810 0)
@@
   (effects (font (size 1.016 1.016)) (justify left))
 )
-(global_label "BP2_BPBUF_L"
+(global_label "BP2_BANDOUT_L"
   (shape output)
   (at 47.620 172.000 0)
   (effects (font (size 1.016 1.016)) (justify left))
 )
-(global_label "BP2_BPBUF_L"
+(global_label "BP2_BANDOUT_L"
   (shape output)
   (at 32.380 174.540 0)
@@
   (effects (font (size 1.016 1.016)) (justify left))
 )
-(global_label "BP2_BPBUF_R"
+(global_label "BP2_BANDOUT_R"
   (shape output)
   (at 47.620 227.000 0)
   (effects (font (size 1.016 1.016)) (justify left))
 )
-(global_label "BP2_BPBUF_R"
+(global_label "BP2_BANDOUT_R"
   (shape output)
   (at 32.380 229.540 0)

Commit message: 0018: block-6 stage 4 - per-band BP TILT (summer+inverter/band)
The per-band tilt was entirely unbuilt (the panel BP1/2/3 TILT knobs had no
hardware control component at all, and only the master tilt was wired). Build
it to match the plugin's groupTiltV[i] = BPn_TILT_PARAM + CV*0.22:
- Per band (svf1/2/3): +1 TL072 (U82-84) as an inverting summer + inverter.
  Summer combines master tilt (BP_TILT_CV, 100k) + the per-band TILT knob
  (RV48-50 bipolar, 100k) + the per-band TILT CV (MOD_BPn_TILT from block-3,
  470k -> x0.213 ~= the plugin's x0.22). -total feeds the R expo base; the
  inverter's +total feeds the L expo base.
- Re-pointed R127_nL/R from the old shared master tilt onto the per-band
  +/-total; removed the shared master inverter (U27-A) so BP_NTILT is gone
  everywhere; U27 kept for its still-live polarity-restore half.
- New parts: U82-84, RV48-50, R135-152, C119-124. New boundary MOD_BPn_TILT.
- Exact tilt-range reference/scaling is Phase-3R (noted), like block-6's other
  calibration items.

All 5 --check gates + parity green; boundary symmetry verified (BP_NTILT gone,
MOD_BPn_TILT symmetric). G5/G6a.

https://claude.ai/code/session_013jFXG5oeMVSYP7iRpwGvtQ
Parts:
- added C121, C122: 100nF, symbol Device:C
- added R141, R142, R144, R145, R146: 100k, symbol Device:R
- added R143: 470k, symbol Device:R
- added RV49: BP2_TILT, POGO_Potentiometer_THT:Potentiometer_Songhuei_9mm_TallTrimmer_Vertical, symbol Device:R_POT
- added U83: TL072, POGO_Package_SO:SOIC-8_3.9x4.9mm_P1.27mm, symbol Amplifier_Operational:OPA1612
Connections:
- net +12V: now also C121.2, RV49.1, U83.4 (V-)
- net -12V: now also C122.2, RV49.3, U83.8 (V+)
- net BP_TILT_CV: now also R141.2; no longer R127_2L.2
- net GND: now also C121.1, C122.1, U83.2 (In-), U83.6 (In-)
- net BP_NTILT renamed BP2_TILT_NEG
- net BP2_TILT_NEG: now also R144.1, R145.2, U83.1 (Out)
- new net BP2_TILTSUM: R141.1, R142.1, R143.1, R144.2, U83.3 (In+)
- new net BP2_TILT_INVN: R145.1, R146.2, U83.5 (In+)
- new net BP2_TILT_KNOB: R142.2, RV49.2 (Wiper)
- new net BP2_TILT_POS: R127_2L.2, R146.1, U83.7 (Out)
- new net MOD_BP2_TILT: R143.2
