File: kicad/pogo-block-3.kicad_sch (KiCad schematic)
At the start: 170 parts, among them J10 LP1_RES, J11 BP_FREQ, J12 BP_TILT, J13 BP1_FREQ, J14 BP1_FOCUS, J15 BP1_DIST, J16 BP2_FREQ, J17 BP2_FOCUS, J18 BP2_DIST, J19 BP3_FREQ, J20 BP3_FOCUS, J21 BP3_DIST, J22 HP_FREQ, J23 HP_RES, J24 LP2_FREQ, J25 LP2_RES, J7 MOD_IN, J8 LP1_FREQ, J9 LP1_TILT, U3 TL074, U4 TL074, U5 TL074, U6 TL074, U7 TL074, U8 TL074, U9 TL074

Commit message: 0015-component-audit: apply component verification fixes
Board-breaking:
- that2180: real MPN THAT2180AL08-U (grade A) + package SIP-8 (THT); vendor
  Package_SIP/SIP-8_2.54mm footprint; fix components.yaml U4/U5 + CLAUDE.md.
  The 2180 has no SMD/SOIC variant.
- bat54s: redraw symbol to real series topology (1=A1, 2=K2, 3=K1;A2 junction);
  swap pins 2<->3 on all 24 BAT54S instances (blocks A/1/3/4) so signal sits on the
  junction (pin3), +12V on K2 (pin2), -12V on A1 (pin1); fix aux-cv-protection.md +
  block-A spec (both mislabeled the signal node as pin 2).

Other:
- R_INV_IN/R_INV_FB: add tol 1% (header-required >60 dB null).
- slide_pot_45mm: MPN RA4522F (Alpha 45mm, Rapid/Banzai); fix datasheet link.
- bzx84c10: add shared BZX84_SER datasheet (committed PDF + sha256); canonical MPN.
- opa1612: add symbol opamp2. bourns_3296w/3224w: fix version strings.
- cd4053 symbol doc# -> SCHS047O; c.yaml pin1 '+' -> '~' (non-polarized).

Jack S/T/TN reconciliation deferred (its own change). Plugin DSP untouched.
Regenerated all schematics, BOM, fp-lib-table, footprint SVGs, panel; 5 gates green.
Connections:
- net +12V: now also D3_1.2 (K2), D3_10.2 (K2), D3_11.2 (K2), D3_12.2 (K2), D3_13.2 (K2), D3_14.2 (K2), D3_15.2 (K2), D3_16.2 (K2), D3_17.2 (K2), D3_18.2 (K2), D3_2.2 (K2), D3_3.2 (K2), D3_4.2 (K2), D3_5.2 (K2), D3_6.2 (K2), D3_7.2 (K2), D3_8.2 (K2), D3_9.2 (K2), D4.2 (K2); no longer D3_1.3 (K2), D3_10.3 (K2), D3_11.3 (K2), D3_12.3 (K2), D3_13.3 (K2), D3_14.3 (K2), D3_15.3 (K2), D3_16.3 (K2), D3_17.3 (K2), D3_18.3 (K2), D3_2.3 (K2), D3_3.3 (K2), D3_4.3 (K2), D3_5.3 (K2), D3_6.3 (K2), D3_7.3 (K2), D3_8.3 (K2), D3_9.3 (K2), D4.3 (K2)

Commit message: 0016: source Song Huei R0904N + repoint panel-pot BOM refs (G6a)
- new part components/parts/songhuei_r0904n (matches lin/log/bipolar pot)
- move taper tags off alpha_rd901f (keeps knob/large/xl knob)
- RV41/RV43 (HP_RES/LP2_RES) Bourns 3296W -> R0904N finger pot
- regen block-2/3/4 schematics (att/LFO/VCA pot footprint) + BOM
Parts:
- RV10, RV11, RV12, RV13, RV14, RV15, RV16, RV17, RV18, RV19, RV20, RV21, RV22, RV23, RV3, RV4, RV5, RV6, RV7, RV8, RV9: footprint POGO_Potentiometer_THT:Potentiometer_Alpha_RD901F-40-00D_Single_Vertical_CircularHoles -> POGO_Potentiometer_THT:Potentiometer_Songhuei_9mm_TallTrimmer_Vertical
Changed lines of the file:
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@@
   (property "Value" "MOD_SCALE" (at 103.000 314.500 0)
     (effects (font (size 1.016 1.016)) (justify left) (hide yes)))
-  (property "Footprint" "POGO_Potentiometer_THT:Potentiometer_Alpha_RD901F-40-00D_Single_Vertical_CircularHoles" (at 100.000 315.000 0)
+  (property "Footprint" "POGO_Potentiometer_THT:Potentiometer_Songhuei_9mm_TallTrimmer_Vertical" (at 100.000 315.000 0)
     (effects (font (size 1.016 1.016)) (hide yes)))
 )
@@
   (property "Value" "MOD_OFFSET" (at 163.000 314.500 0)
     (effects (font (size 1.016 1.016)) (justify left) (hide yes)))
-  (property "Footprint" "POGO_Potentiometer_THT:Potentiometer_Alpha_RD901F-40-00D_Single_Vertical_CircularHoles" (at 160.000 315.000 0)
+  (property "Footprint" "POGO_Potentiometer_THT:Potentiometer_Songhuei_9mm_TallTrimmer_Vertical" (at 160.000 315.000 0)
     (effects (font (size 1.016 1.016)) (hide yes)))
 )
@@
   (property "Value" "LP1_FREQ_ATT" (at 103.000 809.500 0)
     (effects (font (size 1.016 1.016)) (justify left) (hide yes)))
-  (property "Footprint" "POGO_Potentiometer_THT:Potentiometer_Alpha_RD901F-40-00D_Single_Vertical_CircularHoles" (at 100.000 810.000 0)
+  (property "Footprint" "POGO_Potentiometer_THT:Potentiometer_Songhuei_9mm_TallTrimmer_Vertical" (at 100.000 810.000 0)
     (effects (font (size 1.016 1.016)) (hide yes)))
 )
@@
   (property "Value" "LP1_TILT_ATT" (at 163.000 919.500 0)
     (effects (font (size 1.016 1.016)) (justify left) (hide yes)))
-  (property "Footprint" "POGO_Potentiometer_THT:Potentiometer_Alpha_RD901F-40-00D_Single_Vertical_CircularHoles" (at 160.000 920.000 0)
+  (property "Footprint" "POGO_Potentiometer_THT:Potentiometer_Songhuei_9mm_TallTrimmer_Vertical" (at 160.000 920.000 0)
     (effects (font (size 1.016 1.016)) (hide yes)))
 )
@@
   (property "Value" "LP1_RES_ATT" (at 43.000 1084.500 0)
     (effects (font (size 1.016 1.016)) (justify left) (hide yes)))
-  (property "Footprint" "POGO_Potentiometer_THT:Potentiometer_Alpha_RD901F-40-00D_Single_Vertical_CircularHoles" (at 40.000 1085.000 0)
+  (property "Footprint" "POGO_Potentiometer_THT:Potentiometer_Songhuei_9mm_TallTrimmer_Vertical" (at 40.000 1085.000 0)
     (effects (font (size 1.016 1.016)) (hide yes)))
 )
@@
   (property "Value" "BP_FREQ_ATT" (at 103.000 1194.500 0)
     (effects (font (size 1.016 1.016)) (justify left) (hide yes)))
-  (property "Footprint" "POGO_Potentiometer_THT:Potentiometer_Alpha_RD901F-40-00D_Single_Vertical_CircularHoles" (at 100.000 1195.000 0)
+  (property "Footprint" "POGO_Potentiometer_THT:Potentiometer_Songhuei_9mm_TallTrimmer_Vertical" (at 100.000 1195.000 0)
     (effects (font (size 1.016 1.016)) (hide yes)))
 )
@@
   (property "Value" "BP_TILT_ATT" (at 163.000 1304.500 0)
     (effects (font (size 1.016 1.016)) (justify left) (hide yes)))
-  (property "Footprint" "POGO_Potentiometer_THT:Potentiometer_Alpha_RD901F-40-00D_Single_Vertical_CircularHoles" (at 160.000 1305.000 0)
+  (property "Footprint" "POGO_Potentiometer_THT:Potentiometer_Songhuei_9mm_TallTrimmer_Vertical" (at 160.000 1305.000 0)
     (effects (font (size 1.016 1.016)) (hide yes)))
 )
@@
   (property "Value" "BP1_FREQ_ATT" (at 43.000 1469.500 0)
     (effects (font (size 1.016 1.016)) (justify left) (hide yes)))
-  (property "Footprint" "POGO_Potentiometer_THT:Potentiometer_Alpha_RD901F-40-00D_Single_Vertical_CircularHoles" (at 40.000 1470.000 0)
+  (property "Footprint" "POGO_Potentiometer_THT:Potentiometer_Songhuei_9mm_TallTrimmer_Vertical" (at 40.000 1470.000 0)
     (effects (font (size 1.016 1.016)) (hide yes)))
 )
@@
   (property "Value" "BP1_FOCUS_ATT" (at 103.000 1579.500 0)
     (effects (font (size 1.016 1.016)) (justify left) (hide yes)))
-  (property "Footprint" "POGO_Potentiometer_THT:Potentiometer_Alpha_RD901F-40-00D_Single_Vertical_CircularHoles" (at 100.000 1580.000 0)
+  (property "Footprint" "POGO_Potentiometer_THT:Potentiometer_Songhuei_9mm_TallTrimmer_Vertical" (at 100.000 1580.000 0)
     (effects (font (size 1.016 1.016)) (hide yes)))
 )
@@
   (property "Value" "BP1_DIST_ATT" (at 163.000 1689.500 0)
     (effects (font (size 1.016 1.016)) (justify left) (hide yes)))
-  (property "Footprint" "POGO_Potentiometer_THT:Potentiometer_Alpha_RD901F-40-00D_Single_Vertical_CircularHoles" (at 160.000 1690.000 0)
+  (property "Footprint" "POGO_Potentiometer_THT:Potentiometer_Songhuei_9mm_TallTrimmer_Vertical" (at 160.000 1690.000 0)
     (effects (font (size 1.016 1.016)) (hide yes)))
 )
@@
   (property "Value" "BP2_FREQ_ATT" (at 43.000 1854.500 0)
     (effects (font (size 1.016 1.016)) (justify left) (hide yes)))
-  (property "Footprint" "POGO_Potentiometer_THT:Potentiometer_Alpha_RD901F-40-00D_Single_Vertical_CircularHoles" (at 40.000 1855.000 0)
+  (property "Footprint" "POGO_Potentiometer_THT:Potentiometer_Songhuei_9mm_TallTrimmer_Vertical" (at 40.000 1855.000 0)
     (effects (font (size 1.016 1.016)) (hide yes)))
 )
@@
   (property "Value" "BP2_FOCUS_ATT" (at 103.000 1964.500 0)
     (effects (font (size 1.016 1.016)) (justify left) (hide yes)))
-  (property "Footprint" "POGO_Potentiometer_THT:Potentiometer_Alpha_RD901F-40-00D_Single_Vertical_CircularHoles" (at 100.000 1965.000 0)
+  (property "Footprint" "POGO_Potentiometer_THT:Potentiometer_Songhuei_9mm_TallTrimmer_Vertical" (at 100.000 1965.000 0)
     (effects (font (size 1.016 1.016)) (hide yes)))
 )
@@
   (property "Value" "BP2_DIST_ATT" (at 163.000 2074.500 0)
     (effects (font (size 1.016 1.016)) (justify left) (hide yes)))
-  (property "Footprint" "POGO_Potentiometer_THT:Potentiometer_Alpha_RD901F-40-00D_Single_Vertical_CircularHoles" (at 160.000 2075.000 0)
+  (property "Footprint" "POGO_Potentiometer_THT:Potentiometer_Songhuei_9mm_TallTrimmer_Vertical" (at 160.000 2075.000 0)
     (effects (font (size 1.016 1.016)) (hide yes)))
 )
@@
   (property "Value" "BP3_FREQ_ATT" (at 43.000 2239.500 0)
     (effects (font (size 1.016 1.016)) (justify left) (hide yes)))
-  (property "Footprint" "POGO_Potentiometer_THT:Potentiometer_Alpha_RD901F-40-00D_Single_Vertical_CircularHoles" (at 40.000 2240.000 0)
+  (property "Footprint" "POGO_Potentiometer_THT:Potentiometer_Songhuei_9mm_TallTrimmer_Vertical" (at 40.000 2240.000 0)
     (effects (font (size 1.016 1.016)) (hide yes)))
 )
@@
   (property "Value" "BP3_FOCUS_ATT" (at 103.000 2349.500 0)
     (effects (font (size 1.016 1.016)) (justify left) (hide yes)))
-  (property "Footprint" "POGO_Potentiometer_THT:Potentiometer_Alpha_RD901F-40-00D_Single_Vertical_CircularHoles" (at 100.000 2350.000 0)
+  (property "Footprint" "POGO_Potentiometer_THT:Potentiometer_Songhuei_9mm_TallTrimmer_Vertical" (at 100.000 2350.000 0)
     (effects (font (size 1.016 1.016)) (hide yes)))
 )
@@
   (property "Value" "BP3_DIST_ATT" (at 163.000 2459.500 0)
     (effects (font (size 1.016 1.016)) (justify left) (hide yes)))
-  (property "Footprint" "POGO_Potentiometer_THT:Potentiometer_Alpha_RD901F-40-00D_Single_Vertical_CircularHoles" (at 160.000 2460.000 0)
+  (property "Footprint" "POGO_Potentiometer_THT:Potentiometer_Songhuei_9mm_TallTrimmer_Vertical" (at 160.000 2460.000 0)
     (effects (font (size 1.016 1.016)) (hide yes)))
 )
@@
   (property "Value" "HP_FREQ_ATT" (at 43.000 2624.500 0)
     (effects (font (size 1.016 1.016)) (justify left) (hide yes)))
-  (property "Footprint" "POGO_Potentiometer_THT:Potentiometer_Alpha_RD901F-40-00D_Single_Vertical_CircularHoles" (at 40.000 2625.000 0)
+  (property "Footprint" "POGO_Potentiometer_THT:Potentiometer_Songhuei_9mm_TallTrimmer_Vertical" (at 40.000 2625.000 0)
     (effects (font (size 1.016 1.016)) (hide yes)))
 )
@@
   (property "Value" "HP_RES_ATT" (at 103.000 2734.500 0)
     (effects (font (size 1.016 1.016)) (justify left) (hide yes)))
-  (property "Footprint" "POGO_Potentiometer_THT:Potentiometer_Alpha_RD901F-40-00D_Single_Vertical_CircularHoles" (at 100.000 2735.000 0)
+  (property "Footprint" "POGO_Potentiometer_THT:Potentiometer_Songhuei_9mm_TallTrimmer_Vertical" (at 100.000 2735.000 0)
     (effects (font (size 1.016 1.016)) (hide yes)))
 )
@@
   (property "Value" "LP2_FREQ_ATT" (at 163.000 2844.500 0)
     (effects (font (size 1.016 1.016)) (justify left) (hide yes)))
-  (property "Footprint" "POGO_Potentiometer_THT:Potentiometer_Alpha_RD901F-40-00D_Single_Vertical_CircularHoles" (at 160.000 2845.000 0)
+  (property "Footprint" "POGO_Potentiometer_THT:Potentiometer_Songhuei_9mm_TallTrimmer_Vertical" (at 160.000 2845.000 0)
     (effects (font (size 1.016 1.016)) (hide yes)))
 )
@@
   (property "Value" "LP2_RES_ATT" (at 43.000 3009.500 0)
     (effects (font (size 1.016 1.016)) (justify left) (hide yes)))
-  (property "Footprint" "POGO_Potentiometer_THT:Potentiometer_Alpha_RD901F-40-00D_Single_Vertical_CircularHoles" (at 40.000 3010.000 0)
+  (property "Footprint" "POGO_Potentiometer_THT:Potentiometer_Songhuei_9mm_TallTrimmer_Vertical" (at 40.000 3010.000 0)
     (effects (font (size 1.016 1.016)) (hide yes)))
 )
@@
   (property "Value" "VCA_AMT_ATT" (at 103.000 3119.500 0)
     (effects (font (size 1.016 1.016)) (justify left) (hide yes)))
-  (property "Footprint" "POGO_Potentiometer_THT:Potentiometer_Alpha_RD901F-40-00D_Single_Vertical_CircularHoles" (at 100.000 3120.000 0)
-    (effects (font (size 1.016 1.016)) (hide yes)))
-)
+  (property "Footprint" "POGO_Potentiometer_THT:Potentiometer_Songhuei_9mm_TallTrimmer_Vertical" (at 100.000 3120.000 0)
+    (effects (font (size 1.016 1.016)) (hide yes)))
+)

Commit message: 0018: block-3 mod bus aligned to plugin (MOD_SRC, LEDs, VCA, FOCUS→TILT)
Largest block of the alignment pass. Changes:
- MOD_SRC: wire SW7 (DW5) as a 3-way analog source select LFO1/LFO2/EXT
  (DPDT commons bridged); MOD_IN becomes EXT-only (no LFO auto-normal);
  accept LFO1_OUT + LFO2_OUT boundary inputs from block-2.
- Remove the 3 MOD-bus LEDs (POS/NEG/CLIP) + driver U4 + R56-R60: the
  plugin drives no such lights and the locked panel has no footprints
  (7x -> 6x TL074).
- VCA: remove the block-3 VCA_AMT attenuverter (RV5 + inverter); per the
  plugin the raw mod bus normals into VCA_INPUT (no attenuverter) and the
  VCA_AMT depth pot belongs to block-4.
- Rename per-band BP*_FOCUS -> BP*_TILT (plugin/panel have TILT CV; FOCUS/Q
  has no CV input) across nets, components, spec.
- Refresh aux-mod-bus-core + aux-attenuverter; drop the phantom distribution
  buffer (bus drives 18x100k R_SRC_NORM ~5.6k, no buffer needed).
- Destination set: 18 attenuverters + 1 raw VCA normal.

All five --check gates green; parity OK. Block-3 schematic + BOM regenerated.

https://claude.ai/code/session_013jFXG5oeMVSYP7iRpwGvtQ
Parts:
- removed D3_17, D3_18: BAT54S, POGO_Package_TO_SOT_SMD:SOT-23, symbol Diode:BAT54S
- removed J24: LP2_FREQ, POGO_Connector_Audio:Jack_3.5mm_QingPu_WQP-PJ398SM_Vertical_CircularHoles, symbol Device:Audio_Jack_3.5mm_SwitchT
- removed J25: LP2_RES, POGO_Connector_Audio:Jack_3.5mm_QingPu_WQP-PJ398SM_Vertical_CircularHoles, symbol Device:Audio_Jack_3.5mm_SwitchT
- removed R18_17, R18_18: 100k, symbol Device:R
- removed R37_17, R37_18: 100R, symbol Device:R
- removed RV22: LP2_FREQ_ATT, POGO_Potentiometer_THT:Potentiometer_Songhuei_9mm_TallTrimmer_Vertical, symbol Device:R_POT
- removed RV23: LP2_RES_ATT, POGO_Potentiometer_THT:Potentiometer_Songhuei_9mm_TallTrimmer_Vertical, symbol Device:R_POT
- removed RV5: VCA_AMT_ATT, POGO_Potentiometer_THT:Potentiometer_Songhuei_9mm_TallTrimmer_Vertical, symbol Device:R_POT
- removed R_INV_FB_17, R_INV_FB_18, R_INV_FB_19, R_INV_IN_17, R_INV_IN_18, R_INV_IN_19: 10k, symbol Device:R
- C7_1: renamed from D6; value BZX84C10 -> 100nF; footprint POGO_Package_TO_SOT_SMD:SOT-23 -> (none); symbol Diode:D_Zener -> Device:C
- C7_10: renamed from J7; value MOD_IN -> 100nF; footprint POGO_Connector_Audio:Jack_3.5mm_QingPu_WQP-PJ398SM_Vertical_CircularHoles -> (none); symbol Device:Audio_Jack_3.5mm_SwitchT -> Device:C
- C7_11: renamed from R57; value 1k -> 100nF; symbol Device:R -> Device:C
- C7_12: renamed from R59; value 9k9 -> 100nF; symbol Device:R -> Device:C
- C7_13: renamed from LED3; value MOD_POS -> 100nF; footprint POGO_LED_THT:LED_D3.0mm -> (none); symbol Device:LED -> Device:C
- C7_14: renamed from LED5; value MOD_CLIP -> 100nF; footprint POGO_LED_THT:LED_D3.0mm -> (none); symbol Device:LED -> Device:C
- C7_3: renamed from RV4; value MOD_OFFSET -> 100nF; footprint POGO_Potentiometer_THT:Potentiometer_Songhuei_9mm_TallTrimmer_Vertical -> (none); symbol Device:R_POT -> Device:C
- C7_4: renamed from R56; value 1k -> 100nF; symbol Device:R -> Device:C
- C7_5: renamed from R58; value 1k -> 100nF; symbol Device:R -> Device:C
- C7_6: renamed from R60; value 100R -> 100nF; symbol Device:R -> Device:C
- C7_7: renamed from LED4; value MOD_NEG -> 100nF; footprint POGO_LED_THT:LED_D3.0mm -> (none); symbol Device:LED -> Device:C
- C7_8: renamed from RV3; value MOD_SCALE -> 100nF; footprint POGO_Potentiometer_THT:Potentiometer_Songhuei_9mm_TallTrimmer_Vertical -> (none); symbol Device:R_POT -> Device:C
- D3_1: renamed from C7_10; value 100nF -> BAT54S; footprint (none) -> POGO_Package_TO_SOT_SMD:SOT-23; symbol Device:C -> Diode:BAT54S
- D3_2: renamed from C7_7; value 100nF -> BAT54S; footprint (none) -> POGO_Package_TO_SOT_SMD:SOT-23; symbol Device:C -> Diode:BAT54S
- D4: renamed from R14; value 22k -> BAT54S; footprint (none) -> POGO_Package_TO_SOT_SMD:SOT-23; symbol Device:R -> Diode:BAT54S
- D5: renamed from R15; value 100k -> BZX84C10; footprint (none) -> POGO_Package_TO_SOT_SMD:SOT-23; symbol Device:R -> Diode:D_Zener
- D6: renamed from R16_1; value 100k -> BZX84C10; footprint (none) -> POGO_Package_TO_SOT_SMD:SOT-23; symbol Device:R -> Diode:D_Zener
- J10: renamed from J8; value LP1_FREQ -> LP1_RES
- J11: renamed from J9; value LP1_TILT -> BP_FREQ
- J12: renamed from J10; value LP1_RES -> BP_TILT
- J13: renamed from J11; value BP_FREQ -> BP1_FREQ
- J14: renamed from J12; value BP_TILT -> BP1_TILT
- J15: renamed from J13; value BP1_FREQ -> BP1_DIST
- J16: renamed from J14; value BP1_FOCUS -> BP2_FREQ
- J17: renamed from J15; value BP1_DIST -> BP2_TILT
- J18: renamed from J16; value BP2_FREQ -> BP2_DIST
- J19: renamed from J17; value BP2_FOCUS -> BP3_FREQ
- J20: renamed from J18; value BP2_DIST -> BP3_TILT
- J21: renamed from J19; value BP3_FREQ -> BP3_DIST
- J22: renamed from J20; value BP3_FOCUS -> HP_FREQ
- J23: renamed from J21; value BP3_DIST -> HP_RES
- J24: renamed from J22; value HP_FREQ -> LP2_FREQ
- J25: renamed from J23; value HP_RES -> LP2_RES
- J7: renamed from D4; value BAT54S -> MOD_IN; footprint POGO_Package_TO_SOT_SMD:SOT-23 -> POGO_Connector_Audio:Jack_3.5mm_QingPu_WQP-PJ398SM_Vertical_CircularHoles; symbol Diode:BAT54S -> Device:Audio_Jack_3.5mm_SwitchT
- J8: renamed from C7_9; value 100nF -> LP1_FREQ; footprint (none) -> POGO_Connector_Audio:Jack_3.5mm_QingPu_WQP-PJ398SM_Vertical_CircularHoles; symbol Device:C -> Device:Audio_Jack_3.5mm_SwitchT
- J9: renamed from C7_6; value 100nF -> LP1_TILT; footprint (none) -> POGO_Connector_Audio:Jack_3.5mm_QingPu_WQP-PJ398SM_Vertical_CircularHoles; symbol Device:C -> Device:Audio_Jack_3.5mm_SwitchT
- R13: renamed from U9; value TL074 -> 100k; footprint POGO_Package_SO:SOIC-14_3.9x8.7mm_P1.27mm -> (none); symbol Amplifier_Operational:TL074 -> Device:R
- R14: renamed from U9; value TL074 -> 22k; symbol Amplifier_Operational:TL074 -> Device:R
- R15, R16_1, R16_2: renamed from U9; value TL074 -> 100k; symbol Amplifier_Operational:TL074 -> Device:R
- R18_1: renamed from C7_4; value 100nF -> 100k; symbol Device:C -> Device:R
- R18_2: renamed from C7_14; value 100nF -> 100k; symbol Device:C -> Device:R
- R37_1: renamed from C7_3; value 100nF -> 100R; symbol Device:C -> Device:R
- R37_2: renamed from C7_13; value 100nF -> 100R; symbol Device:C -> Device:R
- R99: renamed from R13; value 100k -> 100R
- RV10: renamed from RV8; value LP1_RES_ATT -> BP_TILT_ATT
- RV11: renamed from RV9; value BP_FREQ_ATT -> BP1_FREQ_ATT
- RV12: renamed from RV10; value BP_TILT_ATT -> BP1_TILT_ATT
- RV13: renamed from RV11; value BP1_FREQ_ATT -> BP1_DIST_ATT
- RV14: renamed from RV12; value BP1_FOCUS_ATT -> BP2_FREQ_ATT
- RV15: renamed from RV13; value BP1_DIST_ATT -> BP2_TILT_ATT
- RV16: renamed from RV14; value BP2_FREQ_ATT -> BP2_DIST_ATT
- RV17: renamed from RV15; value BP2_FOCUS_ATT -> BP3_FREQ_ATT
- RV18: renamed from RV16; value BP2_DIST_ATT -> BP3_TILT_ATT
- RV19: renamed from RV17; value BP3_FREQ_ATT -> BP3_DIST_ATT
- RV20: renamed from RV18; value BP3_FOCUS_ATT -> HP_FREQ_ATT
- RV21: renamed from RV19; value BP3_DIST_ATT -> HP_RES_ATT
- RV22: renamed from RV20; value HP_FREQ_ATT -> LP2_FREQ_ATT
- RV23: renamed from RV21; value HP_RES_ATT -> LP2_RES_ATT
- RV3: renamed from R16_2; value 100k -> MOD_SCALE; footprint (none) -> POGO_Potentiometer_THT:Potentiometer_Songhuei_9mm_TallTrimmer_Vertical; symbol Device:R -> Device:R_POT
- RV4: renamed from R99; value 100R -> MOD_OFFSET; footprint (none) -> POGO_Potentiometer_THT:Potentiometer_Songhuei_9mm_TallTrimmer_Vertical; symbol Device:R -> Device:R_POT
- RV6: renamed from C7_2; value 100nF -> LP1_FREQ_ATT; footprint (none) -> POGO_Potentiometer_THT:Potentiometer_Songhuei_9mm_TallTrimmer_Vertical; symbol Device:C -> Device:R_POT
- RV7: renamed from C7_12; value 100nF -> LP1_TILT_ATT; footprint (none) -> POGO_Potentiometer_THT:Potentiometer_Songhuei_9mm_TallTrimmer_Vertical; symbol Device:C -> Device:R_POT
- RV8: renamed from RV6; value LP1_FREQ_ATT -> LP1_RES_ATT
- RV9: renamed from RV7; value LP1_TILT_ATT -> BP_FREQ_ATT
- R_INV_FB_1: renamed from C7_8; value 100nF -> 10k; symbol Device:C -> Device:R
- R_INV_FB_2: renamed from C7_5; value 100nF -> 10k; symbol Device:C -> Device:R
- R_INV_IN_1: renamed from C7_1; value 100nF -> 10k; symbol Device:C -> Device:R
- R_INV_IN_2: renamed from C7_11; value 100nF -> 10k; symbol Device:C -> Device:R
- SW7: renamed from D5; value BZX84C10 -> MOD_SRC; footprint POGO_Package_TO_SOT_SMD:SOT-23 -> (none); symbol Diode:D_Zener -> Switch:SW_Dailywell_DW5
- renumbered D3_8 to D3_10, D3_9 to D3_11, D3_10 to D3_12, D3_11 to D3_13, D3_12 to D3_14, D3_13 to D3_15, D3_14 to D3_16, D3_15 to D3_17, D3_16 to D3_18, D3_1 to D3_3, D3_2 to D3_4, D3_3 to D3_5, D3_4 to D3_6, D3_5 to D3_7, D3_6 to D3_8, D3_7 to D3_9, R18_8 to R18_10, R18_9 to R18_11, R18_10 to R18_12, R18_11 to R18_13, R18_12 to R18_14, R18_13 to R18_15, R18_14 to R18_16, R18_15 to R18_17, R18_16 to R18_18, R18_1 to R18_3, R18_2 to R18_4, R18_3 to R18_5, R18_4 to R18_6, R18_5 to R18_7, R18_6 to R18_8, R18_7 to R18_9, R37_8 to R37_10, R37_9 to R37_11, R37_10 to R37_12, R37_11 to R37_13, R37_12 to R37_14, R37_13 to R37_15, R37_14 to R37_16, R37_15 to R37_17, R37_16 to R37_18, R37_1 to R37_3, R37_2 to R37_4, R37_3 to R37_5, R37_4 to R37_6, R37_5 to R37_7, R37_6 to R37_8, R37_7 to R37_9, R_INV_FB_8 to R_INV_FB_10, R_INV_FB_9 to R_INV_FB_11, R_INV_FB_10 to R_INV_FB_12, R_INV_FB_11 to R_INV_FB_13, R_INV_FB_12 to R_INV_FB_14, R_INV_FB_13 to R_INV_FB_15, R_INV_FB_14 to R_INV_FB_16, R_INV_FB_15 to R_INV_FB_17, R_INV_FB_16 to R_INV_FB_18, R_INV_FB_1 to R_INV_FB_3, R_INV_FB_2 to R_INV_FB_4, R_INV_FB_3 to R_INV_FB_5, R_INV_FB_4 to R_INV_FB_6, R_INV_FB_5 to R_INV_FB_7, R_INV_FB_6 to R_INV_FB_8, R_INV_FB_7 to R_INV_FB_9, R_INV_IN_8 to R_INV_IN_10, R_INV_IN_9 to R_INV_IN_11, R_INV_IN_10 to R_INV_IN_12, R_INV_IN_11 to R_INV_IN_13, R_INV_IN_12 to R_INV_IN_14, R_INV_IN_13 to R_INV_IN_15, R_INV_IN_14 to R_INV_IN_16, R_INV_IN_15 to R_INV_IN_17, R_INV_IN_16 to R_INV_IN_18, R_INV_IN_1 to R_INV_IN_3, R_INV_IN_2 to R_INV_IN_4, R_INV_IN_3 to R_INV_IN_5, R_INV_IN_4 to R_INV_IN_6, R_INV_IN_5 to R_INV_IN_7, R_INV_IN_6 to R_INV_IN_8, R_INV_IN_7 to R_INV_IN_9, U4 to U5, U5 to U6, U6 to U7, U7 to U8, U8 to U9
Connections:
- net JSW_BP1_FOCUS is gone; now on net JSW_BP2_FREQ: R18_9.2
- net JSW_BP2_FOCUS is gone; now on net JSW_BP3_FREQ: R18_12.2
- net JSW_BP3_FOCUS is gone; now on net JSW_HP_FREQ: R18_15.2
- net JTIP_BP1_FOCUS is gone; now on net JTIP_BP2_FREQ: J16.1 (T), R37_9.2
- net JTIP_BP2_FOCUS is gone; now on net JTIP_BP3_FREQ: J19.1 (T), R37_12.2
- net JTIP_BP3_FOCUS is gone; now on net JTIP_HP_FREQ: J22.1 (T), R37_15.2
- net MOD_BP1_FOCUS is gone; now on net MOD_BP2_FREQ: RV14.2 (Wiper)
- net MOD_BP2_FOCUS is gone; now on net MOD_BP3_FREQ: RV17.2 (Wiper)
- net MOD_BP3_FOCUS is gone; now on net MOD_HP_FREQ: RV20.2 (Wiper)
- net VSRC_BP1_FOCUS is gone; now on net VSRC_BP2_FREQ: R37_9.1, RV14.1, R_INV_IN_9.2
- net VSRC_BP2_FOCUS is gone; now on net VSRC_BP3_FREQ: R37_12.1, RV17.1, R_INV_IN_12.2
- net VSRC_BP3_FOCUS is gone; now on net VSRC_HP_FREQ: R37_15.1, RV20.1, R_INV_IN_15.2
- net +12V: now also C7_1.2, C7_3.2, C7_4.2, C7_5.2, C7_6.2, C7_7.2, D3_1.2 (K2), D4.2 (K2), RV4.1; no longer C7_12.2, C7_3.1, J7.2 (K2), J9.2, R16_2.11 (V-), R18_1.2, R37_1.2, RV6.2, R_INV_FB_2.2, R_INV_IN_1.2
- net -12V: now also C7_10.2, C7_11.2, C7_12.2, C7_13.2, C7_14.2, C7_8.2, D3_1.1 (A1), D3_2.1 (A1), D4.1 (A1), RV4.3; no longer C7_3.3, D3_1.2, J7.1 (A1), J8.2, R16_2.4 (V+), R18_2.2, R37_2.2, RV7.2, R_INV_FB_1.2, R_INV_IN_2.2
- net GND: now also C7_1.1, C7_10.1, C7_11.1, C7_12.1, C7_13.1, C7_14.1, C7_3.1, C7_4.1, C7_5.1, C7_7.1, C7_8.1, D6.3 (K), J7.2 (S), J8.2 (S), J9.2 (S), U5.2 (In-), U5.9 (In-); no longer C7_1.3 (K), C7_10.2 (S), C7_13.A, C7_14.A, C7_7.A, D3_1.1, D3_2.1, J8.1, J9.1, R13.2 (In-), R14.6 (In-), R15.9 (In-), R16_1.13 (In-), R18_1.1, R18_2.1, R37_1.1, R37_2.1, RV6.1, RV7.1, R_INV_FB_1.1, R_INV_FB_2.1, R_INV_IN_1.1, R_INV_IN_2.1, U5.3 (In+)
- net INVN_BP1_DIST: now also R_INV_FB_8.2, R_INV_IN_8.1, U6.12 (In+); no longer R_INV_FB_10.2, R_INV_IN_10.1, U7.12 (In+)
- net INVN_BP1_FREQ: now also R_INV_FB_6.2, R_INV_IN_6.1, U6.5 (In+); no longer R_INV_FB_8.2, R_INV_IN_8.1, U7.5 (In+)
- net INVN_BP2_DIST: now also R_INV_FB_11.2, R_INV_IN_11.1, U7.10 (In+); no longer R_INV_FB_13.2, R_INV_IN_13.1, U8.10 (In+)
- net INVN_BP2_FREQ: now also R_INV_FB_9.2, R_INV_IN_9.1, U7.3 (In+); no longer R_INV_FB_11.2, R_INV_IN_11.1, U8.3 (In+)
- net INVN_BP3_DIST: now also R_INV_FB_14.2, R_INV_IN_14.1, U8.5 (In+); no longer R_INV_FB_16.2, R_INV_IN_16.1, U9.5 (In+)
- net INVN_BP3_FREQ: now also R_INV_FB_12.2, R_INV_IN_12.1, U7.12 (In+); no longer R_INV_FB_14.2, R_INV_IN_14.1, U8.12 (In+)
- net INVN_BP_FREQ: now also R_INV_FB_4.2, R_INV_IN_4.1, U5.12 (In+); no longer R_INV_FB_6.2, R_INV_IN_6.1, U6.12 (In+)
- net INVN_BP_TILT: now also R_INV_FB_5.2, R_INV_IN_5.1, U6.3 (In+); no longer R_INV_FB_7.2, R_INV_IN_7.1, U7.3 (In+)
- net INVN_HP_FREQ: now also R_INV_FB_15.2, R_INV_IN_15.1, U8.10 (In+); no longer R_INV_FB_17.2, R_INV_IN_17.1, U9.10 (In+)
- net INVN_HP_RES: now also R_INV_FB_16.2, R_INV_IN_16.1, U8.12 (In+); no longer R_INV_FB_18.2, R_INV_IN_18.1, U9.12 (In+)
- net INVN_LP1_FREQ: now also R_INV_FB_1.2, R_INV_IN_1.1, U5.3 (In+); no longer R_INV_FB_3.2, R_INV_IN_3.1, U6.3 (In+)
- net INVN_LP1_RES: now also R_INV_FB_3.2, R_INV_IN_3.1, U5.10 (In+); no longer R_INV_FB_5.2, R_INV_IN_5.1, U6.10 (In+)
- net INVN_LP1_TILT: now also R_INV_FB_2.2, R_INV_IN_2.1, U5.5 (In+); no longer R_INV_FB_4.2, R_INV_IN_4.1, U6.5 (In+)
- net INVN_LP2_FREQ: now also R_INV_FB_17.2, R_INV_IN_17.1, U9.3 (In+); no longer R13.3 (In+)
- net INVN_LP2_RES: now also R_INV_FB_18.2, R_INV_IN_18.1, U9.5 (In+); no longer R14.5 (In+)
- net JSW_BP1_DIST: now also R18_8.2; no longer R18_10.2
- net JSW_BP1_FREQ: now also R18_6.2; no longer R18_8.2
- net JSW_BP2_DIST: now also R18_11.2; no longer R18_13.2
- net JSW_BP2_FREQ: no longer R18_11.2
- net JSW_BP3_DIST: now also R18_14.2; no longer R18_16.2
- net JSW_BP3_FREQ: no longer R18_14.2
- net JSW_BP_FREQ: now also R18_4.2; no longer R18_6.2
- net JSW_BP_TILT: now also R18_5.2; no longer R18_7.2
- net JSW_HP_FREQ: no longer R18_17.2
- net JSW_HP_RES: now also R18_16.2; no longer R18_18.2
- net JSW_LP1_FREQ: now also R18_1.2; no longer R18_3.2
- net JSW_LP1_RES: now also R18_3.2; no longer R18_5.2
- net JSW_LP1_TILT: now also R18_2.2; no longer R18_4.2
- net JSW_LP2_FREQ: now also R18_17.2
- net JSW_LP2_RES: now also R18_18.2
- net JTIP_BP1_DIST: now also J15.1 (T), R37_8.2; no longer J17.1 (T), R37_10.2
- net JTIP_BP1_FREQ: now also J13.1 (T), R37_6.2; no longer J15.1 (T), R37_8.2
- net JTIP_BP2_DIST: now also J18.1 (T), R37_11.2; no longer J20.1 (T), R37_13.2
- net JTIP_BP2_FREQ: no longer J18.1 (T), R37_11.2
- net JTIP_BP3_DIST: now also J21.1 (T), R37_14.2; no longer J23.1 (T), R37_16.2
- net JTIP_BP3_FREQ: no longer J21.1 (T), R37_14.2
- net JTIP_BP_FREQ: now also J11.1 (T), R37_4.2; no longer J13.1 (T), R37_6.2
- net JTIP_BP_TILT: now also J12.1 (T), R37_5.2; no longer J14.1 (T), R37_7.2
- net JTIP_HP_FREQ: no longer J24.1 (T), R37_17.2
- net JTIP_HP_RES: now also J23.1 (T), R37_16.2; no longer J25.1 (T), R37_18.2
- net JTIP_LP1_FREQ: now also J8.1 (T), R37_1.2; no longer J10.1 (T), R37_3.2
- net JTIP_LP1_RES: now also J10.1 (T), R37_3.2; no longer J12.1 (T), R37_5.2
- net JTIP_LP1_TILT: now also J9.1 (T), R37_2.2; no longer J11.1 (T), R37_4.2
- net JTIP_LP2_FREQ: now also J24.1 (T), R37_17.2
- net JTIP_LP2_RES: now also J25.1 (T), R37_18.2
- net LFO1_OUT: now also SW7.6 (B2)
- net MB_INVN: now also R16_1.1, R16_2.2; no longer D6.1, RV3.2
- net MB_SUMINV: now also R13.2, R14.1, R15.1; no longer D4.1, D5.1, R99.2
- net MOD_BP1_DIST: now also RV13.2 (Wiper); no longer RV15.2 (Wiper)
- net MOD_BP1_FREQ: now also RV11.2 (Wiper); no longer RV13.2 (Wiper)
- net MOD_BP2_DIST: now also RV16.2 (Wiper); no longer RV18.2 (Wiper)
- net MOD_BP2_FREQ: no longer RV16.2 (Wiper)
- net MOD_BP3_DIST: now also RV19.2 (Wiper); no longer RV21.2 (Wiper)
- net MOD_BP3_FREQ: no longer RV19.2 (Wiper)
- net MOD_BP_FREQ: now also RV9.2 (Wiper); no longer RV11.2 (Wiper)
- net MOD_BP_TILT: now also RV10.2 (Wiper); no longer RV12.2 (Wiper)
- net MOD_HP_FREQ: no longer RV22.2 (Wiper)
- net MOD_HP_RES: now also RV21.2 (Wiper); no longer RV23.2 (Wiper)
- net MOD_IN_TIP: now also J7.1 (T), R99.2; no longer C7_10.1 (T), RV4.2
- net MOD_LP1_FREQ: now also RV6.2 (Wiper); no longer RV8.2 (Wiper)
- net MOD_LP1_RES: now also RV8.2 (Wiper); no longer RV10.2 (Wiper)
- net MOD_LP1_TILT: now also RV7.2 (Wiper); no longer RV9.2 (Wiper)
- net MOD_LP2_FREQ: now also RV22.2 (Wiper)
- net MOD_LP2_RES: now also RV23.2 (Wiper)
- net NVSRC_BP1_DIST: now also RV13.3, R_INV_FB_8.1, U6.14 (Out); no longer RV15.3, R_INV_FB_10.1, U7.14 (Out)
- net NVSRC_BP1_FREQ: now also RV11.3, R_INV_FB_6.1, U6.7 (Out); no longer RV13.3, R_INV_FB_8.1, U7.7 (Out)
- net NVSRC_BP2_DIST: now also RV16.3, R_INV_FB_11.1, U7.8 (Out); no longer RV18.3, R_INV_FB_13.1, U8.8 (Out)
- net NVSRC_BP2_FREQ: now also RV14.3, R_INV_FB_9.1, U7.1 (Out); no longer RV16.3, R_INV_FB_11.1, U8.1 (Out)
- net NVSRC_BP3_DIST: now also RV19.3, R_INV_FB_14.1, U8.7 (Out); no longer RV21.3, R_INV_FB_16.1, U9.7 (Out)
- net NVSRC_BP3_FREQ: now also RV17.3, R_INV_FB_12.1, U7.14 (Out); no longer RV19.3, R_INV_FB_14.1, U8.14 (Out)
- net NVSRC_BP_FREQ: now also RV9.3, R_INV_FB_4.1, U5.14 (Out); no longer RV11.3, R_INV_FB_6.1, U6.14 (Out)
- net NVSRC_BP_TILT: now also RV10.3, R_INV_FB_5.1, U6.1 (Out); no longer RV12.3, R_INV_FB_7.1, U7.1 (Out)
- net NVSRC_HP_FREQ: now also RV20.3, R_INV_FB_15.1, U8.8 (Out); no longer RV22.3, R_INV_FB_17.1, U9.8 (Out)
- net NVSRC_HP_RES: now also RV21.3, R_INV_FB_16.1, U8.14 (Out); no longer RV23.3, R_INV_FB_18.1, U9.14 (Out)
- net NVSRC_LP1_FREQ: now also RV6.3, R_INV_FB_1.1, U5.1 (Out); no longer RV8.3, R_INV_FB_3.1, U6.1 (Out)
- net NVSRC_LP1_RES: now also RV8.3, R_INV_FB_3.1, U5.8 (Out); no longer RV10.3, R_INV_FB_5.1, U6.8 (Out)
- net NVSRC_LP1_TILT: now also RV7.3, R_INV_FB_2.1, U5.7 (Out); no longer RV9.3, R_INV_FB_4.1, U6.7 (Out)
- net NVSRC_LP2_FREQ: now also RV22.3, R_INV_FB_17.1, U9.1 (Out); no longer R13.1 (Out)
- net NVSRC_LP2_RES: now also RV23.3, R_INV_FB_18.1, U9.7 (Out); no longer R14.7 (Out)
- net OFFSET_W: now also R15.2, RV4.2 (Wiper); no longer C7_3.2 (Wiper), D5.2
- net SCALE_W: now also R14.2, RV3.2 (Wiper), RV3.3; no longer C7_8.2 (Wiper), C7_8.3, D4.2
- net U9_SPARE: now also U9.12 (In+), U9.14 (Out); no longer R16_1.12 (In+), R16_1.14 (Out)
- net VSRC_BP1_DIST: now also R37_8.1, RV13.1, R_INV_IN_8.2; no longer R37_10.1, RV15.1, R_INV_IN_10.2
- net VSRC_BP1_FREQ: now also R37_6.1, RV11.1, R_INV_IN_6.2; no longer R37_8.1, RV13.1, R_INV_IN_8.2
- net VSRC_BP2_DIST: now also R37_11.1, RV16.1, R_INV_IN_11.2; no longer R37_13.1, RV18.1, R_INV_IN_13.2
- net VSRC_BP2_FREQ: no longer R37_11.1, RV16.1, R_INV_IN_11.2
- net VSRC_BP3_DIST: now also R37_14.1, RV19.1, R_INV_IN_14.2; no longer R37_16.1, RV21.1, R_INV_IN_16.2
- net VSRC_BP3_FREQ: no longer R37_14.1, RV19.1, R_INV_IN_14.2
- net VSRC_BP_FREQ: now also R37_4.1, RV9.1, R_INV_IN_4.2; no longer R37_6.1, RV11.1, R_INV_IN_6.2
- net VSRC_BP_TILT: now also R37_5.1, RV10.1, R_INV_IN_5.2; no longer R37_7.1, RV12.1, R_INV_IN_7.2
- net VSRC_HP_FREQ: no longer R37_17.1, RV22.1, R_INV_IN_17.2
- net VSRC_HP_RES: now also R37_16.1, RV21.1, R_INV_IN_16.2; no longer R37_18.1, RV23.1, R_INV_IN_18.2
- net VSRC_LP1_FREQ: now also R37_1.1, RV6.1, R_INV_IN_1.2; no longer R37_3.1, RV8.1, R_INV_IN_3.2
- net VSRC_LP1_RES: now also R37_3.1, RV8.1, R_INV_IN_3.2; no longer R37_5.1, RV10.1, R_INV_IN_5.2
- net VSRC_LP1_TILT: now also R37_2.1, RV7.1, R_INV_IN_2.2; no longer R37_4.1, RV9.1, R_INV_IN_4.2
- net VSRC_LP2_FREQ: now also R37_17.1, RV22.1, R_INV_IN_17.2
- net VSRC_LP2_RES: now also R37_18.1, RV23.1, R_INV_IN_18.2
- net V_MODBUS: now also R16_2.1, R18_1.1, R18_2.1; no longer RV3.1, U5.2 (In-), U5.5 (In+), U5.9 (In-)
- net V_MODBUS_INV: now also D5.3 (K), R13.1, R16_1.2; no longer D6.2, R99.1, SW7.3 (K)
- net V_SRC: now also RV3.1, SW7.5 (B_COM); no longer C7_8.1, RV4.1
- net ZMID: now also D5.1 (A), D6.1 (A); no longer C7_1.1 (A), SW7.1 (A)
- removed net CLIP_OUT: C7_5.2, U5.8 (Out)
- removed net CLIP_REF: C7_12.1, C7_6.2, U5.10 (In+)
- removed net INVN_BP1_FOCUS: R_INV_FB_9.2, R_INV_IN_9.1, U7.10 (In+)
- removed net INVN_BP2_FOCUS: R_INV_FB_12.2, R_INV_IN_12.1, U8.5 (In+)
- removed net INVN_BP3_FOCUS: R_INV_FB_15.2, R_INV_IN_15.1, U9.3 (In+)
- removed net INVN_VCA_AMT: R15.10 (In+)
- removed net LEDA_CLIP: C7_14.K, C7_5.1
- removed net LEDA_NEG: C7_11.1, C7_7.K
- removed net LEDA_POS: C7_13.K, C7_4.1
- removed net NEG_OUT: C7_11.2, U5.7 (Out)
- removed net NVSRC_BP1_FOCUS: RV14.3, R_INV_FB_9.1, U7.8 (Out)
- removed net NVSRC_BP2_FOCUS: RV17.3, R_INV_FB_12.1, U8.7 (Out)
- removed net NVSRC_BP3_FOCUS: RV20.3, R_INV_FB_15.1, U9.1 (Out)
- removed net NVSRC_VCA_AMT: R15.8 (Out)
- removed net POS_OUT: C7_4.2, U5.1 (Out)
- removed net U4_SPARE: U5.12 (In+), U5.14 (Out)
- new net INVN_BP1_TILT: R_INV_FB_7.2, R_INV_IN_7.1, U6.10 (In+)
- new net INVN_BP2_TILT: R_INV_FB_10.2, R_INV_IN_10.1, U7.5 (In+)
- new net INVN_BP3_TILT: R_INV_FB_13.2, R_INV_IN_13.1, U8.3 (In+)
- new net JSW_BP1_TILT: R18_7.2
- new net JSW_BP2_TILT: R18_10.2
- new net JSW_BP3_TILT: R18_13.2
- new net JTIP_BP1_TILT: J14.1 (T), R37_7.2
- new net JTIP_BP2_TILT: J17.1 (T), R37_10.2
- new net JTIP_BP3_TILT: J20.1 (T), R37_13.2
- new net LFO2_OUT: SW7.3 (A2)
- new net MOD_BP1_TILT: RV12.2 (Wiper)
- new net MOD_BP2_TILT: RV15.2 (Wiper)
- new net MOD_BP3_TILT: RV18.2 (Wiper)
- new net MOD_IN_EXT: R99.1, SW7.1 (A1)
- new net NVSRC_BP1_TILT: RV12.3, R_INV_FB_7.1, U6.8 (Out)
- new net NVSRC_BP2_TILT: RV15.3, R_INV_FB_10.1, U7.7 (Out)
- new net NVSRC_BP3_TILT: RV18.3, R_INV_FB_13.1, U8.1 (Out)
- new net SW_AB_BRIDGE: SW7.2 (A_COM), SW7.4 (B1)
- new net U9_SPARE_C: U9.10 (In+), U9.8 (Out)
- new net VSRC_BP1_TILT: R37_7.1, RV12.1, R_INV_IN_7.2
- new net VSRC_BP2_TILT: R37_10.1, RV15.1, R_INV_IN_10.2
- new net VSRC_BP3_TILT: R37_13.1, RV18.1, R_INV_IN_13.2
Other:
- moved on the sheet: C7_1, D3_10, D3_11, D3_12, D3_13, D3_14, D3_15, D3_16, D3_17, D3_18, D3_3, D3_4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
