File: kicad/pogo-block-3.kicad_sch (KiCad schematic)
At the start: 157 parts, among them J10 LP1_RES, J11 BP_FREQ, J12 BP_TILT, J13 BP1_FREQ, J14 BP1_TILT, J15 BP1_DIST, J16 BP2_FREQ, J17 BP2_TILT, J18 BP2_DIST, J19 BP3_FREQ, J20 BP3_TILT, J21 BP3_DIST, J22 HP_FREQ, J23 HP_RES, J24 LP2_FREQ, J25 LP2_RES, J7 MOD_IN, J8 LP1_FREQ, J9 LP1_TILT, SW7 MOD_SRC, U3 TL074, U5 TL074, U6 TL074, U7 TL074, U8 TL074, U9 TL074

Commit message: 0020 §H: fix mod-bus depth + distribution buffer + offset range (C2/H2/M2)
block-3 mod-bus rewrite (SPICE-validated, user chose raise-impedance):
- C2 (depth): removed the 18x R18 R_SRC_NORM (100k); each jack switch lug now
  normals LOW-Z directly to V_MODBUS. SPICE: ~3% -> ~98% mod depth.
- H2 (drive): raised attenuverter network x5 (R_INV_IN/FB 10k->47k, pot ->50k)
  so 18-dest load drops to ~11mA; re-enabled U3 C/D as a paralleled unity
  distribution buffer (R227/R228 47R share Rs) driving the rail. Within 2x TL074.
- M2 (offset): R15 100k->240k so RV4's +-12V wiper maps to +-5V at the summer.
- Decks: specs/sim/modbus_depth.cir, modbus_load.cir, modbus_hiZ.cir.

block-3 schematic regenerated (141 parts/111 nets); all --check gates + JS/Py
parity green. V_MODBUS = 18 jack lugs + 2 share Rs; no R18 part remains.

https://claude.ai/code/session_013jFXG5oeMVSYP7iRpwGvtQ
Parts:
- removed D3_16, D3_17, D3_18: BAT54S, POGO_Package_TO_SOT_SMD:SOT-23, symbol Diode:BAT54S
- removed J24: LP2_FREQ, POGO_Connector_Audio:Jack_3.5mm_QingPu_WQP-PJ398SM_Vertical_CircularHoles, symbol Device:Audio_Jack_3.5mm_SwitchT
- removed J25: LP2_RES, POGO_Connector_Audio:Jack_3.5mm_QingPu_WQP-PJ398SM_Vertical_CircularHoles, symbol Device:Audio_Jack_3.5mm_SwitchT
- removed R18_16, R18_17, R18_18: 100k, symbol Device:R
- removed R37_17, R37_18: 100R, symbol Device:R
- removed RV22: LP2_FREQ_ATT, POGO_Potentiometer_THT:Potentiometer_Songhuei_9mm_TallTrimmer_Vertical, symbol Device:R_POT
- removed RV23: LP2_RES_ATT, POGO_Potentiometer_THT:Potentiometer_Songhuei_9mm_TallTrimmer_Vertical, symbol Device:R_POT
- removed R_INV_FB_17, R_INV_FB_18, R_INV_IN_17, R_INV_IN_18: 10k, symbol Device:R
- C7_14: renamed from R_INV_FB_1; value 10k -> 100nF; symbol Device:R -> Device:C
- C7_7: renamed from R_INV_IN_1; value 10k -> 100nF; symbol Device:R -> Device:C
- D3_1: renamed from R_INV_IN_2; value 10k -> BAT54S; footprint (none) -> POGO_Package_TO_SOT_SMD:SOT-23; symbol Device:R -> Diode:BAT54S
- D3_11: renamed from R37_10; value 100R -> BAT54S; footprint (none) -> POGO_Package_TO_SOT_SMD:SOT-23; symbol Device:R -> Diode:BAT54S
- D3_12: renamed from J18; value BP2_DIST -> BAT54S; footprint POGO_Connector_Audio:Jack_3.5mm_QingPu_WQP-PJ398SM_Vertical_CircularHoles -> POGO_Package_TO_SOT_SMD:SOT-23; symbol Device:Audio_Jack_3.5mm_SwitchT -> Diode:BAT54S
- D3_13: renamed from RV17; value BP3_FREQ_ATT -> BAT54S; footprint POGO_Potentiometer_THT:Potentiometer_Songhuei_9mm_TallTrimmer_Vertical -> POGO_Package_TO_SOT_SMD:SOT-23; symbol Device:R_POT -> Diode:BAT54S
- D3_14: renamed from R_INV_FB_13; value 10k -> BAT54S; footprint (none) -> POGO_Package_TO_SOT_SMD:SOT-23; symbol Device:R -> Diode:BAT54S
- D3_15: renamed from R_INV_IN_14; value 10k -> BAT54S; footprint (none) -> POGO_Package_TO_SOT_SMD:SOT-23; symbol Device:R -> Diode:BAT54S
- D3_16: renamed from R18_14; value 100k -> BAT54S; footprint (none) -> POGO_Package_TO_SOT_SMD:SOT-23; symbol Device:R -> Diode:BAT54S
- D3_18: renamed from R37_16; value 100R -> BAT54S; footprint (none) -> POGO_Package_TO_SOT_SMD:SOT-23; symbol Device:R -> Diode:BAT54S
- D3_2: renamed from R18_2; value 100k -> BAT54S; footprint (none) -> POGO_Package_TO_SOT_SMD:SOT-23; symbol Device:R -> Diode:BAT54S
- D3_4: renamed from R37_4; value 100R -> BAT54S; footprint (none) -> POGO_Package_TO_SOT_SMD:SOT-23; symbol Device:R -> Diode:BAT54S
- D3_5: renamed from J12; value BP_TILT -> BAT54S; footprint POGO_Connector_Audio:Jack_3.5mm_QingPu_WQP-PJ398SM_Vertical_CircularHoles -> POGO_Package_TO_SOT_SMD:SOT-23; symbol Device:Audio_Jack_3.5mm_SwitchT -> Diode:BAT54S
- D3_6: renamed from RV11; value BP1_FREQ_ATT -> BAT54S; footprint POGO_Potentiometer_THT:Potentiometer_Songhuei_9mm_TallTrimmer_Vertical -> POGO_Package_TO_SOT_SMD:SOT-23; symbol Device:R_POT -> Diode:BAT54S
- D3_7: renamed from R_INV_FB_7; value 10k -> BAT54S; footprint (none) -> POGO_Package_TO_SOT_SMD:SOT-23; symbol Device:R -> Diode:BAT54S
- D3_8: renamed from R_INV_IN_8; value 10k -> BAT54S; footprint (none) -> POGO_Package_TO_SOT_SMD:SOT-23; symbol Device:R -> Diode:BAT54S
- D3_9: renamed from R18_8; value 100k -> BAT54S; footprint (none) -> POGO_Package_TO_SOT_SMD:SOT-23; symbol Device:R -> Diode:BAT54S
- D4: renamed from D6; value BZX84C10 -> BAT54S; symbol Diode:D_Zener -> Diode:BAT54S
- D5: renamed from RV3; value MOD_SCALE -> BZX84C10; footprint POGO_Potentiometer_THT:Potentiometer_Songhuei_9mm_TallTrimmer_Vertical -> POGO_Package_TO_SOT_SMD:SOT-23; symbol Device:R_POT -> Diode:D_Zener
- D6: renamed from RV4; value MOD_OFFSET -> BZX84C10; footprint POGO_Potentiometer_THT:Potentiometer_Songhuei_9mm_TallTrimmer_Vertical -> POGO_Package_TO_SOT_SMD:SOT-23; symbol Device:R_POT -> Diode:D_Zener
- J11: renamed from RV9; value BP_FREQ_ATT -> BP_FREQ; footprint POGO_Potentiometer_THT:Potentiometer_Songhuei_9mm_TallTrimmer_Vertical -> POGO_Connector_Audio:Jack_3.5mm_QingPu_WQP-PJ398SM_Vertical_CircularHoles; symbol Device:R_POT -> Device:Audio_Jack_3.5mm_SwitchT
- J12: renamed from R_INV_FB_5; value 10k -> BP_TILT; footprint (none) -> POGO_Connector_Audio:Jack_3.5mm_QingPu_WQP-PJ398SM_Vertical_CircularHoles; symbol Device:R -> Device:Audio_Jack_3.5mm_SwitchT
- J13: renamed from R_INV_IN_6; value 10k -> BP1_FREQ; footprint (none) -> POGO_Connector_Audio:Jack_3.5mm_QingPu_WQP-PJ398SM_Vertical_CircularHoles; symbol Device:R -> Device:Audio_Jack_3.5mm_SwitchT
- J14: renamed from R18_6; value 100k -> BP1_TILT; footprint (none) -> POGO_Connector_Audio:Jack_3.5mm_QingPu_WQP-PJ398SM_Vertical_CircularHoles; symbol Device:R -> Device:Audio_Jack_3.5mm_SwitchT
- J15: renamed from D3_7; value BAT54S -> BP1_DIST; footprint POGO_Package_TO_SOT_SMD:SOT-23 -> POGO_Connector_Audio:Jack_3.5mm_QingPu_WQP-PJ398SM_Vertical_CircularHoles; symbol Diode:BAT54S -> Device:Audio_Jack_3.5mm_SwitchT
- J16: renamed from R37_8; value 100R -> BP2_FREQ; footprint (none) -> POGO_Connector_Audio:Jack_3.5mm_QingPu_WQP-PJ398SM_Vertical_CircularHoles; symbol Device:R -> Device:Audio_Jack_3.5mm_SwitchT
- J17: renamed from J16; value BP2_FREQ -> BP2_TILT
- J18: renamed from RV15; value BP2_TILT_ATT -> BP2_DIST; footprint POGO_Potentiometer_THT:Potentiometer_Songhuei_9mm_TallTrimmer_Vertical -> POGO_Connector_Audio:Jack_3.5mm_QingPu_WQP-PJ398SM_Vertical_CircularHoles; symbol Device:R_POT -> Device:Audio_Jack_3.5mm_SwitchT
- J19: renamed from R_INV_FB_11; value 10k -> BP3_FREQ; footprint (none) -> POGO_Connector_Audio:Jack_3.5mm_QingPu_WQP-PJ398SM_Vertical_CircularHoles; symbol Device:R -> Device:Audio_Jack_3.5mm_SwitchT
- J20: renamed from R_INV_IN_12; value 10k -> BP3_TILT; footprint (none) -> POGO_Connector_Audio:Jack_3.5mm_QingPu_WQP-PJ398SM_Vertical_CircularHoles; symbol Device:R -> Device:Audio_Jack_3.5mm_SwitchT
- J21: renamed from R18_12; value 100k -> BP3_DIST; footprint (none) -> POGO_Connector_Audio:Jack_3.5mm_QingPu_WQP-PJ398SM_Vertical_CircularHoles; symbol Device:R -> Device:Audio_Jack_3.5mm_SwitchT
- J22: renamed from D3_13; value BAT54S -> HP_FREQ; footprint POGO_Package_TO_SOT_SMD:SOT-23 -> POGO_Connector_Audio:Jack_3.5mm_QingPu_WQP-PJ398SM_Vertical_CircularHoles; symbol Diode:BAT54S -> Device:Audio_Jack_3.5mm_SwitchT
- J23: renamed from R37_14; value 100R -> HP_RES; footprint (none) -> POGO_Connector_Audio:Jack_3.5mm_QingPu_WQP-PJ398SM_Vertical_CircularHoles; symbol Device:R -> Device:Audio_Jack_3.5mm_SwitchT
- J24: renamed from J22; value HP_FREQ -> LP2_FREQ
- J25: renamed from RV21; value HP_RES_ATT -> LP2_RES; footprint POGO_Potentiometer_THT:Potentiometer_Songhuei_9mm_TallTrimmer_Vertical -> POGO_Connector_Audio:Jack_3.5mm_QingPu_WQP-PJ398SM_Vertical_CircularHoles; symbol Device:R_POT -> Device:Audio_Jack_3.5mm_SwitchT
- J7: renamed from C7_1; value 100nF -> MOD_IN; footprint (none) -> POGO_Connector_Audio:Jack_3.5mm_QingPu_WQP-PJ398SM_Vertical_CircularHoles; symbol Device:C -> Device:Audio_Jack_3.5mm_SwitchT
- J8: renamed from D3_1; value BAT54S -> LP1_FREQ; footprint POGO_Package_TO_SOT_SMD:SOT-23 -> POGO_Connector_Audio:Jack_3.5mm_QingPu_WQP-PJ398SM_Vertical_CircularHoles; symbol Diode:BAT54S -> Device:Audio_Jack_3.5mm_SwitchT
- J9: renamed from R37_2; value 100R -> LP1_TILT; footprint (none) -> POGO_Connector_Audio:Jack_3.5mm_QingPu_WQP-PJ398SM_Vertical_CircularHoles; symbol Device:R -> Device:Audio_Jack_3.5mm_SwitchT
- R15: value 100k -> 240k
- R227: renamed from R99; value 100R -> 47R
- R228: renamed from D4; value BAT54S -> 47R; footprint POGO_Package_TO_SOT_SMD:SOT-23 -> (none); symbol Diode:BAT54S -> Device:R
- R37_1: renamed from R18_1; value 100k -> 100R
- R37_11: renamed from J17; value BP2_TILT -> 100R; footprint POGO_Connector_Audio:Jack_3.5mm_QingPu_WQP-PJ398SM_Vertical_CircularHoles -> (none); symbol Device:Audio_Jack_3.5mm_SwitchT -> Device:R
- R37_12: renamed from RV16; value BP2_DIST_ATT -> 100R; footprint POGO_Potentiometer_THT:Potentiometer_Songhuei_9mm_TallTrimmer_Vertical -> (none); symbol Device:R_POT -> Device:R
- R37_13: renamed from R_INV_FB_12; value 10k -> 100R
- R37_14: renamed from R_INV_IN_13; value 10k -> 100R
- R37_15: renamed from R18_13; value 100k -> 100R
- R37_16: renamed from D3_14; value BAT54S -> 100R; footprint POGO_Package_TO_SOT_SMD:SOT-23 -> (none); symbol Diode:BAT54S -> Device:R
- R37_18: renamed from J23; value HP_RES -> 100R; footprint POGO_Connector_Audio:Jack_3.5mm_QingPu_WQP-PJ398SM_Vertical_CircularHoles -> (none); symbol Device:Audio_Jack_3.5mm_SwitchT -> Device:R
- R37_2: renamed from D3_2; value BAT54S -> 100R; footprint POGO_Package_TO_SOT_SMD:SOT-23 -> (none); symbol Diode:BAT54S -> Device:R
- R37_4: renamed from J11; value BP_FREQ -> 100R; footprint POGO_Connector_Audio:Jack_3.5mm_QingPu_WQP-PJ398SM_Vertical_CircularHoles -> (none); symbol Device:Audio_Jack_3.5mm_SwitchT -> Device:R
- R37_5: renamed from RV10; value BP_TILT_ATT -> 100R; footprint POGO_Potentiometer_THT:Potentiometer_Songhuei_9mm_TallTrimmer_Vertical -> (none); symbol Device:R_POT -> Device:R
- R37_6: renamed from R_INV_FB_6; value 10k -> 100R
- R37_7: renamed from R_INV_IN_7; value 10k -> 100R
- R37_8: renamed from R18_7; value 100k -> 100R
- R37_9: renamed from D3_8; value BAT54S -> 100R; footprint POGO_Package_TO_SOT_SMD:SOT-23 -> (none); symbol Diode:BAT54S -> Device:R
- R99: renamed from D5; value BZX84C10 -> 100R; footprint POGO_Package_TO_SOT_SMD:SOT-23 -> (none); symbol Diode:D_Zener -> Device:R
- RV10: renamed from R_INV_IN_5; value 10k -> BP_TILT_ATT; footprint (none) -> POGO_Potentiometer_THT:Potentiometer_Songhuei_9mm_TallTrimmer_Vertical; symbol Device:R -> Device:R_POT
- RV11: renamed from R18_5; value 100k -> BP1_FREQ_ATT; footprint (none) -> POGO_Potentiometer_THT:Potentiometer_Songhuei_9mm_TallTrimmer_Vertical; symbol Device:R -> Device:R_POT
- RV12: renamed from D3_6; value BAT54S -> BP1_TILT_ATT; footprint POGO_Package_TO_SOT_SMD:SOT-23 -> POGO_Potentiometer_THT:Potentiometer_Songhuei_9mm_TallTrimmer_Vertical; symbol Diode:BAT54S -> Device:R_POT
- RV13: renamed from R37_7; value 100R -> BP1_DIST_ATT; footprint (none) -> POGO_Potentiometer_THT:Potentiometer_Songhuei_9mm_TallTrimmer_Vertical; symbol Device:R -> Device:R_POT
- RV14: renamed from J15; value BP1_DIST -> BP2_FREQ_ATT; footprint POGO_Connector_Audio:Jack_3.5mm_QingPu_WQP-PJ398SM_Vertical_CircularHoles -> POGO_Potentiometer_THT:Potentiometer_Songhuei_9mm_TallTrimmer_Vertical; symbol Device:Audio_Jack_3.5mm_SwitchT -> Device:R_POT
- RV15: renamed from RV14; value BP2_FREQ_ATT -> BP2_TILT_ATT
- RV16: renamed from R_INV_FB_10; value 10k -> BP2_DIST_ATT; footprint (none) -> POGO_Potentiometer_THT:Potentiometer_Songhuei_9mm_TallTrimmer_Vertical; symbol Device:R -> Device:R_POT
- RV17: renamed from R_INV_IN_11; value 10k -> BP3_FREQ_ATT; footprint (none) -> POGO_Potentiometer_THT:Potentiometer_Songhuei_9mm_TallTrimmer_Vertical; symbol Device:R -> Device:R_POT
- RV18: renamed from R18_11; value 100k -> BP3_TILT_ATT; footprint (none) -> POGO_Potentiometer_THT:Potentiometer_Songhuei_9mm_TallTrimmer_Vertical; symbol Device:R -> Device:R_POT
- RV19: renamed from D3_12; value BAT54S -> BP3_DIST_ATT; footprint POGO_Package_TO_SOT_SMD:SOT-23 -> POGO_Potentiometer_THT:Potentiometer_Songhuei_9mm_TallTrimmer_Vertical; symbol Diode:BAT54S -> Device:R_POT
- RV20: renamed from R37_13; value 100R -> HP_FREQ_ATT; footprint (none) -> POGO_Potentiometer_THT:Potentiometer_Songhuei_9mm_TallTrimmer_Vertical; symbol Device:R -> Device:R_POT
- RV21: renamed from J21; value BP3_DIST -> HP_RES_ATT; footprint POGO_Connector_Audio:Jack_3.5mm_QingPu_WQP-PJ398SM_Vertical_CircularHoles -> POGO_Potentiometer_THT:Potentiometer_Songhuei_9mm_TallTrimmer_Vertical; symbol Device:Audio_Jack_3.5mm_SwitchT -> Device:R_POT
- RV22: renamed from RV20; value HP_FREQ_ATT -> LP2_FREQ_ATT
- RV23: renamed from R_INV_FB_16; value 10k -> LP2_RES_ATT; footprint (none) -> POGO_Potentiometer_THT:Potentiometer_Songhuei_9mm_TallTrimmer_Vertical; symbol Device:R -> Device:R_POT
- RV3: renamed from J7; value MOD_IN -> MOD_SCALE; footprint POGO_Connector_Audio:Jack_3.5mm_QingPu_WQP-PJ398SM_Vertical_CircularHoles -> POGO_Potentiometer_THT:Potentiometer_Songhuei_9mm_TallTrimmer_Vertical; symbol Device:Audio_Jack_3.5mm_SwitchT -> Device:R_POT
- RV4: renamed from SW7; value MOD_SRC -> MOD_OFFSET; footprint (none) -> POGO_Potentiometer_THT:Potentiometer_Songhuei_9mm_TallTrimmer_Vertical; symbol Switch:SW_Dailywell_DW5 -> Device:R_POT
- RV6: renamed from R37_1; value 100R -> LP1_FREQ_ATT; footprint (none) -> POGO_Potentiometer_THT:Potentiometer_Songhuei_9mm_TallTrimmer_Vertical; symbol Device:R -> Device:R_POT
- RV7: renamed from J9; value LP1_TILT -> LP1_TILT_ATT; footprint POGO_Connector_Audio:Jack_3.5mm_QingPu_WQP-PJ398SM_Vertical_CircularHoles -> POGO_Potentiometer_THT:Potentiometer_Songhuei_9mm_TallTrimmer_Vertical; symbol Device:Audio_Jack_3.5mm_SwitchT -> Device:R_POT
- RV9: renamed from R_INV_FB_4; value 10k -> BP_FREQ_ATT; footprint (none) -> POGO_Potentiometer_THT:Potentiometer_Songhuei_9mm_TallTrimmer_Vertical; symbol Device:R -> Device:R_POT
- R_INV_FB_1: renamed from J8; value LP1_FREQ -> 47k; footprint POGO_Connector_Audio:Jack_3.5mm_QingPu_WQP-PJ398SM_Vertical_CircularHoles -> (none); symbol Device:Audio_Jack_3.5mm_SwitchT -> Device:R
- R_INV_FB_10: renamed from R_INV_FB_9; value 10k -> 47k
- R_INV_FB_11: renamed from R_INV_IN_10; value 10k -> 47k
- R_INV_FB_12: renamed from R18_10; value 100k -> 47k
- R_INV_FB_13: renamed from D3_11; value BAT54S -> 47k; footprint POGO_Package_TO_SOT_SMD:SOT-23 -> (none); symbol Diode:BAT54S -> Device:R
- R_INV_FB_14: renamed from R37_12; value 100R -> 47k
- R_INV_FB_15: renamed from J20; value BP3_TILT -> 47k; footprint POGO_Connector_Audio:Jack_3.5mm_QingPu_WQP-PJ398SM_Vertical_CircularHoles -> (none); symbol Device:Audio_Jack_3.5mm_SwitchT -> Device:R
- R_INV_FB_16: renamed from RV19; value BP3_DIST_ATT -> 47k; footprint POGO_Potentiometer_THT:Potentiometer_Songhuei_9mm_TallTrimmer_Vertical -> (none); symbol Device:R_POT -> Device:R
- R_INV_FB_17: renamed from R_INV_FB_15; value 10k -> 47k
- R_INV_FB_18: renamed from R_INV_IN_16; value 10k -> 47k
- R_INV_FB_2: renamed from RV7; value LP1_TILT_ATT -> 47k; footprint POGO_Potentiometer_THT:Potentiometer_Songhuei_9mm_TallTrimmer_Vertical -> (none); symbol Device:R_POT -> Device:R
- R_INV_FB_3, R_INV_IN_3: value 10k -> 47k
- R_INV_FB_4: renamed from R_INV_IN_4; value 10k -> 47k
- R_INV_FB_5: renamed from R18_4; value 100k -> 47k
- R_INV_FB_6: renamed from D3_5; value BAT54S -> 47k; footprint POGO_Package_TO_SOT_SMD:SOT-23 -> (none); symbol Diode:BAT54S -> Device:R
- R_INV_FB_7: renamed from R37_6; value 100R -> 47k
- R_INV_FB_8: renamed from J14; value BP1_TILT -> 47k; footprint POGO_Connector_Audio:Jack_3.5mm_QingPu_WQP-PJ398SM_Vertical_CircularHoles -> (none); symbol Device:Audio_Jack_3.5mm_SwitchT -> Device:R
- R_INV_FB_9: renamed from RV13; value BP1_DIST_ATT -> 47k; footprint POGO_Potentiometer_THT:Potentiometer_Songhuei_9mm_TallTrimmer_Vertical -> (none); symbol Device:R_POT -> Device:R
- R_INV_IN_1: renamed from RV6; value LP1_FREQ_ATT -> 47k; footprint POGO_Potentiometer_THT:Potentiometer_Songhuei_9mm_TallTrimmer_Vertical -> (none); symbol Device:R_POT -> Device:R
- R_INV_IN_10: renamed from R_INV_IN_9; value 10k -> 47k
- R_INV_IN_11: renamed from R18_9; value 100k -> 47k
- R_INV_IN_12: renamed from D3_10; value BAT54S -> 47k; footprint POGO_Package_TO_SOT_SMD:SOT-23 -> (none); symbol Diode:BAT54S -> Device:R
- R_INV_IN_13: renamed from R37_11; value 100R -> 47k
- R_INV_IN_14: renamed from J19; value BP3_FREQ -> 47k; footprint POGO_Connector_Audio:Jack_3.5mm_QingPu_WQP-PJ398SM_Vertical_CircularHoles -> (none); symbol Device:Audio_Jack_3.5mm_SwitchT -> Device:R
- R_INV_IN_15: renamed from RV18; value BP3_TILT_ATT -> 47k; footprint POGO_Potentiometer_THT:Potentiometer_Songhuei_9mm_TallTrimmer_Vertical -> (none); symbol Device:R_POT -> Device:R
- R_INV_IN_16: renamed from R_INV_FB_14; value 10k -> 47k
- R_INV_IN_17: renamed from R_INV_IN_15; value 10k -> 47k
- R_INV_IN_18: renamed from R18_15; value 100k -> 47k
- R_INV_IN_2: renamed from R_INV_FB_2; value 10k -> 47k
- R_INV_IN_4: renamed from R18_3; value 100k -> 47k
- R_INV_IN_5: renamed from D3_4; value BAT54S -> 47k; footprint POGO_Package_TO_SOT_SMD:SOT-23 -> (none); symbol Diode:BAT54S -> Device:R
- R_INV_IN_6: renamed from R37_5; value 100R -> 47k
- R_INV_IN_7: renamed from J13; value BP1_FREQ -> 47k; footprint POGO_Connector_Audio:Jack_3.5mm_QingPu_WQP-PJ398SM_Vertical_CircularHoles -> (none); symbol Device:Audio_Jack_3.5mm_SwitchT -> Device:R
- R_INV_IN_8: renamed from RV12; value BP1_TILT_ATT -> 47k; footprint POGO_Potentiometer_THT:Potentiometer_Songhuei_9mm_TallTrimmer_Vertical -> (none); symbol Device:R_POT -> Device:R
- R_INV_IN_9: renamed from R_INV_FB_8; value 10k -> 47k
- SW7: renamed from C7_8; value 100nF -> MOD_SRC; symbol Device:C -> Switch:SW_Dailywell_DW5
- renumbered C7_3 to C7_1, C7_11 to C7_10, C7_12 to C7_11, C7_13 to C7_12, C7_14 to C7_13, C7_4 to C7_3, C7_5 to C7_4, C7_6 to C7_5, C7_7 to C7_6, C7_10 to C7_8, D3_9 to D3_10, D3_15 to D3_17, R37_9 to R37_10, R37_15 to R37_17
Connections:
- net JSW_BP1_DIST is gone; now on net +12V: D3_9.2 (K2)
- net JSW_BP1_FREQ is gone; now on net GND: J14.2 (S)
- net JSW_BP1_TILT is gone; now on net JTIP_BP1_DIST: R37_8.2
- net JSW_BP2_DIST is gone; now on net MOD_BP3_TILT: RV18.2 (Wiper)
- net JSW_BP2_FREQ is gone; now on net VSRC_BP2_DIST: R_INV_IN_11.2
- net JSW_BP2_TILT is gone; now on net INVN_BP3_FREQ: R_INV_FB_12.2
- net JSW_BP3_DIST is gone; now on net +12V: D3_16.2 (K2)
- net JSW_BP3_FREQ is gone; now on net GND: J21.2 (S)
- net JSW_BP3_TILT is gone; now on net JTIP_HP_FREQ: R37_15.2
- net JSW_BP_FREQ is gone; now on net INVN_BP_TILT: R_INV_FB_5.2
- net JSW_BP_TILT is gone; now on net MOD_BP1_FREQ: RV11.2 (Wiper)
- net JSW_HP_FREQ is gone; now on net VSRC_LP2_RES: R_INV_IN_18.2
- net JSW_LP1_FREQ is gone; now on net JTIP_LP1_FREQ: R37_1.2
- net JSW_LP1_RES is gone; now on net VSRC_BP_FREQ: R_INV_IN_4.2
- net JSW_LP1_TILT is gone; now on net +12V: D3_2.2 (K2)
- net +12V: now also C7_7.2, D3_1.2 (K2), D3_11.2 (K2), D3_12.2 (K2), D3_13.2 (K2), D3_14.2 (K2), D3_15.2 (K2), D3_18.2 (K2), D3_4.2 (K2), D3_5.2 (K2), D3_6.2 (K2), D3_7.2 (K2), D3_8.2 (K2), D4.2 (K2), RV4.1; no longer D6.1, J15.2 (K2), J22.2 (K2), J7.2, J8.2 (K2), R228.2 (K2), R37_16.2 (K2), R37_2.2 (K2), R37_9.2 (K2), RV12.2 (K2), RV19.2 (K2), R_INV_FB_13.2 (K2), R_INV_FB_6.2 (K2), R_INV_IN_12.2 (K2), R_INV_IN_5.2 (K2)
- net -12V: now also C7_14.2, D3_1.1 (A1), D3_11.1 (A1), D3_12.1 (A1), D3_13.1 (A1), D3_14.1 (A1), D3_15.1 (A1), D3_16.1 (A1), D3_18.1 (A1), D3_2.1 (A1), D3_4.1 (A1), D3_5.1 (A1), D3_6.1 (A1), D3_7.1 (A1), D3_8.1 (A1), D3_9.1 (A1), D4.1 (A1), RV4.3; no longer D6.3, J15.1 (A1), J22.1 (A1), J8.1 (A1), R228.1 (A1), R37_16.1 (A1), R37_2.1 (A1), R37_9.1 (A1), RV12.1 (A1), RV19.1 (A1), R_INV_FB_13.1 (A1), R_INV_FB_6.1 (A1), R_INV_IN_12.1 (A1), R_INV_IN_5.1 (A1), SW7.2
- net GND: now also C7_14.1, C7_7.1, D6.3 (K), J11.2 (S), J12.2 (S), J13.2 (S), J15.2 (S), J16.2 (S), J18.2 (S), J19.2 (S), J20.2 (S), J22.2 (S), J23.2 (S), J25.2 (S), J7.2 (S), J8.2 (S), J9.2 (S); no longer D3_12.2 (S), D3_5.2 (S), D4.3 (K), J7.1, R37_11.2 (S), R37_18.2 (S), R37_4.2 (S), RV14.2 (S), RV21.2 (S), RV3.2 (S), RV7.2 (S), R_INV_FB_1.2 (S), R_INV_FB_15.2 (S), R_INV_FB_8.2 (S), R_INV_IN_14.2 (S), R_INV_IN_7.2 (S), SW7.1, U3.13 (In-), U3.9 (In-)
- net INVN_BP1_DIST: now also R_INV_FB_8.2, R_INV_IN_8.1; no longer D3_8.1, R_INV_IN_9.2
- net INVN_BP1_FREQ: now also R_INV_FB_6.2, R_INV_IN_6.1; no longer J13.1, R37_6.2
- net INVN_BP1_TILT: now also R_INV_FB_7.2, R_INV_IN_7.1; no longer D3_7.2, R37_7.1
- net INVN_BP2_DIST: now also R_INV_FB_11.2, R_INV_IN_11.1; no longer J19.2, RV17.1
- net INVN_BP2_FREQ: now also R_INV_FB_9.2, R_INV_IN_9.1; no longer R_INV_FB_10.2, R_INV_IN_10.1
- net INVN_BP2_TILT: now also R_INV_FB_10.2, R_INV_IN_10.1; no longer RV16.2, R_INV_FB_11.1
- net INVN_BP3_DIST: now also R_INV_FB_14.2, R_INV_IN_14.1; no longer D3_15.1, R_INV_IN_16.2
- net INVN_BP3_FREQ: now also R_INV_IN_12.1; no longer J20.1, R37_13.2
- net INVN_BP3_TILT: now also R_INV_FB_13.2, R_INV_IN_13.1; no longer D3_14.2, R37_14.1
- net INVN_BP_FREQ: now also R_INV_FB_4.2, R_INV_IN_4.1; no longer RV9.2, R_INV_FB_4.1
- net INVN_BP_TILT: now also R_INV_IN_5.1; no longer J12.2, RV10.1
- net INVN_HP_FREQ: now also R_INV_FB_15.2, R_INV_IN_15.1; no longer R_INV_FB_17.2, R_INV_IN_17.1
- net INVN_HP_RES: now also R_INV_FB_16.2, R_INV_IN_16.1; no longer RV23.2, R_INV_FB_18.1
- net INVN_LP1_FREQ: now also R_INV_FB_1.2, R_INV_IN_1.1; no longer C7_14.2, C7_7.1
- net INVN_LP1_TILT: now also R_INV_FB_2.2, R_INV_IN_2.1; no longer D3_1.1, R_INV_IN_2.2
- net INVN_LP2_FREQ: now also R_INV_FB_17.2, R_INV_IN_17.1
- net INVN_LP2_RES: now also R_INV_FB_18.2, R_INV_IN_18.1
- net JTIP_BP1_DIST: now also J15.1 (T); no longer J16.2, RV14.1 (T)
- net JTIP_BP1_FREQ: now also J13.1 (T), R37_6.2; no longer R_INV_FB_7.2, R_INV_IN_7.1 (T)
- net JTIP_BP1_TILT: now also J14.1 (T), R37_7.2; no longer RV13.2, R_INV_FB_8.1 (T)
- net JTIP_BP2_DIST: now also J18.1 (T), R37_11.2; no longer D3_12.1 (T), R_INV_IN_13.2
- net JTIP_BP2_FREQ: now also J16.1 (T), R37_9.2; no longer J17.1 (T), R37_10.2
- net JTIP_BP2_TILT: now also J17.1 (T), R37_10.2; no longer D3_11.2, R37_11.1 (T)
- net JTIP_BP3_DIST: now also J21.1 (T), R37_14.2; no longer J23.2, RV21.1 (T)
- net JTIP_BP3_FREQ: now also J19.1 (T), R37_12.2; no longer R_INV_FB_14.2, R_INV_IN_14.1 (T)
- net JTIP_BP3_TILT: now also J20.1 (T), R37_13.2; no longer RV20.2, R_INV_FB_15.1 (T)
- net JTIP_BP_FREQ: now also J11.1 (T), R37_4.2; no longer D3_4.2, R37_4.1 (T)
- net JTIP_BP_TILT: now also J12.1 (T), R37_5.2; no longer D3_5.1 (T), R_INV_IN_6.2
- net JTIP_HP_FREQ: now also J22.1 (T); no longer J24.1 (T), R37_17.2
- net JTIP_HP_RES: now also J23.1 (T), R37_16.2; no longer D3_18.2, R37_18.1 (T)
- net JTIP_LP1_FREQ: now also J8.1 (T); no longer RV6.2, R_INV_FB_1.1 (T)
- net JTIP_LP1_TILT: now also J9.1 (T), R37_2.2; no longer J9.2, RV7.1 (T)
- net JTIP_LP2_FREQ: now also J24.1 (T), R37_17.2
- net JTIP_LP2_RES: now also J25.1 (T), R37_18.2
- net LFO1_OUT: now also SW7.6 (B2); no longer RV4.6 (B2)
- net LFO2_OUT: now also SW7.3 (A2); no longer RV4.3 (A2)
- net MOD_BP1_DIST: now also RV13.2 (Wiper); no longer R_INV_FB_9.2 (Wiper)
- net MOD_BP1_FREQ: no longer D3_6.2 (Wiper)
- net MOD_BP1_TILT: now also RV12.2 (Wiper); no longer R_INV_IN_8.2 (Wiper)
- net MOD_BP2_DIST: now also RV16.2 (Wiper); no longer R37_12.2 (Wiper)
- net MOD_BP2_FREQ: now also RV14.2 (Wiper); no longer RV15.2 (Wiper)
- net MOD_BP2_TILT: now also RV15.2 (Wiper); no longer J18.2 (Wiper)
- net MOD_BP3_DIST: now also RV19.2 (Wiper); no longer R_INV_FB_16.2 (Wiper)
- net MOD_BP3_FREQ: now also RV17.2 (Wiper); no longer D3_13.2 (Wiper)
- net MOD_BP3_TILT: no longer R_INV_IN_15.2 (Wiper)
- net MOD_BP_FREQ: now also RV9.2 (Wiper); no longer J11.2 (Wiper)
- net MOD_BP_TILT: now also RV10.2 (Wiper); no longer R37_5.2 (Wiper)
- net MOD_HP_FREQ: now also RV20.2 (Wiper); no longer RV22.2 (Wiper)
- net MOD_HP_RES: now also RV21.2 (Wiper); no longer J25.2 (Wiper)
- net MOD_IN_EXT: now also R99.1, SW7.1 (A1); no longer R227.1, RV4.1 (A1)
- net MOD_IN_TIP: now also J7.1 (T), R99.2; no longer R227.2, RV3.1 (T)
- net MOD_LP1_FREQ: now also RV6.2 (Wiper); no longer R_INV_IN_1.2 (Wiper)
- net MOD_LP1_TILT: now also RV7.2 (Wiper); no longer R_INV_FB_2.2 (Wiper)
- net MOD_LP2_FREQ: now also RV22.2 (Wiper)
- net MOD_LP2_RES: now also RV23.2 (Wiper)
- net NVSRC_BP1_DIST: now also RV13.3, R_INV_FB_8.1; no longer R_INV_FB_9.3, R_INV_IN_9.1
- net NVSRC_BP1_FREQ: now also RV11.3, R_INV_FB_6.1; no longer D3_6.3, R37_6.1
- net NVSRC_BP1_TILT: now also RV12.3, R_INV_FB_7.1; no longer D3_7.1, R_INV_IN_8.3
- net NVSRC_BP2_DIST: now also RV16.3, R_INV_FB_11.1; no longer J19.1, R37_12.3
- net NVSRC_BP2_FREQ: now also RV14.3, R_INV_FB_9.1; no longer RV15.3, R_INV_FB_10.1
- net NVSRC_BP2_TILT: now also RV15.3, R_INV_FB_10.1; no longer J18.3, RV16.1
- net NVSRC_BP3_DIST: now also RV19.3, R_INV_FB_14.1; no longer R_INV_FB_16.3, R_INV_IN_16.1
- net NVSRC_BP3_FREQ: now also RV17.3, R_INV_FB_12.1; no longer D3_13.3, R37_13.1
- net NVSRC_BP3_TILT: now also RV18.3, R_INV_FB_13.1; no longer D3_14.1, R_INV_IN_15.3
- net NVSRC_BP_FREQ: now also RV9.3, R_INV_FB_4.1; no longer J11.3, RV9.1
- net NVSRC_BP_TILT: now also RV10.3, R_INV_FB_5.1; no longer J12.1, R37_5.3
- net NVSRC_HP_FREQ: now also RV20.3, R_INV_FB_15.1; no longer RV22.3, R_INV_FB_17.1
- net NVSRC_HP_RES: now also RV21.3, R_INV_FB_16.1; no longer J25.3, RV23.1
- net NVSRC_LP1_FREQ: now also RV6.3, R_INV_FB_1.1; no longer C7_14.1, R_INV_IN_1.3
- net NVSRC_LP1_TILT: now also RV7.3, R_INV_FB_2.1; no longer R_INV_FB_2.3, R_INV_IN_2.1
- net NVSRC_LP2_FREQ: now also RV22.3, R_INV_FB_17.1
- net NVSRC_LP2_RES: now also RV23.3, R_INV_FB_18.1
- net OFFSET_W: now also RV4.2 (Wiper); no longer D6.2 (Wiper)
- net SCALE_W: now also RV3.2 (Wiper), RV3.3; no longer D5.2 (Wiper), D5.3
- net SW_AB_BRIDGE: now also SW7.2 (A_COM), SW7.4 (B1); no longer RV4.2 (A_COM), RV4.4 (B1)
- net VSRC_BP1_DIST: now also R37_8.1, RV13.1, R_INV_IN_8.2; no longer D3_8.2, J16.1, R_INV_FB_9.1
- net VSRC_BP1_FREQ: now also R37_6.1, RV11.1, R_INV_IN_6.2; no longer D3_6.1, J13.2, R_INV_FB_7.1
- net VSRC_BP1_TILT: now also R37_7.1, RV12.1, R_INV_IN_7.2; no longer R37_7.2, RV13.1, R_INV_IN_8.1
- net VSRC_BP2_DIST: now also R37_11.1, RV16.1; no longer R37_12.1, RV17.2, R_INV_IN_13.1
- net VSRC_BP2_FREQ: now also R37_9.1, RV14.1, R_INV_IN_9.2; no longer R37_10.1, RV15.1, R_INV_IN_10.2
- net VSRC_BP2_TILT: now also R37_10.1, RV15.1, R_INV_IN_10.2; no longer D3_11.1, J18.1, R_INV_FB_11.2
- net VSRC_BP3_DIST: now also R37_14.1, RV19.1, R_INV_IN_14.2; no longer D3_15.2, J23.1, R_INV_FB_16.1
- net VSRC_BP3_FREQ: now also R37_12.1, RV17.1, R_INV_IN_12.2; no longer D3_13.1, J20.2, R_INV_FB_14.1
- net VSRC_BP3_TILT: now also R37_13.1, RV18.1, R_INV_IN_13.2; no longer R37_14.2, RV20.1, R_INV_IN_15.1
- net VSRC_BP_FREQ: now also R37_4.1, RV9.1; no longer D3_4.1, J11.1, R_INV_FB_4.2
- net VSRC_BP_TILT: now also RV10.1, R_INV_IN_5.2; no longer RV10.2, R_INV_IN_6.1
- net VSRC_HP_FREQ: now also R37_15.1, RV20.1, R_INV_IN_15.2; no longer R37_17.1, RV22.1, R_INV_IN_17.2
- net VSRC_HP_RES: now also R37_16.1, RV21.1, R_INV_IN_16.2; no longer D3_18.1, J25.1, R_INV_FB_18.2
- net VSRC_LP1_FREQ: now also R37_1.1, R_INV_IN_1.2; no longer C7_7.2, R_INV_IN_1.1
- net VSRC_LP1_TILT: now also R37_2.1, RV7.1, R_INV_IN_2.2; no longer D3_1.2, J9.1, R_INV_FB_2.1
- net VSRC_LP2_FREQ: now also R37_17.1, RV22.1, R_INV_IN_17.2
- net VSRC_LP2_RES: now also R37_18.1, RV23.1
- net V_MODBUS: now also R227.1, R228.1; no longer D3_16.1, D3_2.1, D3_9.1, J14.1, J21.1, R16_2.1, R37_1.1, R37_15.1, R37_8.1, RV11.1, RV18.1, R_INV_FB_12.1, R_INV_FB_5.1, R_INV_IN_11.1, R_INV_IN_18.1, R_INV_IN_4.1, U3.7 (Out)
- net V_MODBUS_INV: now also D5.3 (K); no longer R99.3 (K)
- net V_SRC: now also RV3.1, SW7.5 (B_COM); no longer D5.1, RV4.5 (B_COM)
- net ZMID: now also D5.1 (A), D6.1 (A); no longer D4.1 (A), R99.1 (A)
- net U3_SPARE_3 renamed BUF_C_OUT
- net BUF_C_OUT: now also R227.2
- net U3_SPARE_4 renamed BUF_D_OUT
- net BUF_D_OUT: now also R228.2
- new net V_MODBUS_RAW: R16_2.1, U3.13 (In-), U3.7 (Out), U3.9 (In-)
