File: kicad/pogo-block-7.kicad_sch (KiCad schematic)
At the start: 67 parts, among them U49 LM13700, U50 LM13700, U51 LM13700, U52 LM13700, U53 OPA1612, U54 OPA1612, U55 THAT340, U66 TL072

Commit message: 0018: block-7 HP filter aligned to plugin (polarity bug fix + Q collapse)
Adversarial review found a real behavioral divergence: HP output had a
spurious G=-1 inverting buffer on the SUM_AMP node, double-inverting vs the
plugin (HPFilter pre-negates so the SUM_AMP node IS the HP tap). Fixed:
- Convert U53/U54 half-B from inverting buffer to a UNITY NON-INVERTING
  FOLLOWER on the SUM_AMP node (mirrors LP1's LP buffer); HP_OUT now matches
  the plugin polarity. R100-R103 removed.
- Collapse HP Q from 2 LM13700 (U51/U52, cell-A each) to ONE (U51 cell A=L,
  cell B=R), matching the LP1/LP2 shared-Q precedent. U52 + C97/C98 +
  R_QB_* spare-termination removed.
- RV18 (Q_max) value set to 100k.
- Lifted STALE §2/§3 banners; corrected aux-ota-c-svf's wrong HP-polarity
  algebra + ASCII, THAT340 SOIC-8->SOIC-14 in aux-expo-converter, and the
  aux-q-control HP IC note + Used-By board names.
- Confirmed faithful (= LP1): RES CV /10 (knob-domain), mono shared-expo
  cutoff, self-oscillation, 632Hz V/oct, raw FREQ CV.

All 5 --check gates + parity green; HP_OUT->block-8 boundary intact.

https://claude.ai/code/session_013jFXG5oeMVSYP7iRpwGvtQ
Parts:
- removed C100, C101, C102, C103, C104, C105, C106, C96, C97, C98, C99: 100nF, symbol Device:C
- C100: renamed from C89; value 10nF -> 100nF
- C101: renamed from C90; value 10nF -> 100nF
- C29A: renamed from U55; value THAT340 -> 47nF; footprint POGO_Package_SO:SOIC-14_3.9x8.7mm_P1.27mm -> (none); symbol POGO:THAT340 -> Device:C
- C86: renamed from R115; value 10k -> 100nF; symbol Device:R -> Device:C
- C87: renamed from R_QB_IABC_L; value 100k -> 10nF; symbol Device:R -> Device:C
- C88: renamed from R_QB_IABC_R; value 100k -> 10nF; symbol Device:R -> Device:C
- C89: renamed from R_QB_OUT_L; value 1k -> 10nF; symbol Device:R -> Device:C
- C90: renamed from R_QB_OUT_R; value 1k -> 10nF; symbol Device:R -> Device:C
- C91: renamed from RV16; value HP_FREF -> 100nF; footprint POGO_Potentiometer_SMD:Potentiometer_Bourns_3224W -> (none); symbol Device:R_POT -> Device:C
- C92: renamed from RV17; value HP_1VOCT -> 100nF; footprint POGO_Potentiometer_SMD:Potentiometer_Bourns_3224W -> (none); symbol Device:R_POT -> Device:C
- C93: renamed from RV18; value HP_QMAX -> 100nF; footprint POGO_Potentiometer_SMD:Potentiometer_Bourns_3224W -> (none); symbol Device:R_POT -> Device:C
- C94: renamed from D12; value 1N4148W -> 100nF; footprint POGO_Diode_SMD:D_SOD-123 -> (none); symbol Device:D -> Device:C
- C96: renamed from C87; value 10nF -> 100nF
- C99: renamed from C88; value 10nF -> 100nF
- D12: renamed from R114; value 10k -> 1N4148W; footprint (none) -> POGO_Diode_SMD:D_SOD-123; symbol Device:R -> Device:D
- R104: renamed from R99; value 1k -> 1M
- R105: renamed from R100; value 100k -> 1M
- R110: renamed from R105; value 1M -> 47k
- R111: renamed from R106; value 100k -> 1k
- R112: renamed from R107; value 100k -> 10k
- R113: renamed from R108; value 100k -> 10k
- R114: renamed from R109; value 1M -> 10k
- R115: renamed from R110; value 47k -> 10k
- R30: renamed from C29D; value 47nF -> 100k; symbol Device:C -> Device:R
- R96: renamed from R95; value 100k -> 1k
- RV16: renamed from R111; value 1k -> HP_FREF; footprint (none) -> POGO_Potentiometer_SMD:Potentiometer_Bourns_3224W; symbol Device:R -> Device:R_POT
- RV17: renamed from R112; value 10k -> HP_1VOCT; footprint (none) -> POGO_Potentiometer_SMD:Potentiometer_Bourns_3224W; symbol Device:R -> Device:R_POT
- RV18: renamed from R113; value 10k -> HP_QMAX; footprint (none) -> POGO_Potentiometer_SMD:Potentiometer_Bourns_3224W; symbol Device:R -> Device:R_POT
- U53, U54, U66: footprint POGO_Package_SO:SOIC-8_3.9x4.9mm_P1.27mm -> (none)
- U53: renamed from U52; value LM13700 -> OPA1612; footprint POGO_Package_SO:SOIC-16_3.9x9.9mm_P1.27mm -> POGO_Package_SO:SOIC-8_3.9x4.9mm_P1.27mm; symbol Amplifier_Operational:LM13700 -> Amplifier_Operational:OPA1612
- U54: renamed from U53; footprint (none) -> POGO_Package_SO:SOIC-8_3.9x4.9mm_P1.27mm
- U55: renamed from U66; value TL072 -> THAT340; footprint (none) -> POGO_Package_SO:SOIC-14_3.9x8.7mm_P1.27mm; symbol Amplifier_Operational:OPA1612 -> POGO:THAT340
- U66: renamed from U54; value OPA1612 -> TL072; footprint (none) -> POGO_Package_SO:SOIC-8_3.9x4.9mm_P1.27mm
- renumbered C91 to C102, C92 to C103, C93 to C104, C94 to C105, C95 to C106, C29A to C29B, C29B to C29C, C29C to C29D, C86 to C95, R101 to R106, R102 to R107, R103 to R108, R104 to R109, R30 to R31, R31 to R92, R92 to R93, R93 to R94, R94 to R95, R96 to R97, R97 to R98, R98 to R99
Connections:
- net +12V: now also C101.2, C103.2, C105.2, C91.2, C93.2, C95.2, C99.2, R109.2, RV18.1, U53.4 (V-), U54.4 (V-), U66.4 (V-); no longer C102.2, C104.2, C106.2, C93.1, R114.2, U53.14 (In+_B), U54.4 (V-), U55.4 (V-), U66.4 (V-)
- net -12V: now also C100.2, C102.2, C104.2, C106.2, C92.2, C94.2, C96.2, R111.1, R112.1, R113.1, R114.1, R115.1, U53.8 (V+), U54.8 (V+), U55.11 (SUB), U55.4 (SUB), U66.8 (V+); no longer C103.2, C105.2, C29A.11 (SUB), C29A.4 (SUB), C86.1, D12.1, RV16.1, RV17.1, RV18.1, U53.3 (In+_A), U54.8 (V+), U55.8 (V+), U66.8 (V+)
- net BP_OUT_L: now also R30.2; no longer R31.2
- net BP_OUT_R: now also R31.2; no longer R92.2
- net GND: now also C29A.1, C86.1, C91.1, C92.1, C93.1, C94.1, D12.K, R96.1, RV18.3, U53.2 (In-), U54.2 (In-), U66.2 (In-); no longer C93.3, C94.K, R104.1, R30.1, U51.11 (V+), U51.12 (Out_B), U53.11 (V+), U53.12 (Out_B), U53.2 (In-), U53.6 (In-), U54.2 (In-), U54.6 (In-), U66.2 (In-)
- net HP_EXPO_BASE: now also RV17.1, U55.6 (Q3_B); no longer C29A.6 (Q3_B), C92.1
- net HP_EXPO_EMIT: now also R111.2, U55.10 (Q4_E), U55.5 (Q3_E); no longer C29A.10 (Q4_E), C29A.5 (Q3_E), RV16.2
- net HP_HPINV_L: now also R94.1, U53.1 (Out), U53.6 (In-); no longer R105.2, R95.1, U53.1 (Out)
- net HP_HPINV_R: now also R95.1, U54.1 (Out), U54.6 (In-); no longer R106.2, R96.1, U54.1 (Out)
- net HP_IABC: now also C87.2, C88.2, U55.7 (Q3_C); no longer C29A.7 (Q3_C), C96.2, C99.2
- net HP_IREF: now also C86.2, RV16.1, U55.8 (Q4_C), U55.9 (Q4_B); no longer C29A.8 (Q4_C), C29A.9 (Q4_B), C91.1, C95.2
- net HP_IREF_TR: now also R109.1, RV16.2 (Wiper), RV16.3; no longer C91.2 (Wiper), C91.3, R114.1
- net HP_IRES_SUM: now also R106.1, R107.1, R108.2, U66.3 (In+); no longer R111.1, R112.1, R113.2, U66.3 (In+)
- net HP_LIN_A_L: now also R96.2; no longer R97.2
- net HP_LIN_A_R: now also R98.2; no longer R99.2
- net HP_LIN_B_L: now also R97.2; no longer R98.2
- net HP_LIN_B_R: now also R99.2; no longer R104.2
- net HP_OUT_L: now also U53.5 (In+), U53.7 (Out); no longer R107.1, U53.7 (Out)
- net HP_OUT_R: now also U54.5 (In+), U54.7 (Out); no longer R108.1, U54.7 (Out)
- net HP_QIABC_L: now also C89.2, R104.1; no longer C100.2, R109.1
- net HP_QIABC_R: now also C90.2, R105.1, U51.9 (BufOut_B); no longer C101.2, R110.1, U53.8 (BufOut_A)
- net HP_RES: now also R107.2; no longer R112.2
- net HP_SUMINV_L: now also R30.1, R92.1, R94.2, U53.3 (In+); no longer R31.1, R93.1, R95.2, U53.3 (In+)
- net HP_SUMINV_R: now also R31.1, R93.1, R95.2, U51.12 (Out_B), U51.13 (In-_B), U54.3 (In+); no longer R92.1, R94.1, R96.2, U53.4 (In-_A), U53.5 (Out_A), U54.3 (In+)
- net HP_V1CAP_L: now also C29A.2; no longer C29B.2
- net HP_V1CAP_R: now also C29C.2; no longer C29D.2
- net HP_V1_L: now also R112.2; no longer RV17.2
- net HP_V1_R: now also R114.2, U51.11 (V+); no longer D12.2, U53.6 (V-)
- net HP_V2CAP_L: now also C29B.2; no longer C29C.2
- net HP_V2CAP_R: now also C29D.2; no longer R30.2
- net HP_V2_L: now also R113.2, R92.2; no longer R93.2, RV18.2
- net HP_V2_R: now also R115.2, R93.2; no longer C86.2, R94.2
- net HP_VBIAS: now also R106.2, RV18.2 (Wiper); no longer C93.2 (Wiper), R111.2
- net HP_VCTRL: now also R110.2; no longer R115.2
- net HP_VIRES: now also D12.A, R104.2, R105.2, R108.1, U66.1 (Out); no longer C94.A, R109.2, R110.2, R113.1, U66.1 (Out)
- net HP_VOCT_TR: now also R110.1, RV17.2 (Wiper), RV17.3; no longer C92.2 (Wiper), C92.3, R115.1
- removed net HP_INVBUF_L: R105.1, R107.2, U53.5 (In+)
- removed net HP_INVBUF_R: R106.1, R108.2, U54.5 (In+)
- removed net HP_QB_IABC_L: C87.2, U51.9 (BufOut_B)
- removed net HP_QB_IABC_R: C88.2, U53.9 (BufOut_B)
- removed net HP_QB_OUT_L: C89.2, U51.13 (In-_B)
- removed net HP_QB_OUT_R: C90.2, U53.13 (In-_B)
Other:
- moved on the sheet: U53B, U54B, U66B

Commit message: 0020 §A: expo V/oct divider fix - block-7 HP (template, tempco resolved)
First expo-divider fix (C1). block-7 HP (mono, 1 expo):
- R110 R_VOCT 47k->49.9k (E96; SPICE centers 17.92mV/oct = V_T*ln2 at mid-trim,
  sweeps 19.65..16.42 mV/V across RV17 -> symmetric +-10% authority).
- R229 tempco shunt (Vishay TFPT 1k, +4110ppm/K) HP_EXPO_BASE->GND. Resolves in
  BOM to TFPT0805L1001FM + POGO_Resistor_SMD footprint + datasheet (G6a/b paid off).
- Fixes the railed-expo bug: CV now sees ~18mV/oct at the base, not full V/oct.

block-7 schematic regenerated (57 parts/36 nets); all --check gates green.
This is the validated template for block-8 (mono) + block-5 (stereo, +tilt §B).

https://claude.ai/code/session_013jFXG5oeMVSYP7iRpwGvtQ
Parts:
- added C106: 100nF, symbol Device:C
- C86: renamed from C87; value 10nF -> 100nF
- C90: renamed from C91; value 100nF -> 10nF
- D12: renamed from C86; value 100nF -> 1N4148W; footprint (none) -> POGO_Diode_SMD:D_SOD-123; symbol Device:C -> Device:D
- R110: value 47k -> 49k9
- R115: renamed from RV16; value HP_FREF -> 10k; footprint POGO_Potentiometer_SMD:Potentiometer_Bourns_3224W -> (none); symbol Device:R_POT -> Device:R
- R229: renamed from R112; value 10k -> 1k; footprint (none) -> POGO_Resistor_SMD:R_0805_2012Metric
- RV16: renamed from RV17; value HP_1VOCT -> HP_FREF
- RV17: renamed from RV18; value HP_QMAX -> HP_1VOCT
- RV18: renamed from D12; value 1N4148W -> HP_QMAX; footprint POGO_Diode_SMD:D_SOD-123 -> POGO_Potentiometer_SMD:Potentiometer_Bourns_3224W; symbol Device:D -> Device:R_POT
- renumbered C101 to C100, C102 to C101, C103 to C102, C104 to C103, C105 to C104, C106 to C105, C88 to C87, C89 to C88, C90 to C89, C92 to C91, C93 to C92, C94 to C93, C95 to C94, C96 to C95, C99 to C96, C100 to C99, R113 to R112, R114 to R113, R115 to R114
Connections:
- net +12V: now also C101.2, C103.2, C105.2, C91.2, C93.2, C95.2, C99.2, RV18.1; no longer C100.2, C102.2, C104.2, C90.2, C92.2, C94.2, C96.2, RV17.1
- net -12V: now also C100.2, C102.2, C104.2, C92.2, C94.2, C96.2, R115.1, C106.2; no longer C101.2, C103.2, C105.2, C91.2, C93.2, C95.2, C99.2, R229.1
- net GND: now also D12.K, R229.1, RV18.3, C106.1; no longer D12.1, RV17.3, RV18.K
- net HP_EXPO_BASE: now also R229.2, RV17.1; no longer RV16.1
- net HP_IABC: now also C88.2; no longer C86.2
- net HP_IREF: now also C86.2, RV16.1; no longer D12.2, R115.1
- net HP_IREF_TR: now also RV16.2 (Wiper), RV16.3; no longer R115.2 (Wiper), R115.3
- net HP_QIABC_L: now also C89.2; no longer C88.2
- net HP_QIABC_R: now also C90.2; no longer C89.2
- net HP_V1_L: now also R112.2; no longer R229.2
- net HP_V1_R: now also R114.2; no longer R113.2
- net HP_V2_L: now also R113.2; no longer R112.2
- net HP_V2_R: now also R115.2; no longer R114.2
- net HP_VBIAS: now also RV18.2 (Wiper); no longer RV17.2 (Wiper)
- net HP_VIRES: now also D12.A; no longer RV18.A
- net HP_VOCT_TR: now also RV17.2 (Wiper), RV17.3; no longer RV16.2 (Wiper), RV16.3

Commit message: 0020 §C+§D: block-7 HP OTA tap + Q-cell R_Iabc
§C (H5): tap v1/v2 from the unbuffered LM13700 OTA outputs (pins 5/12), not the
Darlington buffers (8/9) which inject ~1.26V DC into the next OTA (SPICE
ota_svf_loop.cir). Removed R112-R115 buffer pulldowns; buffer pins 7/8/9/10 ->
no_connect. f_ref unchanged (cap still on OTA out).

§D/M5 (partial): R104/R105 R_Iabc 1M->100k (the LM13700 Iabc pin sits ~-10.8V,
not GND -> 1M delivered ~14x too much Iabc). The deeper negative-V_ires IRES_AMP
bias redesign + clamp-polarity flip is a Phase-3R/trim-backed [NV] item deferred
to the block-5 combined-edit pass (shares the same pattern); clamp D12 unchanged
meanwhile.

block-7 schematic regenerated (53 parts/32 nets); all --check gates green, 0 FAIL.

https://claude.ai/code/session_013jFXG5oeMVSYP7iRpwGvtQ
Parts:
- removed C103, C104, C105, C106: 100nF, symbol Device:C
- C86: renamed from RV16; value HP_FREF -> 100nF; footprint POGO_Potentiometer_SMD:Potentiometer_Bourns_3224W -> (none); symbol Device:R_POT -> Device:C
- C87: renamed from RV17; value HP_1VOCT -> 10nF; footprint POGO_Potentiometer_SMD:Potentiometer_Bourns_3224W -> (none); symbol Device:R_POT -> Device:C
- C88: renamed from RV18; value HP_QMAX -> 10nF; footprint POGO_Potentiometer_SMD:Potentiometer_Bourns_3224W -> (none); symbol Device:R_POT -> Device:C
- C89: renamed from D12; value 1N4148W -> 10nF; footprint POGO_Diode_SMD:D_SOD-123 -> (none); symbol Device:D -> Device:C
- C90: renamed from C86; value 100nF -> 10nF
- C91: renamed from C87; value 10nF -> 100nF
- C92: renamed from C88; value 10nF -> 100nF
- C93: renamed from C89; value 10nF -> 100nF
- C94: renamed from C90; value 10nF -> 100nF
- D12: renamed from R115; value 10k -> 1N4148W; footprint (none) -> POGO_Diode_SMD:D_SOD-123; symbol Device:R -> Device:D
- R104, R105: value 1M -> 100k
- RV16: renamed from R112; value 10k -> HP_FREF; footprint (none) -> POGO_Potentiometer_SMD:Potentiometer_Bourns_3224W; symbol Device:R -> Device:R_POT
- RV17: renamed from R113; value 10k -> HP_1VOCT; footprint (none) -> POGO_Potentiometer_SMD:Potentiometer_Bourns_3224W; symbol Device:R -> Device:R_POT
- RV18: renamed from R114; value 10k -> HP_QMAX; footprint (none) -> POGO_Potentiometer_SMD:Potentiometer_Bourns_3224W; symbol Device:R -> Device:R_POT
- renumbered C94 to C100, C95 to C101, C96 to C102, C99 to C103, C100 to C104, C101 to C105, C102 to C106, C91 to C95, C92 to C96, C93 to C99
Connections:
- net +12V: now also C91.2, C93.2, RV18.1; no longer C88.1
- net -12V: now also C92.2, C94.2; no longer D12.1, RV16.1, RV17.1, RV18.1
- net GND: now also C86.1, C87.1, C88.1, C89.1, D12.K, RV18.3; no longer C88.3, C89.K
- net HP_EXPO_BASE: now also RV17.1; no longer C87.1
- net HP_IABC: now also C87.2, C88.2; no longer C91.2, C92.2
- net HP_IREF: now also C86.2, RV16.1; no longer C86.1, C90.2
- net HP_IREF_TR: now also RV16.2 (Wiper), RV16.3; no longer C86.2 (Wiper), C86.3
- net HP_QIABC_L: now also C89.2; no longer C93.2
- net HP_QIABC_R: now also C90.2; no longer C94.2
- net HP_V1_L: now also C29A.2, U49.4 (In-_A); no longer RV16.2, U49.1 (Iabc_A)
- net HP_V1_R: now also C29C.2, U50.4 (In-_A); no longer RV18.2, U50.1 (Iabc_A)
- net HP_V2_L: now also C29B.2, U49.13 (In-_B); no longer RV17.2, U49.16 (Iabc_B)
- net HP_V2_R: now also C29D.2, U50.13 (In-_B); no longer D12.2, U50.16 (Iabc_B)
- net HP_VBIAS: now also RV18.2 (Wiper); no longer C88.2 (Wiper)
- net HP_VIRES: now also D12.A; no longer C89.A
- net HP_VOCT_TR: now also RV17.2 (Wiper), RV17.3; no longer C87.2 (Wiper), C87.3
- removed net HP_V1CAP_L: C29A.2, U49.2 (DiodeBias_A), U49.4 (In-_A)
- removed net HP_V1CAP_R: C29C.2, U50.2 (DiodeBias_A), U50.4 (In-_A)
- removed net HP_V2CAP_L: C29B.2, U49.13 (In-_B), U49.15 (DiodeBias_B)
- removed net HP_V2CAP_R: C29D.2, U50.13 (In-_B), U50.15 (DiodeBias_B)
