File: kicad/pogo-block-6-dist1.kicad_sch (KiCad schematic)
At the start: 62 parts, among them U31 CD4053, U34 TL072, U35 TL072, U40 TL072, U41 TL072, U75 CD4053

Commit message: 0018: block-6 stage 2 - distortion BEFORE bandpass (0017 reorder)
The core 0017 change: flip the per-band order from SVF->DIST to DIST->SVF to
match the plugin (Pogo.cpp:443-451). Realized as a net re-point across the 7
split sections (no part changes):
  LP1_OUT / BP3IN  ->  distN (R18/R20/R22 distortion inputs)
                   ->  mux out (BPn_DISTOUT)  ->  svfN SUM_AMP (R13)
                   ->  SVF v1 buffer (BPn_BANDOUT / BP3_TAP)  ->  mix wet summer
- BP1/BP2 take the LP1 band; BP3 takes BP3IN (the ALT/LP1 selector, stage 3).
- BP3 OUT tap now taken post-bandpass (BP3_TAP = svf3 v1), matching the plugin
  (prevOut[2]); block-B keeps the BP3_TAP net name (no block-B change).
- spec §1/§2 updated: signal order, DIST knob, ALT path (through-VCA/BP3-only),
  BP3 tap point.

Boundary symmetry verified for all re-pointed nets; all 5 --check gates +
parity green.

https://claude.ai/code/session_013jFXG5oeMVSYP7iRpwGvtQ
Connections:
- net BP1_BPBUF_L renamed LP1_OUT_L
- net BP1_BPBUF_R renamed LP1_OUT_R
- net BP1_DIST_L renamed BP1_DISTOUT_L
- net BP1_DIST_R renamed BP1_DISTOUT_R
Changed lines of the file:
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@@
   (effects (font (size 1.016 1.016)) (justify left))
 )
-(global_label "BP1_BPBUF_L"
+(global_label "LP1_OUT_L"
   (shape output)
   (at 40.000 373.810 0)
   (effects (font (size 1.016 1.016)) (justify left))
 )
-(global_label "BP1_BPBUF_L"
+(global_label "LP1_OUT_L"
   (shape output)
   (at 160.000 373.810 0)
   (effects (font (size 1.016 1.016)) (justify left))
 )
-(global_label "BP1_BPBUF_L"
+(global_label "LP1_OUT_L"
   (shape output)
   (at 100.000 428.810 0)
   (effects (font (size 1.016 1.016)) (justify left))
 )
-(global_label "BP1_BPBUF_L"
+(global_label "LP1_OUT_L"
   (shape output)
   (at 40.000 538.810 0)
   (effects (font (size 1.016 1.016)) (justify left))
 )
-(global_label "BP1_BPBUF_L"
+(global_label "LP1_OUT_L"
   (shape output)
   (at 100.000 538.810 0)
   (effects (font (size 1.016 1.016)) (justify left))
 )
-(global_label "BP1_BPBUF_R"
+(global_label "LP1_OUT_R"
   (shape output)
   (at 40.000 758.810 0)
   (effects (font (size 1.016 1.016)) (justify left))
 )
-(global_label "BP1_BPBUF_R"
+(global_label "LP1_OUT_R"
   (shape output)
   (at 160.000 758.810 0)
   (effects (font (size 1.016 1.016)) (justify left))
 )
-(global_label "BP1_BPBUF_R"
+(global_label "LP1_OUT_R"
   (shape output)
   (at 100.000 813.810 0)
   (effects (font (size 1.016 1.016)) (justify left))
 )
-(global_label "BP1_BPBUF_R"
+(global_label "LP1_OUT_R"
   (shape output)
   (at 40.000 923.810 0)
   (effects (font (size 1.016 1.016)) (justify left))
 )
-(global_label "BP1_BPBUF_R"
+(global_label "LP1_OUT_R"
   (shape output)
   (at 100.000 923.810 0)
@@
   (effects (font (size 1.016 1.016)) (justify left))
 )
-(global_label "BP1_DIST_L"
+(global_label "BP1_DISTOUT_L"
   (shape output)
   (at 48.890 50.160 0)
   (effects (font (size 1.016 1.016)) (justify left))
 )
-(global_label "BP1_DIST_R"
+(global_label "BP1_DISTOUT_R"
   (shape output)
   (at 48.890 42.540 0)

Commit message: 0018: block-6 stage 5 - variable DRIVE (THAT2180 VCA per band)
Build the per-band variable-drive stage the plugin needs (driveCv into the
waveshaper). A stereo THAT2180 current-in/I-V-out VCA per band, inserted at the
distortion input, mirroring the proven block-4 cell pin-for-pin:
  band -> R_in(20k) -> THAT2180.1 ; .8 -> TL074 I/V(-) + R_f(20k) -> BPn_DRIVEOUT
  -> SC/HC/WF cells.  Ec+ (pin2) via Bourns unity trim <- V_DRIVE_CTRL.
Drive control: per-band DRIVE knob (RV33/36/39) + DRIVE CV (MOD_BPn_DIST from
block-3) summed (TL074 half) into Ec+; knob=0.20 ~= unity. A single dB-law VGA
per band approximates the plugin's per-mode gain (SC exp vs HC/WF linear) -- a
documented deviation; exact knob->Ec+ dB law + unity bias are Phase-3R (like
block-4's Ec+ scaling).

Parts: +6 THAT2180 (U85-90), +3 TL074 (U91-93 I/V+summer), +6 Ec+ trims
(RV51-56), R153-176, decoupling. New boundary MOD_BPn_DIST; BPn_DRIVEOUT
internal. RV33/36/39 reused.

NOTE: the I/V stage inverts (as in block-4) -> one inversion added to the BP
wet path; reconcile in the S7 mix polarity-restore so wet sums with dry.

(An initial LM13700-OTA-VGA attempt was rolled back: its input wasn't scaled to
the OTA linear range -- would saturate on +-5V audio. Rebuilt on THAT2180 per
user.) All 5 --check gates + parity green; wiring reviewed vs block-4 template.

https://claude.ai/code/session_013jFXG5oeMVSYP7iRpwGvtQ
Parts:
- added C110_U85n, C110_U85p, C110_U86n, C110_U86p, C110_U91n, C110_U91p: 100nF, symbol Device:C
- added R153, R154, R155, R156: 20k, symbol Device:R
- added R157, R158, R159, R160: 100k, symbol Device:R
- added RV33: BP1_DIST, POGO_Potentiometer_THT:Potentiometer_Alpha_RD901F-40-00D_Single_Vertical_CircularHoles, symbol Device:R_POT
- added RV51: BP1_DRIVE_UNITY_L, POGO_Potentiometer_SMD:Potentiometer_Bourns_3224W, symbol Device:R_POT
- added RV52: BP1_DRIVE_UNITY_R, POGO_Potentiometer_SMD:Potentiometer_Bourns_3224W, symbol Device:R_POT
- added U85, U86: THAT2180, POGO_Package_SIP:SIP-8_2.54mm, symbol POGO:THAT2180
- added U91: TL074, symbol Amplifier_Operational:TL074
Connections:
- net +12V: now also C110_U85p.2, C110_U86p.2, C110_U91p.2, U85.5 (V-), U86.5 (V-), U91.11 (V-)
- net -12V: now also C110_U85n.2, C110_U86n.2, C110_U91n.2, U85.7 (V+), U86.7 (V+), U91.4 (V+)
- net GND: now also C110_U85n.1, C110_U85p.1, C110_U86n.1, C110_U86p.1, C110_U91n.1, C110_U91p.1, RV33.3, U85.1 (Input), U85.2 (Ec+), U85.3 (Ec-), U86.1 (Input), U86.2 (Ec+), U86.3 (Ec-), U91.13 (In-), U91.2 (In-), U91.6 (In-), U91.9 (In-)
- net LP1_OUT_L: now also R153.2; no longer C_WF_1La.2, C_WF_1Lb.2, R18_1L.2, R20_1L.2, R22_1L.2
- net LP1_OUT_R: now also R154.2; no longer C_WF_1Ra.2, C_WF_1Rb.2, R18_1R.2, R20_1R.2, R22_1R.2
- net V5LOGIC: now also R159.2, RV33.1
- new net BP1_DRIVEIN_L: R153.1, U85.6 (Gnd)
- new net BP1_DRIVEIN_R: R154.1, U86.6 (Gnd)
- new net BP1_DRIVEIV_L: R155.2, U91.3 (In+)
- new net BP1_DRIVEIV_R: R156.2, U91.5 (In+)
- new net BP1_DRIVEOUT_L: C_WF_1La.2, C_WF_1Lb.2, R155.1, R18_1L.2, R20_1L.2, R22_1L.2, U91.1 (Out)
- new net BP1_DRIVEOUT_R: C_WF_1Ra.2, C_WF_1Rb.2, R156.1, R18_1R.2, R20_1R.2, R22_1R.2, U91.7 (Out)
- new net BP1_DRIVE_KNOB: R157.2, RV33.2 (Wiper)
- new net BP1_DRIVE_SPARE: U91.12 (In+), U91.14 (Out)
- new net BP1_DRIVE_SUM: R157.1, R158.1, R159.1, R160.2, U91.10 (In+)
- new net EC_BP1_DRIVE_L: RV51.2 (Wiper), RV51.3, U85.4 (Sym)
- new net EC_BP1_DRIVE_R: RV52.2 (Wiper), RV52.3, U86.4 (Sym)
- new net MOD_BP1_DIST: R158.2
- new net V_DRIVE_CTRL_1: R160.1, RV51.1, RV52.1, U91.8 (Out)

Commit message: 0018: block-6 stage 6 - per-band CLIP LED drivers
The plugin lights BPn_CLIP when max(|distOut_L|,|distOut_R|) > 4V; the panel
has the CLIP LEDs but no hardware drove them. Build a per-band window
detector on the distortion output (BPn_DISTOUT_L/R, the CD4053 mux output):
- TL074 (U94/U95/U96) as 4 comparators per band: DISTOUT_L>+4, <-4,
  DISTOUT_R>+4, <-4, with ~2.2M hysteresis. Outputs diode-OR (D14_*) into
  the panel CLIP LED via a current-limit R.
- Shared +/-4V threshold from a 20k/10k divider off +/-12 (dist1), exported
  as VREF_P4/VREF_N4 boundary nets to dist2/dist3.
- CLIP LED component rows added for BP1/2/3.

All 5 --check gates + parity green. Exact threshold trim is Phase-3R.

https://claude.ai/code/session_013jFXG5oeMVSYP7iRpwGvtQ
Parts:
- added BP1_CLIP_LED: BP1_CLIP, POGO_LED_THT:LED_D3.0mm, symbol Device:LED
- added C110_U94n, C110_U94p, C111_N4, C111_P4: 100nF, symbol Device:C
- added D14_1a, D14_1b, D14_1c, D14_1d: 1N4148W, POGO_Diode_SMD:D_SOD-123, symbol Device:D
- added R177, R178, R179, R180, R190, R191: 100k, symbol Device:R
- added R181, R182, R183, R184: 2.2M, symbol Device:R
- added R185: 1k, symbol Device:R
- added R186, R188: 20k, symbol Device:R
- added R187, R189: 10k, symbol Device:R
- added U94: TL074, symbol Amplifier_Operational:TL074
Connections:
- net +12V: now also C110_U94p.2, R186.2, U94.11 (V-)
- net -12V: now also C110_U94n.2, R188.2, U94.4 (V+)
- net BP1_DISTOUT_L: now also R177.2, R178.2
- net BP1_DISTOUT_R: now also R179.2, R180.2
- net GND: now also BP1_CLIP_LED.A, C110_U94n.1, C110_U94p.1, C111_N4.1, C111_P4.1, R187.1, R189.1
- new net BP1_CLIP_A_INP: R177.1, R181.1, U94.2 (In-)
- new net BP1_CLIP_A_OUT: D14_1a.K, R181.2, U94.1 (Out)
- new net BP1_CLIP_B_INN: R178.1, U94.5 (In+)
- new net BP1_CLIP_B_INP: R182.1, R190.1, U94.6 (In-)
- new net BP1_CLIP_B_OUT: D14_1b.K, R182.2, U94.7 (Out)
- new net BP1_CLIP_C_INP: R179.1, R183.1, U94.9 (In-)
- new net BP1_CLIP_C_OUT: D14_1c.K, R183.2, U94.8 (Out)
- new net BP1_CLIP_D_INN: R180.1, U94.12 (In+)
- new net BP1_CLIP_D_INP: R184.1, R191.1, U94.13 (In-)
- new net BP1_CLIP_D_OUT: D14_1d.K, R184.2, U94.14 (Out)
- new net BP1_CLIP_LEDA: BP1_CLIP_LED.K, R185.1
- new net BP1_CLIP_OR: D14_1a.A, D14_1b.A, D14_1c.A, D14_1d.A, R185.2
- new net VREF_N4: C111_N4.2, R188.1, R189.2, R190.2, R191.2
- new net VREF_P4: C111_P4.2, R186.1, R187.2, U94.10 (In+), U94.3 (In+)

Commit message: 0020 HIGH-3: VCA Ec+ injection trims + V_CTRL buffer (10 cells, last cluster)
Replaced the useless series-rheostat-into-high-Z-Ec+ unity trims (~0.004dB
authority) with SPICE-validated voltage-injection trims across all 10 VCA cells:
- block-4 (4 cells: main L/R + ALT L/R): +U97 TL072 buffers the unbuffered AMT
  wiper -> V_CTRL_BUF -> 4x R_ec(10k) -> Ec+ (decouples the cells). Trims RV1/2/46/47
  500ohm->10k as dividers across a shared ±1.2V ref (R233/R234), wiper->R_inj(1M)->Ec+.
- block-6 dist1/2/3 (6 DRIVE cells): same injection trim; V_DRIVE_CTRL_n is already
  an op-amp output (low-Z) so no extra buffer - just per-section ±ref divider + R_ec/R_inj.
  RV51-56 500ohm->10k.
SPICE vca_ecplus_full.cir: g_ctrl 0.984, ±2dB unity authority, nulls bias offset.
New: U97, R233-R260, C117/C118; ~30 parts. All --check gates + JS/Py parity green,
0 schematic FAIL. (Absolute 6.1mV/dB is [NV], absorbed by the ±2dB trim.)

https://claude.ai/code/session_013jFXG5oeMVSYP7iRpwGvtQ
Parts:
- added C111_N4, C111_P4: 100nF, symbol Device:C
- added R186, R188: 20k, symbol Device:R
- added R187, R189: 10k, symbol Device:R
- BP1_CLIP_LED: renamed from C111_N4; value 100nF -> BP1_CLIP; footprint (none) -> POGO_LED_THT:LED_D3.0mm; symbol Device:C -> Device:LED
- C110_U85n, C110_U86n, C110_U86p, C110_U91p: renamed from U94; value TL074 -> 100nF; symbol Amplifier_Operational:TL074 -> Device:C
- C110_U85p: renamed from U94; value TL074 -> 100nF; footprint POGO_Package_SO:SOIC-14_3.9x8.7mm_P1.27mm -> (none); symbol Amplifier_Operational:TL074 -> Device:C
- C110_U94n: renamed from R182; value 2.2M -> 100nF; symbol Device:R -> Device:C
- C110_U94p: renamed from R181; value 2.2M -> 100nF; symbol Device:R -> Device:C
- D14_1a: renamed from R187; value 10k -> 1N4148W; footprint (none) -> POGO_Diode_SMD:D_SOD-123; symbol Device:R -> Device:D
- D14_1b: renamed from R188; value 20k -> 1N4148W; footprint (none) -> POGO_Diode_SMD:D_SOD-123; symbol Device:R -> Device:D
- D14_1c: renamed from R189; value 10k -> 1N4148W; footprint (none) -> POGO_Diode_SMD:D_SOD-123; symbol Device:R -> Device:D
- D14_1d: renamed from C111_P4; value 100nF -> 1N4148W; footprint (none) -> POGO_Diode_SMD:D_SOD-123; symbol Device:C -> Device:D
- R177: renamed from R183; value 2.2M -> 100k
- R178: renamed from R184; value 2.2M -> 100k
- R179: renamed from R185; value 1k -> 100k
- R181: renamed from R191; value 100k -> 2.2M
- R182: renamed from D14_1a; value 1N4148W -> 2.2M; footprint POGO_Diode_SMD:D_SOD-123 -> (none); symbol Device:D -> Device:R
- R183: renamed from D14_1b; value 1N4148W -> 2.2M; footprint POGO_Diode_SMD:D_SOD-123 -> (none); symbol Device:D -> Device:R
- R184: renamed from D14_1c; value 1N4148W -> 2.2M; footprint POGO_Diode_SMD:D_SOD-123 -> (none); symbol Device:D -> Device:R
- R185: renamed from D14_1d; value 1N4148W -> 1k; footprint POGO_Diode_SMD:D_SOD-123 -> (none); symbol Device:D -> Device:R
- R190: renamed from BP1_CLIP_LED; value BP1_CLIP -> 100k; footprint POGO_LED_THT:LED_D3.0mm -> (none); symbol Device:LED -> Device:R
- R191: renamed from R186; value 20k -> 100k
- R243: renamed from RV33; value BP1_DIST -> 45k3; footprint POGO_Potentiometer_THT:Potentiometer_Alpha_RD901F-40-00D_Single_Vertical_CircularHoles -> (none); symbol Device:R_POT -> Device:R
- R244: renamed from C110_U85p; value 100nF -> 45k3; symbol Device:C -> Device:R
- R245: renamed from C110_U85n; value 100nF -> 10k; symbol Device:C -> Device:R
- R246: renamed from C110_U86p; value 100nF -> 10k; symbol Device:C -> Device:R
- R247: renamed from C110_U86n; value 100nF -> 1M; symbol Device:C -> Device:R
- R248: renamed from C110_U91p; value 100nF -> 1M; symbol Device:C -> Device:R
- RV33: renamed from C110_U91n; value 100nF -> BP1_DIST; footprint (none) -> POGO_Potentiometer_THT:Potentiometer_Alpha_RD901F-40-00D_Single_Vertical_CircularHoles; symbol Device:C -> Device:R_POT
- U94: renamed from R179; value 100k -> TL074; symbol Device:R -> Amplifier_Operational:TL074
- U94: renamed from R178; value 100k -> TL074; symbol Device:R -> Amplifier_Operational:TL074
- U94: renamed from C110_U94n; value 100nF -> TL074; footprint (none) -> POGO_Package_SO:SOIC-14_3.9x8.7mm_P1.27mm; symbol Device:C -> Amplifier_Operational:TL074
- U94: renamed from R180; value 100k -> TL074; symbol Device:R -> Amplifier_Operational:TL074
- U94: renamed from R177; value 100k -> TL074; symbol Device:R -> Amplifier_Operational:TL074
- renumbered C110_U94p to C110_U91n, R190 to R180
Connections:
- net +12V: now also C110_U85p.2, C110_U86p.2, C110_U91p.2, C110_U94p.2, R243.2, U94.11 (V-), R186.2; no longer C110_U91n.2, C110_U91p.11 (V-), R191.2, R244.2, R246.2, R248.2
- net -12V: now also C110_U85n.2, C110_U86n.2, C110_U91n.2, C110_U94n.2, R244.2, U94.4 (V+), R188.2; no longer C110_U91p.4 (V+), D14_1b.2, R245.2, R247.2, RV33.2, U94.2
- net BP1_CLIP_A_INP: now also R177.1, R181.1, U94.2 (In-); no longer C110_U85p.2 (In-), C110_U94p.1, U94.1
- net BP1_CLIP_A_OUT: now also D14_1a.K, R181.2, U94.1 (Out); no longer C110_U85p.1 (Out), C110_U94p.2, R182.K
- net BP1_CLIP_B_INN: now also R178.1, U94.5 (In+); no longer C110_U85n.5 (In+), U94.1
- net BP1_CLIP_B_INP: now also R182.1, R190.1, U94.6 (In-); no longer C110_U85n.6 (In-), C110_U94n.1, R180.1
- net BP1_CLIP_B_OUT: now also D14_1b.K, R182.2, U94.7 (Out); no longer C110_U85n.7 (Out), C110_U94n.2, R183.K
- net BP1_CLIP_C_INP: now also R179.1, R183.1, U94.9 (In-); no longer C110_U86p.9 (In-), R177.1, U94.1
- net BP1_CLIP_C_OUT: now also D14_1c.K, R183.2, U94.8 (Out); no longer C110_U86p.8 (Out), R177.2, R184.K
- net BP1_CLIP_D_INN: now also R180.1, U94.12 (In+); no longer C110_U86n.12 (In+), U94.1
- net BP1_CLIP_D_INP: now also R184.1, R191.1, U94.13 (In-); no longer C110_U86n.13 (In-), R178.1, R181.1
- net BP1_CLIP_D_OUT: now also D14_1d.K, R184.2, U94.14 (Out); no longer C110_U86n.14 (Out), R178.2, R185.K
- net BP1_CLIP_LEDA: now also BP1_CLIP_LED.K, R185.1; no longer R179.1, R190.K
- net BP1_CLIP_OR: now also D14_1a.A, D14_1b.A, D14_1c.A, D14_1d.A, R185.2; no longer R179.2, R182.A, R183.A, R184.A, R185.A
- net BP1_DISTOUT_L: now also R177.2, R178.2; no longer U94.2, U94.2
- net BP1_DISTOUT_R: now also R179.2, R180.2; no longer U94.2, U94.2
- net BP1_DRIVE_KNOB: now also RV33.2 (Wiper); no longer R243.2 (Wiper)
- net EC_BP1_DRIVE_L: now also R245.1, R247.1; no longer RV51.2 (Wiper), RV51.3
- net EC_BP1_DRIVE_R: now also R246.1, R248.1; no longer RV52.2 (Wiper), RV52.3
- net GND: now also BP1_CLIP_LED.A, C110_U85n.1, C110_U85p.1, C110_U86n.1, C110_U86p.1, C110_U91p.1, C110_U94n.1, C110_U94p.1, RV33.3, C111_N4.1, C111_P4.1, R187.1, R189.1; no longer BP1_CLIP_LED.1, D14_1a.1, D14_1c.1, D14_1d.1, R190.A, R243.3, R244.1, R245.1, R246.1, R247.1, R248.1, RV33.1, U94.1
- net V5LOGIC: now also RV33.1; no longer R243.1
- net VREF_N4: now also R190.2, R191.2, C111_N4.2, R188.1, R189.2; no longer BP1_CLIP_LED.2, D14_1b.1, D14_1c.2, R180.2, R181.2
- net VREF_P4: now also U94.10 (In+), U94.3 (In+), C111_P4.2, R186.1, R187.2; no longer C110_U85p.3 (In+), C110_U86p.10 (In+), D14_1a.2, D14_1d.2, R191.1
- net V_DRIVE_CTRL_1: now also R245.2, R246.2; no longer RV51.1, RV52.1
- new net REF_N1: R244.1, RV51.1, RV52.1
- new net REF_P1: R243.1, RV51.3, RV52.3
- new net TRIMW_BP1_L: R247.2, RV51.2 (Wiper)
- new net TRIMW_BP1_R: R248.2, RV52.2 (Wiper)
Other:
- moved on the sheet: C110_U91n, U94E

Commit message: 0025: FIX the HIGH-3 ref-divider bug the SPICE-math gate found (block-4 + block-6)
ref_divider.cir derived REF_P from the actual netlist and got +-0.32V, not the
+-1.2V spec.md:166 + the 0020 HIGH-3 design claimed. Root cause (my error in
0020): R233/R234 sized 45.3k assuming a SINGLE 10k bridge, but all 4 unity trims
(RV1/RV2/RV46/RV47) load REF_P<->REF_N in PARALLEL = 2.5k -> REF_P collapses to
0.32V -> Ec+ injection authority was ~+-0.5dB, not the intended +-2dB. block-6
DRIVE refs had the same bug (2 pots = 5k bridge).

FIX:
- block-4: R233/R234 45k3->11k3 (-> +1.195V at the 2.5k load).
- block-6 dist1/2/3: R243/244/249/250/255/256 45k3->22k6 (-> +1.2V at the 5k load).
- ref_divider deck now pins +1.195V + binds R233=11k3, so a regression to 45k3
  FAILS the gate. Regenerated block-4/dist1/2/3 schematics + BOM.

All 7 --check gates green (incl. SPICE). Second real design error the SPICE-math
methodology has found; first to correct live netlist component values.

https://claude.ai/code/session_013jFXG5oeMVSYP7iRpwGvtQ
Parts:
- R243, R244: value 45k3 -> 22k6
Changed lines of the file:
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@@
   (property "Reference" "R243" (at 43.000 1418.000 0)
     (effects (font (size 1.27 1.27)) (justify left)))
-  (property "Value" "45k3" (at 43.000 1414.500 0)
+  (property "Value" "22k6" (at 43.000 1414.500 0)
     (effects (font (size 1.016 1.016)) (justify left) (hide yes)))
 )
@@
   (property "Reference" "R244" (at 103.000 1418.000 0)
     (effects (font (size 1.27 1.27)) (justify left)))
-  (property "Value" "45k3" (at 103.000 1414.500 0)
+  (property "Value" "22k6" (at 103.000 1414.500 0)
     (effects (font (size 1.016 1.016)) (justify left) (hide yes)))
 )
