File: kicad/pogo-block-6-dist3.kicad_sch (KiCad schematic)
At the start: 105 parts, among them U33 CD4053, U38 TL072, U39 TL072, U44 TL072, U45 TL072, U77 CD4053, U81 CD4053, U89 THAT2180, U90 THAT2180, U93 TL074, U96 TL074

Commit message: 0020 §E: make ALT_BP_L/R fully independent (Lane A plugin + hardware)
User direction: instead of a dual-switch jack (which would break the M8 panel
standard) to reproduce the R->L normal, make ALT L and R INDEPENDENT. This
dissolves the §E problem - each jack self-detects via its own switch lug, no
new part, no panel change, cleaner stereo behavior.

PLUGIN (Lane A; G3 pending in VCV Rack):
- Pogo.cpp: altR = altRConn ? PreGain(...) : 0 (dropped R->L normal);
  bp3InR = altRConn ? VcaBlock(...) : bandR (was altLConn||altRConn). L same.
- plugin.json 2.0.0 -> 2.1.0.

HARDWARE (follows):
- block-1: J4 mirrors J3 -> ALT_R_DET:[J4.3] + R225 22k tip pulldown; removed
  J4.3 from ALT_L_IN (R->L normal gone). New boundary ALT_R_DET.
- block-6-dist3: split U81 selects - X/L (pin11) stays ALT_L_DET; Y/R (pin10)
  now ALT_R_DET + R226 100k pull-up. New boundary ALT_R_DET.
- components.yaml +R225 +R226 (no new part type). Regenerated sch/BOM/viz.

All --check gates green; ALT_R_DET boundary resolves across both sheets.
Reclassifies 0020 as A/B mixed. Supersedes the dual-switch-jack plan.

https://claude.ai/code/session_013jFXG5oeMVSYP7iRpwGvtQ
Parts:
- added BP3_CLIP_LED: BP3_CLIP, POGO_LED_THT:LED_D3.0mm, symbol Device:LED
- C110_U93n: renamed from U96; value TL074 -> 100nF; footprint POGO_Package_SO:SOIC-14_3.9x8.7mm_P1.27mm -> (none); symbol Amplifier_Operational:TL074 -> Device:C
- C110_U96n: renamed from R203; value 100k -> 100nF; symbol Device:R -> Device:C
- D16_3d: renamed from BP3_CLIP_LED; value BP3_CLIP -> 1N4148W; footprint POGO_LED_THT:LED_D3.0mm -> POGO_Diode_SMD:D_SOD-123; symbol Device:LED -> Device:D
- R172: renamed from R173; value 100k -> 20k
- R176: renamed from RV55; value BP3_DRIVE_UNITY_L -> 100k; footprint POGO_Potentiometer_SMD:Potentiometer_Bourns_3224W -> (none); symbol Device:R_POT -> Device:R
- R206: renamed from R207; value 2.2M -> 100k
- R210: renamed from R211; value 1k -> 2.2M
- R211: renamed from R212; value 100k -> 1k
- R213: renamed from D16_3a; value 1N4148W -> 100k; footprint POGO_Diode_SMD:D_SOD-123 -> (none); symbol Device:D -> Device:R
- R226: renamed from U89; value THAT2180 -> 100k; footprint POGO_Package_SIP:SIP-8_2.54mm -> (none); symbol POGO:THAT2180 -> Device:R
- RV39: renamed from C110_U89p; value 100nF -> BP3_DIST; footprint (none) -> POGO_Potentiometer_THT:Potentiometer_Alpha_RD901F-40-00D_Single_Vertical_CircularHoles; symbol Device:C -> Device:R_POT
- RV55: renamed from RV56; value BP3_DRIVE_UNITY_R -> BP3_DRIVE_UNITY_L
- RV56: renamed from RV39; value BP3_DIST -> BP3_DRIVE_UNITY_R; footprint POGO_Potentiometer_THT:Potentiometer_Alpha_RD901F-40-00D_Single_Vertical_CircularHoles -> POGO_Potentiometer_SMD:Potentiometer_Bourns_3224W
- U90: renamed from U93; value TL074 -> THAT2180; footprint POGO_Package_SO:SOIC-14_3.9x8.7mm_P1.27mm -> POGO_Package_SIP:SIP-8_2.54mm; symbol Amplifier_Operational:TL074 -> POGO:THAT2180
- U93, U96: footprint (none) -> POGO_Package_SO:SOIC-14_3.9x8.7mm_P1.27mm
- U93: renamed from R169; value 20k -> TL074; symbol Device:R -> Amplifier_Operational:TL074
- U96: renamed from C110_U96p; value 100nF -> TL074; symbol Device:C -> Amplifier_Operational:TL074
- renumbered C110_U90p to C110_U89n, C110_U89n to C110_U89p, C110_U93p to C110_U90n, C110_U90n to C110_U90p, C110_U93n to C110_U93p, C110_U96n to C110_U96p, D16_3b to D16_3a, D16_3c to D16_3b, D16_3d to D16_3c, R170 to R169, R171 to R170, R172 to R171, R174 to R173, R175 to R174, R176 to R175, R204 to R203, R205 to R204, R206 to R205, R208 to R207, R209 to R208, R210 to R209, R213 to R212, U90 to U89
Connections:
- net +12V: now also C110_U89p.2, C110_U90p.2, C110_U93p.2, C110_U96p.2, R226.2, U90.5 (V-), U93.11 (V-), U96.11 (V-); no longer C110_U89n.2, C110_U90n.2, R226.5 (V-), RV39.2, U93.11 (V-), U96.11 (V-), U96.2
- net -12V: now also C110_U89n.2, C110_U90n.2, C110_U93n.2, C110_U96n.2, U90.7 (V+), U93.4 (V+), U96.4 (V+); no longer C110_U89p.2, C110_U90p.2, C110_U93p.2, C110_U96p.2, R226.7 (V+), U93.4 (V+), U96.4 (V+)
- net ALT_L_DET: no longer U81.8 (VSS)
- net BP3IN_L: now also R169.2; no longer U93.2
- net BP3IN_R: now also R170.2; no longer R169.2
- net BP3_CLIP_A_INP: now also R203.1, R207.1, U96.2 (In-); no longer C110_U93n.2 (In-), C110_U96n.1, R206.1
- net BP3_CLIP_A_OUT: now also D16_3a.K, R207.2, U96.1 (Out); no longer C110_U93n.1 (Out), R206.2, R213.K
- net BP3_CLIP_B_INN: now also R204.1, U96.5 (In+); no longer R203.1, U96.5 (In+)
- net BP3_CLIP_B_INP: now also R208.1, R212.1, U96.6 (In-); no longer R207.1, R211.1, U96.6 (In-)
- net BP3_CLIP_B_OUT: now also D16_3b.K, R208.2, U96.7 (Out); no longer D16_3a.K, R207.2, U96.7 (Out)
- net BP3_CLIP_C_INP: now also R205.1, R209.1, U96.9 (In-); no longer R204.1, R208.1, U96.9 (In-)
- net BP3_CLIP_C_OUT: now also D16_3c.K, R209.2, U96.8 (Out); no longer D16_3b.K, R208.2, U96.8 (Out)
- net BP3_CLIP_D_INN: now also R206.1, U96.12 (In+); no longer R205.1, U96.12 (In+)
- net BP3_CLIP_D_INP: now also R210.1, R213.1, U96.13 (In-); no longer R209.1, R212.1, U96.13 (In-)
- net BP3_CLIP_D_OUT: now also D16_3d.K, R210.2, U96.14 (Out); no longer D16_3c.K, R209.2, U96.14 (Out)
- net BP3_CLIP_LEDA: now also R211.1, BP3_CLIP_LED.K; no longer D16_3d.K, R210.1
- net BP3_CLIP_OR: now also D16_3d.A, R211.2; no longer R210.2, R213.A
- net BP3_DISTOUT_L: now also R204.2; no longer C110_U96n.2
- net BP3_DISTOUT_R: now also R206.2; no longer R204.2
- net BP3_DRIVEIN_L: now also R169.1, U89.6 (Gnd); no longer R226.6 (Gnd), U93.1
- net BP3_DRIVEIN_R: now also R170.1, U90.6 (Gnd); no longer R169.1, U89.6 (Gnd)
- net BP3_DRIVEIV_L: now also R171.2, U93.3 (In+); no longer R170.2, U90.3 (In+)
- net BP3_DRIVEIV_R: now also R172.2, U93.5 (In+); no longer R171.2, U93.5 (In+)
- net BP3_DRIVEOUT_L: now also R171.1, U93.1 (Out); no longer R170.1, U90.1 (Out)
- net BP3_DRIVEOUT_R: now also R172.1, U93.7 (Out); no longer R171.1, U93.7 (Out)
- net BP3_DRIVE_KNOB: now also R173.2, RV39.2 (Wiper); no longer R172.2, RV56.2 (Wiper)
- net BP3_DRIVE_SPARE: now also U93.12 (In+), U93.14 (Out); no longer U93.12 (In+), U93.14 (Out)
- net BP3_DRIVE_SUM: now also R175.1, R176.2, U93.10 (In+); no longer R172.1, R175.2, U93.10 (In+)
- net EC_BP3_DRIVE_L: now also RV55.2 (Wiper), RV55.3, U89.4 (Sym); no longer R176.2 (Wiper), R176.3, R226.4 (Sym)
- net EC_BP3_DRIVE_R: now also RV56.2 (Wiper), RV56.3, U90.4 (Sym); no longer RV55.2 (Wiper), RV55.3, U89.4 (Sym)
- net GND: now also C110_U93n.1, C110_U96n.1, RV39.3, U90.1 (Input), U90.3 (Ec-), U93.13 (In-), U93.2 (In-), U93.6 (In-), U93.9 (In-), BP3_CLIP_LED.A; no longer D16_3d.A, R226.1 (Input), R226.2 (Ec+), R226.3 (Ec-), RV39.1, RV56.3, U93.13 (In-), U93.6 (In-), U93.9 (In-), U96.1
- net MOD_BP3_DIST: now also R174.2; no longer R173.2
- net V5LOGIC: now also R175.2, RV39.1; no longer R174.2, RV56.1
- net VREF_N4: now also R213.2; no longer R211.2
- net VREF_P4: now also U96.10 (In+), U96.3 (In+); no longer C110_U93n.3 (In+), U96.10 (In+)
- net V_DRIVE_CTRL_3: now also RV56.1, U93.8 (Out); no longer R175.1, U93.8 (Out)
- new net ALT_R_DET: R226.1, U81.8 (VSS)
Other:
- moved on the sheet: U93A, U93B, U93C, U93E, U96A, U96B, U96C

Commit message: 0020 HIGH-3: VCA Ec+ injection trims + V_CTRL buffer (10 cells, last cluster)
Replaced the useless series-rheostat-into-high-Z-Ec+ unity trims (~0.004dB
authority) with SPICE-validated voltage-injection trims across all 10 VCA cells:
- block-4 (4 cells: main L/R + ALT L/R): +U97 TL072 buffers the unbuffered AMT
  wiper -> V_CTRL_BUF -> 4x R_ec(10k) -> Ec+ (decouples the cells). Trims RV1/2/46/47
  500ohm->10k as dividers across a shared ±1.2V ref (R233/R234), wiper->R_inj(1M)->Ec+.
- block-6 dist1/2/3 (6 DRIVE cells): same injection trim; V_DRIVE_CTRL_n is already
  an op-amp output (low-Z) so no extra buffer - just per-section ±ref divider + R_ec/R_inj.
  RV51-56 500ohm->10k.
SPICE vca_ecplus_full.cir: g_ctrl 0.984, ±2dB unity authority, nulls bias offset.
New: U97, R233-R260, C117/C118; ~30 parts. All --check gates + JS/Py parity green,
0 schematic FAIL. (Absolute 6.1mV/dB is [NV], absorbed by the ±2dB trim.)

https://claude.ai/code/session_013jFXG5oeMVSYP7iRpwGvtQ
Parts:
- added BP3_CLIP_LED: BP3_CLIP, POGO_LED_THT:LED_D3.0mm, symbol Device:LED
- added D16_3a, D16_3b, D16_3c, D16_3d: 1N4148W, POGO_Diode_SMD:D_SOD-123, symbol Device:D
- added R213: 100k, symbol Device:R
- C110_U89n, C110_U90n, C110_U90p, C110_U93p: renamed from U96; value TL074 -> 100nF; symbol Amplifier_Operational:TL074 -> Device:C
- C110_U89p: renamed from U96; value TL074 -> 100nF; footprint POGO_Package_SO:SOIC-14_3.9x8.7mm_P1.27mm -> (none); symbol Amplifier_Operational:TL074 -> Device:C
- C110_U96n: renamed from R208; value 2.2M -> 100nF; symbol Device:R -> Device:C
- C110_U96p: renamed from R207; value 2.2M -> 100nF; symbol Device:R -> Device:C
- R203: renamed from R209; value 2.2M -> 100k
- R204: renamed from R210; value 2.2M -> 100k
- R205: renamed from R211; value 1k -> 100k
- R207: renamed from R213; value 100k -> 2.2M
- R208: renamed from D16_3a; value 1N4148W -> 2.2M; footprint POGO_Diode_SMD:D_SOD-123 -> (none); symbol Device:D -> Device:R
- R209: renamed from D16_3b; value 1N4148W -> 2.2M; footprint POGO_Diode_SMD:D_SOD-123 -> (none); symbol Device:D -> Device:R
- R210: renamed from D16_3c; value 1N4148W -> 2.2M; footprint POGO_Diode_SMD:D_SOD-123 -> (none); symbol Device:D -> Device:R
- R211: renamed from D16_3d; value 1N4148W -> 1k; footprint POGO_Diode_SMD:D_SOD-123 -> (none); symbol Device:D -> Device:R
- R212: renamed from BP3_CLIP_LED; value BP3_CLIP -> 100k; footprint POGO_LED_THT:LED_D3.0mm -> (none); symbol Device:LED -> Device:R
- R255: renamed from RV39; value BP3_DIST -> 45k3; footprint POGO_Potentiometer_THT:Potentiometer_Alpha_RD901F-40-00D_Single_Vertical_CircularHoles -> (none); symbol Device:R_POT -> Device:R
- R256: renamed from C110_U89p; value 100nF -> 45k3; symbol Device:C -> Device:R
- R257: renamed from C110_U89n; value 100nF -> 10k; symbol Device:C -> Device:R
- R258: renamed from C110_U90p; value 100nF -> 10k; symbol Device:C -> Device:R
- R259: renamed from C110_U90n; value 100nF -> 1M; symbol Device:C -> Device:R
- R260: renamed from C110_U93p; value 100nF -> 1M; symbol Device:C -> Device:R
- RV39: renamed from C110_U93n; value 100nF -> BP3_DIST; footprint (none) -> POGO_Potentiometer_THT:Potentiometer_Alpha_RD901F-40-00D_Single_Vertical_CircularHoles; symbol Device:C -> Device:R_POT
- U96: renamed from R205; value 100k -> TL074; symbol Device:R -> Amplifier_Operational:TL074
- U96: renamed from R203; value 100k -> TL074; symbol Device:R -> Amplifier_Operational:TL074
- U96: renamed from R206; value 100k -> TL074; symbol Device:R -> Amplifier_Operational:TL074
- U96: renamed from C110_U96n; value 100nF -> TL074; footprint (none) -> POGO_Package_SO:SOIC-14_3.9x8.7mm_P1.27mm; symbol Device:C -> Amplifier_Operational:TL074
- U96: renamed from R204; value 100k -> TL074; symbol Device:R -> Amplifier_Operational:TL074
- renumbered C110_U96p to C110_U93n, R212 to R206
Connections:
- net +12V: now also C110_U89p.2, C110_U90p.2, C110_U93p.2, C110_U96p.2, R255.2, U96.11 (V-); no longer C110_U93n.2, C110_U93p.11 (V-), R256.2, R258.2, R260.2
- net -12V: now also C110_U89n.2, C110_U90n.2, C110_U93n.2, C110_U96n.2, R256.2, U96.4 (V+); no longer C110_U93p.4 (V+), R257.2, R259.2, RV39.2, U96.2
- net BP3_CLIP_A_INP: now also R203.1, R207.1, U96.2 (In-); no longer C110_U89p.2 (In-), C110_U96p.1, U96.1
- net BP3_CLIP_A_OUT: now also R207.2, U96.1 (Out), D16_3a.K; no longer C110_U89p.1 (Out), C110_U96p.2, R208.K
- net BP3_CLIP_B_INN: now also R204.1, U96.5 (In+); no longer C110_U89n.5 (In+), U96.1
- net BP3_CLIP_B_INP: now also R208.1, R212.1, U96.6 (In-); no longer C110_U89n.6 (In-), C110_U96n.1, R206.1
- net BP3_CLIP_B_OUT: now also R208.2, U96.7 (Out), D16_3b.K; no longer C110_U89n.7 (Out), C110_U96n.2, R209.K
- net BP3_CLIP_C_INP: now also R205.1, R209.1, U96.9 (In-); no longer C110_U90p.9 (In-), R203.1, U96.1
- net BP3_CLIP_C_OUT: now also R209.2, U96.8 (Out), D16_3c.K; no longer C110_U90p.8 (Out), R203.2, R210.K
- net BP3_CLIP_D_INN: now also R206.1, U96.12 (In+); no longer C110_U90n.12 (In+), U96.1
- net BP3_CLIP_D_INP: now also R210.1, U96.13 (In-), R213.1; no longer C110_U90n.13 (In-), R204.1, R207.1
- net BP3_CLIP_D_OUT: now also R210.2, U96.14 (Out), D16_3d.K; no longer C110_U90n.14 (Out), R204.2, R211.K
- net BP3_CLIP_LEDA: now also R211.1, BP3_CLIP_LED.K; no longer R205.1, R212.K
- net BP3_CLIP_OR: now also R211.2, D16_3a.A, D16_3b.A, D16_3c.A, D16_3d.A; no longer R205.2, R208.A, R209.A, R210.A, R211.A
- net BP3_DISTOUT_L: now also R203.2, R204.2; no longer U96.2, U96.2
- net BP3_DISTOUT_R: now also R205.2, R206.2; no longer U96.2, U96.2
- net BP3_DRIVE_KNOB: now also RV39.2 (Wiper); no longer R255.2 (Wiper)
- net EC_BP3_DRIVE_L: now also R257.1, R259.1; no longer RV55.2 (Wiper), RV55.3
- net EC_BP3_DRIVE_R: now also R258.1, R260.1; no longer RV56.2 (Wiper), RV56.3
- net GND: now also C110_U89n.1, C110_U89p.1, C110_U90n.1, C110_U90p.1, C110_U93p.1, C110_U96n.1, C110_U96p.1, RV39.3, BP3_CLIP_LED.A; no longer R212.A, R255.3, R256.1, R257.1, R258.1, R259.1, R260.1, RV39.1, U96.1
- net V5LOGIC: now also RV39.1; no longer R255.1
- net VREF_N4: now also R212.2, R213.2; no longer R206.2, R207.2
- net VREF_P4: now also U96.10 (In+), U96.3 (In+); no longer C110_U89p.3 (In+), C110_U90p.10 (In+)
- net V_DRIVE_CTRL_3: now also R257.2, R258.2; no longer RV55.1, RV56.1
- new net REF_N3: R256.1, RV55.1, RV56.1
- new net REF_P3: R255.1, RV55.3, RV56.3
- new net TRIMW_BP3_L: R259.2, RV55.2 (Wiper)
- new net TRIMW_BP3_R: R260.2, RV56.2 (Wiper)
Other:
- moved on the sheet: C110_U93n, U96E

Commit message: 0025: FIX the HIGH-3 ref-divider bug the SPICE-math gate found (block-4 + block-6)
ref_divider.cir derived REF_P from the actual netlist and got +-0.32V, not the
+-1.2V spec.md:166 + the 0020 HIGH-3 design claimed. Root cause (my error in
0020): R233/R234 sized 45.3k assuming a SINGLE 10k bridge, but all 4 unity trims
(RV1/RV2/RV46/RV47) load REF_P<->REF_N in PARALLEL = 2.5k -> REF_P collapses to
0.32V -> Ec+ injection authority was ~+-0.5dB, not the intended +-2dB. block-6
DRIVE refs had the same bug (2 pots = 5k bridge).

FIX:
- block-4: R233/R234 45k3->11k3 (-> +1.195V at the 2.5k load).
- block-6 dist1/2/3: R243/244/249/250/255/256 45k3->22k6 (-> +1.2V at the 5k load).
- ref_divider deck now pins +1.195V + binds R233=11k3, so a regression to 45k3
  FAILS the gate. Regenerated block-4/dist1/2/3 schematics + BOM.

All 7 --check gates green (incl. SPICE). Second real design error the SPICE-math
methodology has found; first to correct live netlist component values.

https://claude.ai/code/session_013jFXG5oeMVSYP7iRpwGvtQ
Parts:
- R255, R256: value 45k3 -> 22k6
Changed lines of the file:
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@@
   (property "Reference" "R255" (at 163.000 1473.000 0)
     (effects (font (size 1.27 1.27)) (justify left)))
-  (property "Value" "45k3" (at 163.000 1469.500 0)
+  (property "Value" "22k6" (at 163.000 1469.500 0)
     (effects (font (size 1.016 1.016)) (justify left) (hide yes)))
 )
@@
   (property "Reference" "R256" (at 43.000 1528.000 0)
     (effects (font (size 1.27 1.27)) (justify left)))
-  (property "Value" "45k3" (at 43.000 1524.500 0)
+  (property "Value" "22k6" (at 43.000 1524.500 0)
     (effects (font (size 1.016 1.016)) (justify left) (hide yes)))
 )
